File: misko.sch (EAGLE design)
At the start: 0 parts

Commit message: - ongoing conversion of splan schematic into eagle
Parts:
- added C1: (no value), resistor:C-EUC1206
- added C2, C4, C5, C7, C8, C9: 0.47µF, resistor:C-EUC0805
- added C3: 0.1µF, resistor:C-EUC1206
- added C6: 0.1µF, resistor:C-EUC0805
- added IC1: MC1525TT, microchip:MC1525TT
- added IC2: FT230XS, ftdichip:FT230XS
- added LED1: (no value), led:LEDSML1206
- added LED2, LED3: yellow, led:LEDSML1206
- added R1: (no value), resistor:R-EU_R1206
- added R10, R12, R16, R17, R18, R8: 47k, rcl:R-EU_R0805
- added R11, R13, R19, R20, R21, R9: 1k, rcl:R-EU_R0805
- added R14, R15: 21, rcl:R-EU_R0805
- added R2, R3: 3k3, rcl:R-EU_R0805
- added R4, R5: 1k, resistor:R-EU_R1206
- added R6, R7: 21, resistor:R-EU_R1206
- added S1: up, switch-omron:10-XX
- added S2: GPRS push, switch-omron:10-XX
- added S3: right, switch-omron:10-XX
- added S4: left, switch-omron:10-XX
- added S5: Bluetooth, switch-omron:10-XX
- added S6: down, switch-omron:10-XX
- added U1: ATMEGA1281-16AU, Atmel_By_element14_Batch_1-00:ATMEGA1281-16AU
- added U2: SN74HCT14DR, Texas Instruments_By_element14_Batch_1:SN74HCT14DR
- added U3: SN74LVC1G3157DBVR - BT switch, Texas Instruments_By_element14_Batch_1:SN74LVC1G3157DBVR
- added U4: SN74LVC1G3157DBVR - GPS switch, Texas Instruments_By_element14_Batch_1:SN74LVC1G3157DBVR
- added U5: TMP36GRTZ-REEL7, TMP36GRTZ:TMP36GRTZ-REEL7
- added U6: TPS63030DSKT, Texas Instruments_By_element14_Batch_1:TPS63030DSKT
- added U7: MCP73871-2AAI/ML, Microchip-MCP73871-2AAI_ML:MCP73871-2AAI/ML
Connections:
- new net 5V0: IC2.VCC
- new net ADXL345_INT1_INTERRUPT_PIN: U1.(ICP3/CLKO/INT7)_PE7
- new net ANALOG_SW_CTRL_PIN: U1.(TOSC2)_PG3, U3.S, U4.S
- new net BAT_A_PIN: U1.PF3_(ADC3)
- new net BLUETOOTH_TX: U4.B1
- new net BLUETOOTH_WAKEUP_PIN: U1.(OC0A/OC1C/PCINT7)_PB7
- new net GND: C2.1, C3.2, C4.1, C5.1, C7.1, C8.1, C9.1, IC2.GND, IC2.GND@1, R16.1, R17.1, R18.1, R19.1, R21.1, S1.P, S1.P1, S2.P, S2.P1, S3.P, S3.P1, S4.P, S4.P1, S4.S, S4.S1, S5.P, S5.P1, S5.S, S5.S1, S6.P, S6.P1, S6.S, S6.S1, U1.GND, U1.GND_2, U1.GND_3, U2.GND, U3.GND
- new net GPS_GREEN_LED_PIN: U1.PC7_(A15)
- new net GPS_POWER_CTL_PIN: U1.(T0)_PD7
- new net GPS_RED_LED_PIN: U1.PC6_(A14)
- new net GPS_SW_SERIAL_RX: U1.(OC2A/_PCINT4)_PB4, U3.B2, U4.A
- new net GPS_SW_SERIAL_TX: U1.(OC1A/PCINT5)_PB5, U3.B1
- new net GPS_TX: U4.B2
- new net GPS_WAKEUP_PIN: U1.(TOSC1)_PG4
- new net I2C_SCL_PIN: U1.(SCL/INT0)_PD0
- new net I2C_SDA_PIN: U1.(SDA/INT1)_PD1
- new net JTAG_TCL_PIN: U1.PF4_(ADC4/TCK)
- new net JTAG_TDI_PIN: U1.PF7_(ADC7/TDI)
- new net JTAG_TDO_PIN: U1.PF6_(ADC6/TDO)
- new net JTAG_TMS_PIN: U1.PF5_(ADC5/TMS)
- new net MCP73871_CHARGE_STATUS_1_PIN: U1.PA2_(AD2)
- new net MCP73871_CHARGE_STATUS_2_PIN: U1.PA1_(AD1)
- new net MCP73871_POWER_GOOD_PIN: U1.PA0_(AD0)
- new net MENU_BLUETOOTH_POWER_TOGGLE_PIN: U1.PC1_(A9), U2.5Y
- new net MENU_DOWN_BUTTON_PIN: U1.PC2_(A10), U2.6Y
- new net MENU_GPRS_PUSH_BUTTON_PIN: U1.PC4_(A12), U2.2Y
- new net MENU_LEFT_BUTTON_PIN: U1.PC0_(A8), U2.4Y
- new net MENU_RIGHT_BUTTON_PIN: U1.PC5_(A13), U2.3Y
- new net MENU_UP_BUTTON_PIN: U1.PC3_(A11), U2.1Y
- new net N$1: IC1.GND
- new net N$10: C3.1, IC2.!RESET, IC2.3V3OUT, IC2.VCCIO
- new net N$12: U5.GND
- new net N$14: R8.1, R9.1, S1.S, S1.S1
- new net N$16: R12.1, R13.1, S3.S, S3.S1
- new net N$2: U4.GND
- new net N$21: R10.1, R11.1, S2.S, S2.S1
- new net N$3: IC2.TXD, R2.2
- new net N$4: IC2.CBUS2, LED3.C
- new net N$5: IC2.CBUS1, LED2.C
- new net N$6: LED3.A, R4.2
- new net N$7: IC2.USBDP, R7.2
- new net N$8: LED2.A, R5.1
- new net N$9: IC2.USBDM, R6.1
- new net PDI_UART0_CTS_PIN: IC2.!CTS, U1.(OC0B)_PG5
- new net PDI_UART0_RX_PIN: R2.1, U1.(RXD0/PCINT8/PDI)_PE0
- new net PDI_UART0_TX_PIN: IC2.RXD, R3.1, R3.2, U1.(TXD0/PDO)_PE1
- new net S1: C2.2, R8.2, U2.1A
- new net S2: C4.2, R10.2, U2.2A
- new net S3: C5.2, R12.2, U2.3A
- new net S4: C7.2, R18.2, U2.4A
- new net S5: C8.2, R17.2, U2.5A
- new net S6: C9.2, R16.2, U2.6A
- new net SD_CARD_DETECT_PIN: U1.(OC1B/PCINT6)_PB6
- new net SIM800C_CTS_PIN: U1.(ICP1)_PD4
- new net SIM800C_POWER_PIN: U1.(T1)_PD6
- new net SIM800C_RX_PIN: U1.(RXD1/INT2)_PD2
- new net SIM800C_STATUS_PIN: U1.(XCK1)_PD5
- new net SIM800C_TX_PIN: U1.(TXD1/INT3)_PD3
- new net SPI_FRAM_SS_PIN: U1.(~SS/PCINT0)_PB0
- new net SPI_MISO_PIN: U1.(MISO/PCINT3)_PB3
- new net SPI_MOSI_PIN: U1.(MOSI/PCINT2)_PB2
- new net SPI_OLED_A0_PIN: U1.(OC3B/INT4)_PE4
- new net SPI_OLED_RESET_PIN: U1.(OC3A/AIN1)_PE3
- new net SPI_SCK_PIN: U1.(SCK/PCINT1)_PB1
- new net SPI_SS_ADXL345_PIN: U1.(XCK0/AIN0)_PE2
- new net SPI_SS_OLED_PIN: U1.(OC3C/INT5)_PE5
- new net SPI_SS_SD_CARD_PIN: U1.(T3/INT6)_PE6
- new net TMP36_SHUTDOWN_PIN: U1.PA3_(AD3), U5.~SHDN
- new net TMP36_VSENSE_PIN: U1.PF0_(ADC0), U5.VOUT
- new net USB_D+: R7.1
- new net USB_D-: R6.2
- new net VCC: IC1.VIN, R11.2, R13.2, R19.2, R20.2, R21.2, R9.2, U1.VCC, U1.VCC_2, U2.VCC, U3.VCC, U4.VCC, U5.+VS
- new net VCC_SENSE_PIN: U1.PF1_(ADC1)
- new net V_USB: R4.1, R5.2
Other:
- note added: "Keyboard"
