File: misko_3_board.sch (EAGLE design)
At the start: 165 parts, among them CN1 LiPo Battery, IC1 MC1525TT, IC2 FT230XS, IC3 LTC4425, IC4 FM25W256-SOIC, M10 mid, Q1 FDN304P, T10 top, U1 ATMEGA1281-16AU, U2 SN74HCT14DR, U3 SN74LVC1G3157DBVR - BT switch, U4 SN74LVC1G3157DBVR - GPS switch, U5 TMP36GRTZ-REEL7, U7 MCP73871-2AAI/ML, X3 FH12-24S-0.5SH

Commit message: - replaced JST-PH with through-hole variant
Parts:
- CN1: device SIM800C:JST_2PIN-SMT -> SIM800C:JST_2PIN-THM-RA
Changed lines of the file:
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@@
 <grid distance="0.1" unitdist="inch" unit="inch" style="lines" multiple="1" display="yes" altdistance="0.01" altunitdist="inch" altunit="inch"/>
 <layers>
-<layer number="1" name="Top" color="4" fill="1" visible="no" active="no"/>
-<layer number="2" name="Route2" color="1" fill="3" visible="no" active="no"/>
-<layer number="3" name="Route3" color="4" fill="3" visible="no" active="no"/>
-<layer number="4" name="Route4" color="1" fill="4" visible="no" active="no"/>
-<layer number="5" name="Route5" color="4" fill="4" visible="no" active="no"/>
-<layer number="6" name="Route6" color="1" fill="8" visible="no" active="no"/>
-<layer number="7" name="Route7" color="4" fill="8" visible="no" active="no"/>
-<layer number="8" name="Route8" color="1" fill="2" visible="no" active="no"/>
-<layer number="9" name="Route9" color="4" fill="2" visible="no" active="no"/>
-<layer number="10" name="Route10" color="1" fill="7" visible="no" active="no"/>
-<layer number="11" name="Route11" color="4" fill="7" visible="no" active="no"/>
-<layer number="12" name="Route12" color="1" fill="5" visible="no" active="no"/>
-<layer number="13" name="Route13" color="4" fill="5" visible="no" active="no"/>
-<layer number="14" name="Route14" color="1" fill="6" visible="no" active="no"/>
-<layer number="15" name="Route15" color="4" fill="6" visible="no" active="no"/>
-<layer number="16" name="Bottom" color="1" fill="1" visible="no" active="no"/>
-<layer number="17" name="Pads" color="2" fill="1" visible="no" active="no"/>
-<layer number="18" name="Vias" color="2" fill="1" visible="no" active="no"/>
-<layer number="19" name="Unrouted" color="6" fill="1" visible="no" active="no"/>
-<layer number="20" name="Dimension" color="15" fill="1" visible="no" active="no"/>
-<layer number="21" name="tPlace" color="7" fill="1" visible="no" active="no"/>
-<layer number="22" name="bPlace" color="7" fill="1" visible="no" active="no"/>
-<layer number="23" name="tOrigins" color="15" fill="1" visible="no" active="no"/>
-<layer number="24" name="bOrigins" color="15" fill="1" visible="no" active="no"/>
-<layer number="25" name="tNames" color="7" fill="1" visible="no" active="no"/>
-<layer number="26" name="bNames" color="7" fill="1" visible="no" active="no"/>
-<layer number="27" name="tValues" color="7" fill="1" visible="no" active="no"/>
-<layer number="28" name="bValues" color="7" fill="1" visible="no" active="no"/>
+<layer number="1" name="Top" color="4" fill="1" visible="yes" active="no"/>
+<layer number="2" name="Route2" color="1" fill="3" visible="yes" active="no"/>
+<layer number="3" name="Route3" color="4" fill="3" visible="yes" active="no"/>
+<layer number="4" name="Route4" color="1" fill="4" visible="yes" active="no"/>
+<layer number="5" name="Route5" color="4" fill="4" visible="yes" active="no"/>
+<layer number="6" name="Route6" color="1" fill="8" visible="yes" active="no"/>
+<layer number="7" name="Route7" color="4" fill="8" visible="yes" active="no"/>
+<layer number="8" name="Route8" color="1" fill="2" visible="yes" active="no"/>
+<layer number="9" name="Route9" color="4" fill="2" visible="yes" active="no"/>
+<layer number="10" name="Route10" color="1" fill="7" visible="yes" active="no"/>
+<layer number="11" name="Route11" color="4" fill="7" visible="yes" active="no"/>
+<layer number="12" name="Route12" color="1" fill="5" visible="yes" active="no"/>
+<layer number="13" name="Route13" color="4" fill="5" visible="yes" active="no"/>
+<layer number="14" name="Route14" color="1" fill="6" visible="yes" active="no"/>
+<layer number="15" name="Route15" color="4" fill="6" visible="yes" active="no"/>
+<layer number="16" name="Bottom" color="1" fill="1" visible="yes" active="no"/>
+<layer number="17" name="Pads" color="2" fill="1" visible="yes" active="no"/>
+<layer number="18" name="Vias" color="2" fill="1" visible="yes" active="no"/>
+<layer number="19" name="Unrouted" color="6" fill="1" visible="yes" active="no"/>
+<layer number="20" name="Dimension" color="15" fill="1" visible="yes" active="no"/>
+<layer number="21" name="tPlace" color="7" fill="1" visible="yes" active="no"/>
+<layer number="22" name="bPlace" color="7" fill="1" visible="yes" active="no"/>
+<layer number="23" name="tOrigins" color="15" fill="1" visible="yes" active="no"/>
+<layer number="24" name="bOrigins" color="15" fill="1" visible="yes" active="no"/>
+<layer number="25" name="tNames" color="7" fill="1" visible="yes" active="no"/>
+<layer number="26" name="bNames" color="7" fill="1" visible="yes" active="no"/>
+<layer number="27" name="tValues" color="7" fill="1" visible="yes" active="no"/>
+<layer number="28" name="bValues" color="7" fill="1" visible="yes" active="no"/>
 <layer number="29" name="tStop" color="7" fill="3" visible="no" active="no"/>
 <layer number="30" name="bStop" color="7" fill="6" visible="no" active="no"/>
@@
 <layer number="35" name="tGlue" color="7" fill="4" visible="no" active="no"/>
 <layer number="36" name="bGlue" color="7" fill="5" visible="no" active="no"/>
-<layer number="37" name="tTest" color="7" fill="1" visible="no" active="no"/>
-<layer number="38" name="bTest" color="7" fill="1" visible="no" active="no"/>
+<layer number="37" name="tTest" color="7" fill="1" visible="yes" active="no"/>
+<layer number="38" name="bTest" color="7" fill="1" visible="yes" active="no"/>
 <layer number="39" name="tKeepout" color="4" fill="11" visible="no" active="no"/>
 <layer number="40" name="bKeepout" color="1" fill="11" visible="no" active="no"/>
@@
 <layer number="44" name="Drills" color="7" fill="1" visible="no" active="no"/>
 <layer number="45" name="Holes" color="7" fill="1" visible="no" active="no"/>
-<layer number="46" name="Milling" color="3" fill="1" visible="no" active="no"/>
-<layer number="47" name="Measures" color="7" fill="1" visible="no" active="no"/>
-<layer number="48" name="Document" color="7" fill="1" visible="no" active="no"/>
-<layer number="49" name="Reference" color="7" fill="1" visible="no" active="no"/>
-<layer number="50" name="dxf" color="7" fill="1" visible="no" active="no"/>
-<layer number="51" name="tDocu" color="7" fill="1" visible="no" active="no"/>
-<layer number="52" name="bDocu" color="7" fill="1" visible="no" active="no"/>
-<layer number="53" name="tGND_GNDA" color="7" fill="9" visible="no" active="no"/>
-<layer number="54" name="bGND_GNDA" color="1" fill="9" visible="no" active="no"/>
-<layer number="56" name="wert" color="7" fill="1" visible="no" active="no"/>
-<layer number="57" name="tCAD" color="7" fill="1" visible="no" active="no"/>
+<layer number="46" name="Milling" color="3" fill="1" visible="yes" active="no"/>
+<layer number="47" name="Measures" color="7" fill="1" visible="yes" active="no"/>
+<layer number="48" name="Document" color="7" fill="1" visible="yes" active="no"/>
+<layer number="49" name="Reference" color="7" fill="1" visible="yes" active="no"/>
+<layer number="50" name="dxf" color="7" fill="1" visible="yes" active="no"/>
+<layer number="51" name="tDocu" color="7" fill="1" visible="yes" active="no"/>
+<layer number="52" name="bDocu" color="7" fill="1" visible="yes" active="no"/>
+<layer number="53" name="tGND_GNDA" color="7" fill="9" visible="yes" active="no"/>
+<layer number="54" name="bGND_GNDA" color="1" fill="9" visible="yes" active="no"/>
+<layer number="56" name="wert" color="7" fill="1" visible="yes" active="no"/>
+<layer number="57" name="tCAD" color="7" fill="1" visible="yes" active="no"/>
 <layer number="90" name="Modules" color="5" fill="1" visible="yes" active="yes"/>
 <layer number="91" name="Nets" color="2" fill="1" visible="yes" active="yes"/>
@@
 <part name="C14" library="resistor" deviceset="C-EU" device="C0805" value="0.1µF"/>
 <part name="GND36" library="supply1" deviceset="GND" device=""/>
-<part name="CN1" library="SIM800C" deviceset="JST_2PIN" device="-SMT" value="LiPo Battery"/>
+<part name="CN1" library="SIM800C" deviceset="JST_2PIN" device="-THM-RA" value="LiPo Battery"/>
 <part name="U$2" library="ORG1510-MK4 GPS module" deviceset="ORG1510-MK4" device=""/>
 <part name="R1" library="resistor" deviceset="R-EU_" device="R0805" value="220"/>

Commit message: - further progress on top deck board (oled space marked in tplace), joystick added, missing JTAG header and led/switch header
Parts:
- removed C32, C33, C34, C35: 4.7µF, rcl:C-EUC0805
- removed D2: (no value), semicon-smd-ipc:D-SOD-80
- removed GPRS: gprs, switch-omron:10-XX
- removed L4: 33µH, rcl:L-US
- removed R55: 910k, resistor:R-EU_R1206
- removed R56: 160k, resistor:R-EU_R1206
- removed U$6: V_REG_TPS61040SMD, SparkFun-PowerIC:V_REG_TPS61040SMD
- removed X3: FH12-24S-0.5SH, con-hirose:FH12-24S-0.5SH
- added C12: 4.7µF / 25V, rcl:C-EUC0805
- added C30: 0.47µF, resistor:C-EUC0805
- added GPRS_PUSH: BT, switch-omron:10-XX
- added OLED: FH12-30S-0.5SH, con-hirose:FH12-30S-0.5SH
- added R22: 47k, rcl:R-EU_R0805
- added SV2: (no value), con-lstb:MA05-1
- added V_GPS1: PTR1TP14R, testpad:PTR1TP14R
- C36: value 4.7µF -> 1µF
- C37, C40: value 0.1µF -> 1µF
- C38: value 10µF -> 1µF
- C39: value 4.7µF / 25V -> 2.2µF
- IC5: value (none) -> 74HCT1G32
- R54: value 160k -> 1k; device resistor:R-EU_R1206 -> rcl:R-EU_R0805
- R57: value 910k -> 390k
Connections:
- net GPRS renamed CENTER
- removed net BUTTON_GPRS: GPRS.S, GPRS.S1, R16.1, R19.1
- removed net N$41: GPS_GREEN_LED.C, R46.2
- removed net N$43: GPS_RED_LED.C, R45.2
- removed net N$73: D2.A, L4.1, U$6.SW
- removed net N$76: C35.1, R55.1, R56.2, U$6.FB
- removed net OLED_POWER_ON-OFF: R54.2, U$6.EN
- removed net PG2: BL20.16, ML20.16, TL20.16, U1.PG2_(ALE)
- removed net VOLED: C33.2, C34.2, C35.2, C37.2, C38.2, D2.C, R55.2, X3-23.1
- new net CAP1N: C40.1, OLED-5.1
- new net CAP1P: C40.2, OLED-4.1
- new net CAP2N: C36.1, OLED-3.1
- new net CAP2P: C36.2, OLED-2.1
- new net GPRS_BUTTON: GPRS_PUSH.S, GPRS_PUSH.S1, R22.1, R54.1
- new net GPRS_PUSH: BL20.16, C30.2, ML20.16, R22.2, TL20.16
- new net GREEN_LED: GPS_GREEN_LED.C, R46.2, SV2.4
- new net MENU_CENTER_BUTTON_PIN: U1.PC5_(A13), U2.4Y
- new net N$3: SV2.2
- new net OLED_VCC: C39.2, OLED-28.1
- new net RED_LED: GPS_RED_LED.C, R45.2, SV2.5
- net BLUE_LED: now also SV2.3
- net BUTTON_CENTER: now also R16.1, R19.1
- net DOWN: now also BR20.14, MR20.14, TR20.14, U2.6A; no longer BR20.12, MR20.12, TR20.12, U2.2A
- net GND: now also C12.1, C30.1, GPRS_PUSH.P, GPRS_PUSH.P1, OLED-10.1, OLED-11.1, OLED-12.1, OLED-16.1, OLED-17.1, OLED-21.1, OLED-22.1, OLED-23.1, OLED-24.1, OLED-25.1, OLED-29.1, OLED-8.1; no longer C32.1, C33.1, C34.1, C36.1, C40.1, GPRS.P, GPRS.P1, R54.1, R56.1, U$6.GND, X3-1.1, X3-11.1, X3-12.1, X3-2.1, X3-24.1, X3-3.1, X3-6.1, X3-7.1
- net GPRS_LED: now also SV2.1
- net GPS_ON_OFF: now also BL20.12, ML20.12, TL20.12; no longer BL20.11, ML20.11, TL20.11
- net GPS_TX: now also BL20.11, ML20.11, TL20.11; no longer BL20.12, ML20.12, TL20.12
- net IREF: now also OLED-26.1; no longer X3-21.1
- net MENU_DOWN_BUTTON_PIN: now also U1.PC3_(A11), U2.6Y; no longer U1.PC1_(A9), U2.2Y
- net MENU_GPRS_PUSH_BUTTON_PIN: now also U1.PG2_(ALE); no longer U1.PC5_(A13), U2.4Y
- net MENU_RIGHT_BUTTON_PIN: now also U1.PC2_(A10), U2.3Y; no longer U1.PC3_(A11), U2.6Y
- net MENU_UP_BUTTON_PIN: now also U1.PC1_(A9), U2.2Y; no longer U1.PC2_(A10), U2.3Y
- net RIGHT: now also BR20.13, MR20.13, TR20.13, U2.3A; no longer BR20.14, MR20.14, TR20.14, U2.6A
- net SPI_MOSI_PIN: now also OLED-19.1; no longer X3-14.1
- net SPI_OLED_D/C_PIN: now also BR20.2, MR20.2, OLED-15.1, TR20.2, U1.(OC0A/OC1C/PCINT7)_PB7; no longer BR20.3, MR20.3, TR20.3, U1.(TOSC2)_PG3, X3-10.1
- net SPI_OLED_RESET_PIN: now also BR20.3, MR20.3, OLED-14.1, TR20.3, U1.(TOSC2)_PG3; no longer BR20.2, MR20.2, TR20.2, U1.(OC0A/OC1C/PCINT7)_PB7, X3-9.1
- net SPI_SCK_PIN: now also OLED-18.1; no longer X3-13.1
- net SPI_SS_OLED_PIN: now also OLED-13.1; no longer X3-8.1
- net UP: now also BR20.12, MR20.12, TR20.12, U2.2A; no longer BR20.13, MR20.13, TR20.13, U2.3A
- net VCC: now also C37.2, OLED-9.1, R54.2; no longer C32.2, C36.2, C40.2, L4.2, U$6.VIN, X3-5.1
- net VCOMH: now also C12.2, OLED-27.1; no longer C39.2, X3-22.1
- net VGPS: now also V_GPS1.TP
- net V_LIION_REGULATED: now also C38.2, OLED-6.1
Other:
- note removed: "OLED Panel Power Supply"
- moved on the sheet: ANT2, BLUETOOTH, BT, C25, C26, C27, C28, C36, C37, C38, C39, C40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

Commit message: - final steps on 3-deck boards: copper mask, ground vias, 4th board for led/switches (to be mounted on lid)
Parts:
- removed BLUETOOTH, GPRS_PUSH: BT, switch-omron:10-XX
- removed SV2: (no value), con-lstb:MA05-1
- removed U$13: JTAGHEADER, DS1031-14 - IDC socket:JTAGHEADER
- added BLUETOOTH_SWITCH: BT, jumper:JP1E
- added BOARD, LID: 1.27-10-PIN-HEADER, 1.27mm 10pin header:1.27-10-PIN-HEADER
- added GPRS_SWITCH: GPRS, jumper:JP1E
- added JTAG: JTAG-1.27-10-PIN-HEADER, JTAG 1.27mm 10pin header:JTAG-1.27-10-PIN-HEADER
Connections:
- net GPIO6 renamed BT_GPIO6
- net N$39 renamed BT_RST
- removed net GPRS_PUSH: BL20.16, C30.2, ML20.16, R22.2, TL20.16
- removed net N$3: SV2.2
- net BLUE_LED: now also BOARD.3, LID.3; no longer SV2.3
- net BUTTON_BLUETOOTH: now also BLUETOOTH_SWITCH.2, BOARD.9, LID.9; no longer BLUETOOTH.S, BLUETOOTH.S1
- net GND: now also BLUETOOTH_SWITCH.1, BOARD.5, GPRS_SWITCH.1, JTAG.GND1, JTAG.GND2, LID.5; no longer BLUETOOTH.P, BLUETOOTH.P1, GPRS_PUSH.P, GPRS_PUSH.P1, U$13.GND1, U$13.GND2
- net GPRS_BUTTON: now also BOARD.7, GPRS_SWITCH.2, LID.7; no longer GPRS_PUSH.S, GPRS_PUSH.S1
- net GPRS_LED: now also BOARD.10, LID.10; no longer SV2.1
- net GREEN_LED: now also BOARD.1, LID.1; no longer SV2.4
- net JTAG_TCL_PIN: now also JTAG.TCK; no longer U$13.TCK
- net JTAG_TDI_PIN: now also JTAG.TDI; no longer U$13.TDI
- net JTAG_TDO_PIN: now also JTAG.TDO; no longer U$13.TDO
- net JTAG_TMS_PIN: now also JTAG.TMS; no longer U$13.TMS
- net MENU_GPRS_PUSH_BUTTON_PIN: now also BL20.16, C30.2, ML20.16, R22.2, TL20.16
- net RED_LED: now also BOARD.2, LID.2; no longer SV2.5
- net RESET: now also JTAG.RESET; no longer U$13.RESET
- net VCC: now also BOARD.6, JTAG.VCC, LID.6; no longer U$13.VCC
Other:
- moved on the sheet: ANT2, BT, C1, C16, C27, C28, C3, C30, C41, C8, GPS, JP2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

Commit message: - switched to 6x6 SPST-NO switches, corrected a minor ammount of ratlines
Parts:
- removed BLUETOOTH_SWITCH: BT, jumper:JP1E
- removed GPRS_SWITCH: GPRS, jumper:JP1E
- added BLUETOOTH: bt, switch-omron:10-XX
- added GPRS: gprs, switch-omron:10-XX
Connections:
- removed net PD7: U1.(T0)_PD7
- removed net PG0: U1.PG0_(~WR)
- removed net PG1: U1.PG1_(~RD)
- net BUTTON_BLUETOOTH: now also BLUETOOTH.S, BLUETOOTH.S1; no longer BLUETOOTH_SWITCH.2
- net GND: now also BLUETOOTH.P, BLUETOOTH.P1, GPRS.P, GPRS.P1; no longer BLUETOOTH_SWITCH.1, GPRS_SWITCH.1
- net GPRS_BUTTON: now also GPRS.S, GPRS.S1; no longer GPRS_SWITCH.2
Changed lines of the file:
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@@
 <part name="BOARD" library="1.27mm 10pin header" deviceset="1.27-10-PIN-HEADER" device=""/>
 <part name="LID" library="1.27mm 10pin header" deviceset="1.27-10-PIN-HEADER" device=""/>
-<part name="GPRS_SWITCH" library="jumper" deviceset="JP1E" device="" value="GPRS"/>
-<part name="BLUETOOTH_SWITCH" library="jumper" deviceset="JP1E" device="" value="BT"/>
+<part name="BLUETOOTH" library="switch-omron" deviceset="10-XX" device="" value="bt"/>
+<part name="GPRS" library="switch-omron" deviceset="10-XX" device="" value="gprs"/>
 </parts>
 <sheets>
@@
 <instance part="BOARD" gate="G$1" x="567.69" y="811.53"/>
 <instance part="LID" gate="G$1" x="648.97" y="812.8"/>
-<instance part="GPRS_SWITCH" gate="A" x="189.23" y="414.02" rot="R90"/>
-<instance part="BLUETOOTH_SWITCH" gate="A" x="189.23" y="375.92" rot="R90"/>
+<instance part="BLUETOOTH" gate="1" x="190.5" y="378.46" rot="R270"/>
+<instance part="GPRS" gate="1" x="189.23" y="416.56" rot="R270"/>
 </instances>
 <busses>
@@
 </segment>
 <segment>
-<pinref part="GPRS_SWITCH" gate="A" pin="1"/>
-<wire x1="191.77" y1="414.02" x2="195.58" y2="414.02" width="0.1524" layer="91"/>
-<label x="195.58" y="414.02" size="1.778" layer="95" ratio="9"/>
-</segment>
-<segment>
 <pinref part="C30" gate="G$1" pin="1"/>
 <wire x1="214.64" y1="406.39" x2="205.74" y2="406.39" width="0.1524" layer="91"/>
@@
 </segment>
 <segment>
-<pinref part="BLUETOOTH_SWITCH" gate="A" pin="1"/>
-<wire x1="191.77" y1="375.92" x2="194.31" y2="375.92" width="0.1524" layer="91"/>
-<label x="194.31" y="375.92" size="1.778" layer="95" ratio="9"/>
-</segment>
-<segment>
 <pinref part="C8" gate="G$1" pin="1"/>
 <wire x1="207.1" y1="368.24" x2="215.9" y2="368.3" width="0.1524" layer="91"/>
@@
 <wire x1="299.72" y1="-406.4" x2="289.56" y2="-406.4" width="0.1524" layer="91"/>
 </segment>
+<segment>
+<pinref part="GPRS" gate="1" pin="P"/>
+<pinref part="GPRS" gate="1" pin="P1"/>
+<wire x1="184.15" y1="416.56" x2="184.15" y2="414.02" width="0.1524" layer="91"/>
+<wire x1="184.15" y1="416.56" x2="175.26" y2="416.56" width="0.1524" layer="91"/>
+<junction x="184.15" y="416.56"/>
+<label x="175.26" y="416.56" size="1.778" layer="95" ratio="9"/>
+</segment>
+<segment>
+<pinref part="BLUETOOTH" gate="1" pin="P"/>
+<pinref part="BLUETOOTH" gate="1" pin="P1"/>
+<wire x1="185.42" y1="378.46" x2="185.42" y2="375.92" width="0.1524" layer="91"/>
+<wire x1="185.42" y1="378.46" x2="173.99" y2="378.46" width="0.1524" layer="91"/>
+<junction x="185.42" y="378.46"/>
+<label x="173.99" y="378.46" size="1.778" layer="95" ratio="9"/>
+</segment>
 </net>
 <net name="5V0" class="1">
@@
 <junction x="213.36" y="378.46"/>
 <label x="208.07" y="378.12" size="1.778" layer="95" rot="R90"/>
-<pinref part="BLUETOOTH_SWITCH" gate="A" pin="2"/>
-<wire x1="191.77" y1="378.46" x2="213.36" y2="378.46" width="0.1524" layer="91"/>
+<wire x1="195.58" y1="378.46" x2="213.36" y2="378.46" width="0.1524" layer="91"/>
+<pinref part="BLUETOOTH" gate="1" pin="S"/>
+<pinref part="BLUETOOTH" gate="1" pin="S1"/>
+<wire x1="195.58" y1="378.46" x2="195.58" y2="375.92" width="0.1524" layer="91"/>
+<junction x="195.58" y="378.46"/>
 </segment>
 <segment>
@@
 </segment>
 </net>
-<net name="PG0" class="0">
-<segment>
-<pinref part="U1" gate="A" pin="PG0_(~WR)"/>
-<wire x1="154.94" y1="822.96" x2="162.56" y2="822.96" width="0.1524" layer="91"/>
-<label x="162.56" y="822.96" size="1.778" layer="95"/>
-</segment>
-</net>
 <net name="V_SUPERCAP_SENSE_PIN" class="0">
 <segment>
@@
 </segment>
 </net>
-<net name="PG1" class="0">
-<segment>
-<pinref part="U1" gate="A" pin="PG1_(~RD)"/>
-<wire x1="154.94" y1="820.42" x2="162.56" y2="820.42" width="0.1524" layer="91"/>
-<label x="162.56" y="820.42" size="1.778" layer="95"/>
-</segment>
-</net>
-<net name="PD7" class="0">
-<segment>
-<pinref part="U1" gate="A" pin="(T0)_PD7"/>
-<wire x1="154.94" y1="741.68" x2="162.56" y2="741.68" width="0.1524" layer="91"/>
-<label x="162.56" y="741.68" size="1.778" layer="95"/>
-</segment>
-</net>
 <net name="LTC4425_EN" class="2">
 <segment>
@@
 <junction x="213.36" y="416.56"/>
 <label x="207.01" y="416.56" size="1.778" layer="95" ratio="9" rot="R90"/>
-<pinref part="GPRS_SWITCH" gate="A" pin="2"/>
-<wire x1="191.77" y1="416.56" x2="213.36" y2="416.56" width="0.1524" layer="91"/>
+<wire x1="199.39" y1="416.56" x2="213.36" y2="416.56" width="0.1524" layer="91"/>
+<pinref part="GPRS" gate="1" pin="S"/>
+<pinref part="GPRS" gate="1" pin="S1"/>
+<wire x1="194.31" y1="416.56" x2="194.31" y2="414.02" width="0.1524" layer="91"/>
+<wire x1="213.36" y1="416.56" x2="194.31" y2="416.56" width="0.1524" layer="91"/>
+<junction x="194.31" y="416.56"/>
 </segment>
 <segment>
