File: misko_3_board.sch (EAGLE design)
At the start: 171 parts, among them IC1 MC1525TT, IC2 FT230XS, IC3 LTC4425, IC4 FM25W256-SOIC, IC5 74HCT1G32, M10 mid, Q1 BSS84, T10 top, U1 ATMEGA1281-16AU, U2 SN74HCT14DR, U5 TMP36GRTZ, U6 TPS3808G33DBVT, U7 MCP73871-2AAI/ML, U8 SIM800

Commit message: - finished board & schematic, corrected BOM
Parts:
- removed 8MHZ: 8MHz, special:OSCILATOR
- removed B10: bottom, con-lstb:MA10-1
- removed BL20: bottom left, con-lsta:FE20-1
- removed BOARD, LID: 1.27-10-PIN-HEADER, 1.27mm 10pin header:1.27-10-PIN-HEADER
- removed BR20: bottom right, con-lsta:FE20-1
- removed M10: mid, con-lstb:MA10-1
- removed T10: top, con-lstb:MA10-1
- removed TL20: top left, con-lsta:FE20-1
- removed TR20: top right, con-lsta:FE20-1
- removed U$10: DJNR3015-1R5, DJNR3015-1R5 Inductor:DJNR3015-1R5
- removed U$9: TPS63031, TI TPS63031:TPS63001DRCR
- removed U1: ATMEGA1281-16AU, Atmel_By_element14_Batch_1-00:ATMEGA1281-16AU
- removed U5: TMP36GRTZ, TMP36GRTZ:TMP36GRTZ-REEL7
- removed U7: MCP73871-2AAI/ML, Microchip-MCP73871-2AAI_ML:MCP73871-2AAI/ML
- removed VCC5: PTR1TP14R, testpad:PTR1TP14R
- added CONN1: bottom, con-lstb:MA10-1
- added CONN12: board, 1.27mm 10pin header:1.27-10-PIN-HEADER
- added CONN13: lid, 1.27mm 10pin header:1.27-10-PIN-HEADER
- added CONN2: bottom left, con-lsta:FE20-1
- added CONN3: bottom right, con-lsta:FE20-1
- added CONN4: mid, con-lstb:MA10-1
- added CONN7: top, con-lstb:MA10-1
- added CONN8: top left, con-lsta:FE20-1
- added CONN9: top right, con-lsta:FE20-1
- added IC12: LTC4425, LTC4425 Supercap Charger:LTC4425
- added IC15: 74HCT1G32, 74HCT1G32GW:74HCT1G32GW-DC
- added IC16: FM25W256-SOIC, FM25W256 FERAM:FM25W256-SOIC
- added IC7: FT230XS, ftdichip:FT230XS
- added L1: 33µH, rcl:L-US
- added T1: BSS84, transistor-small-signal:BSS84
- added TP1: GND, testpad:TPPAD1-17Y
- CONN10: value JTAG-1.27-10-PIN-HEADER -> JTAG
- IC1: value MC1525TT -> ATMEGA1281-16AU; device microchip:MC1525TT -> Atmel_By_element14_Batch_1-00:ATMEGA1281-16AU
- IC2: value FT230XS -> MC1525TT; device ftdichip:FT230XS -> microchip:MC1525TT
- IC3: value LTC4425 -> TMP36GRTZ; device LTC4425 Supercap Charger:LTC4425 -> TMP36GRTZ:TMP36GRTZ-REEL7
- IC4: value FM25W256-SOIC -> TPS63031; device FM25W256 FERAM:FM25W256-SOIC -> TI TPS63031:TPS63001DRCR
- IC5: value 74HCT1G32 -> MCP73871-2AAI/ML; device 74HCT1G32GW:74HCT1G32GW-DC -> Microchip-MCP73871-2AAI_ML:MCP73871-2AAI/ML
- L2: value 33µH -> DJNR3015-1R5; device rcl:L-US -> DJNR3015-1R5 Inductor:DJNR3015-1R5
- Q1: value BSS84 -> 8MHz; device transistor-small-signal:BSS84 -> special:OSCILATOR
- R1: value 10k -> NTC 10k
- R14, R42, R43, R44, R52, R53, R55, R57: device rcl:R-EU_M0805 -> rcl:R-EU_R0805
- R49: value 4.7k -> 4k7
- TP10, TP11: value PTR1TP14R -> VGPS
- TP2: value PTR1B1,27 -> VCC; device testpad:PTR1B1,27 -> testpad:PTR1TP14R
- TP3: value PTR1TP14R -> Analogue Switch CRTL Pin
- TP4: value PTR1TP14R -> VCC
- TP5: value PTR1B1,27 -> GPS Power CTRL Pin
- TP6: value GND -> GPS Power CTRL Pin; device testpad:TPPAD1-17Y -> testpad:PTR1B1,27
- TP7: value PTR1B1,27 -> SIM800 Power CTRL Pin
- TP8: value PTR1TP14R -> VLiIon Regulated
- TP9: value PTR1TP14R -> Bluetooth Wakeup Pin
- renumbered ANT to CONN15, BLUETOOTH to S5, BT to TP9, BT-SW to IC8, BT_LED to LED5, GND to IC10, GPRS to S4, GPRS_LED to LED6, GPS-SW to IC9, GPS_GREEN_LED to LED1, GPS_POWER_CTL_PIN to TP5, GPS_RED_LED to LED2, I2C to CONN11, JTAG to CONN10, LIION to CONN16, ML20 to CONN5, MR20 to CONN6, NTC to R1, OLED to IC18, POWER to S2, RESET to S1, SIM800 to TP7, SJ1 to JP2, SJ2 to JP3, SUPERCAP to C43, U$11 to CONN14, U$12 to S3, U$13 to Q2, U$3 to IC13, U$4 to IC14, U$5 to IC17, U$6 to IC19, U$7 to IC20, U2 to IC6, U6 to IC11, U8 to IC21, USB_RX_LED to LED3, USB_TX_LED to LED4, VCC to TP4, VCC1 to TP3, V_GPS to TP10, V_GPS1 to TP11, V_LIION to TP8
Connections:
- net 5V0: now also CONN3.20, CONN9.20, IC5.*TE, IC5.CE, IC5.IN, IC5.IN_2, IC5.PROG2, IC5.SEL, IC7.VCC; no longer BR20.20, IC2.VCC, TR20.20, U7.*TE, U7.CE, U7.IN, U7.IN_2, U7.PROG2, U7.SEL
- net ADXL345SDA: now also IC15.Y; no longer IC5.Y
- net ADXL345_INT1_INTERRUPT_PIN: now also IC1.(ICP3/CLKO/INT7)_PE7; no longer U1.(ICP3/CLKO/INT7)_PE7
- net ANALOG_SW_CTRL_PIN: now also CONN3.1, CONN9.1, IC1.(OC1B/PCINT6)_PB6; no longer BR20.1, TR20.1, U1.(OC1B/PCINT6)_PB6
- net AREF: now also IC1.AREF, IC2.VO; no longer IC1.VO, U1.AREF
- net AVCC: now also IC1.AVCC, IC2.VIN, L1.2; no longer IC1.VIN, L2.2, U1.AVCC
- net BAT_A_PIN: now also IC1.PF3_(ADC3); no longer U1.PF3_(ADC3)
- net BLUETOOTH: now also CONN3.15, CONN9.15; no longer BR20.15, TR20.15
- net BLUETOOTH_WAKEUP_PIN: now also CONN2.13, CONN8.13, IC1.PA3_(AD3), T1.G; no longer BL20.13, Q1.G, TL20.13, U1.PA3_(AD3)
- net BLUE_LED: now also CONN12.3, CONN13.3, CONN2.15, CONN8.15, T1.D; no longer BL20.15, BOARD.3, LID.3, Q1.D, TL20.15
- net BUTTON_BLUETOOTH: now also CONN12.9, CONN13.9; no longer BOARD.9, LID.9
- net BUZZER: now also CONN2.14, CONN8.14, IC1.PA7_(AD7); no longer BL20.14, TL20.14, U1.PA7_(AD7)
- net CBUS1: now also IC7.CBUS1; no longer IC2.CBUS1
- net CBUS2: now also IC7.CBUS2; no longer IC2.CBUS2
- net CENTER: now also CONN3.16, CONN9.16; no longer BR20.16, TR20.16
- net DOWN: now also CONN3.14, CONN9.14; no longer BR20.14, TR20.14
- net EN: now also CONN2.20, CONN8.20, IC4.EN; no longer BL20.20, TL20.20, U$9.EN
- net GND: now also CONN1.9, CONN12.5, CONN13.5, CONN2.5, CONN3.5, CONN4.9, CONN7.9, CONN8.5, CONN9.5, IC1.GND_2, IC1.GND_3, IC12.GND, IC15.GND, IC16.GND, IC4.PGND, IC4.POWERPAD, IC5.EP, IC5.VSS, IC5.VSS_2, IC7.GND, IC7.GND@1, TP1.TP; no longer B10.9, BL20.5, BOARD.5, BR20.5, IC2.GND@1, IC5.GND, LID.5, M10.9, T10.9, TL20.5, TP6.TP, TR20.5, U$9.GND, U$9.PGND, U$9.POWERPAD, U1.GND, U1.GND_2, U1.GND_3, U5.GND, U7.EP, U7.VSS, U7.VSS_2
- net GPRS_BUTTON: now also CONN12.7, CONN13.7; no longer BOARD.7, LID.7
- net GPRS_NETLIGHT: now also CONN12.10, CONN13.10, CONN3.18, CONN9.18; no longer BOARD.10, BR20.18, LID.10, TR20.18
- net GPS_GREEN_LED_PIN: now also CONN2.17, CONN8.17, IC1.PC7_(A15); no longer BL20.17, TL20.17, U1.PC7_(A15)
- net GPS_POWER_CTL_PIN: now also CONN2.12, CONN8.12, IC1.PA2_(AD2), TP6.TP; no longer BL20.12, TL20.12, TP2.TP, U1.PA2_(AD2)
- net GPS_RED_LED_PIN: now also CONN2.18, CONN8.18, IC1.PC6_(A14); no longer BL20.18, TL20.18, U1.PC6_(A14)
- net GPS_SW_SERIAL_RX: now also CONN1.2, CONN4.2, CONN7.2, IC1.(OC2A/_PCINT4)_PB4; no longer B10.2, M10.2, T10.2, U1.(OC2A/_PCINT4)_PB4
- net GPS_SW_SERIAL_TX: now also CONN1.1, CONN4.1, CONN7.1, IC1.(OC1A/PCINT5)_PB5; no longer B10.1, M10.1, T10.1, U1.(OC1A/PCINT5)_PB5
- net GPS_TX: now also CONN2.11, CONN8.11; no longer BL20.11, TL20.11
- net GPS_WAKEUP_PIN: now also CONN2.10, CONN8.10, IC1.PA1_(AD1); no longer BL20.10, TL20.10, U1.PA1_(AD1)
- net GREEN_LED: now also CONN12.1, CONN13.1; no longer BOARD.1, LID.1
- net I2C_SCL_PIN: now also IC1.(SCL/INT0)_PD0; no longer U1.(SCL/INT0)_PD0
- net I2C_SDA_PIN: now also IC1.(SDA/INT1)_PD1; no longer U1.(SDA/INT1)_PD1
- net JTAG_TCL_PIN: now also CONN2.6, CONN8.6, IC1.PF4_(ADC4/TCK); no longer BL20.6, TL20.6, U1.PF4_(ADC4/TCK)
- net JTAG_TDI_PIN: now also CONN2.9, CONN8.9, IC1.PF7_(ADC7/TDI); no longer BL20.9, TL20.9, U1.PF7_(ADC7/TDI)
- net JTAG_TDO_PIN: now also CONN2.8, CONN8.8, IC1.PF6_(ADC6/TDO); no longer BL20.8, TL20.8, U1.PF6_(ADC6/TDO)
- net JTAG_TMS_PIN: now also CONN2.7, CONN8.7, IC1.PF5_(ADC5/TMS); no longer BL20.7, TL20.7, U1.PF5_(ADC5/TMS)
- net L1: now also IC4.L1, L2.L1; no longer U$10.L1, U$9.L1
- net L2: now also IC4.L2, L2.L2; no longer U$10.L2, U$9.L2
- net LEFT: now also CONN3.11, CONN9.11; no longer BR20.11, TR20.11
- net LTC4425_EN: now also IC12.EN; no longer IC3.EN
- net LTC4425_PROG: now also IC12.PROG; no longer IC3.PROG
- net MCP73871_CHARGE_STATUS_1_PIN: now also IC1.PA4_(AD4), IC5.STAT1/*LBO; no longer U1.PA4_(AD4), U7.STAT1/*LBO
- net MCP73871_CHARGE_STATUS_2_PIN: now also IC1.PA5_(AD5), IC5.STAT2; no longer U1.PA5_(AD5), U7.STAT2
- net MCP73871_POWER_GOOD_PIN: now also IC1.PA6_(AD6), IC5.*PG; no longer U1.PA6_(AD6), U7.*PG
- net MENU_BLUETOOTH_POWER_TOGGLE_PIN: now also IC1.PC4_(A12); no longer U1.PC4_(A12)
- net MENU_CENTER_BUTTON_PIN: now also IC1.PC5_(A13); no longer U1.PC5_(A13)
- net MENU_DOWN_BUTTON_PIN: now also IC1.PC3_(A11); no longer U1.PC3_(A11)
- net MENU_GPRS_PUSH_BUTTON_PIN: now also CONN2.16, CONN8.16, IC1.PG2_(ALE); no longer BL20.16, TL20.16, U1.PG2_(ALE)
- net MENU_LEFT_BUTTON_PIN: now also IC1.PC0_(A8); no longer U1.PC0_(A8)
- net MENU_RIGHT_BUTTON_PIN: now also IC1.PC2_(A10); no longer U1.PC2_(A10)
- net MENU_UP_BUTTON_PIN: now also IC1.PC1_(A9); no longer U1.PC1_(A9)
- net N$10: now also IC7.!RESET, IC7.3V3OUT, IC7.VCCIO; no longer IC2.!RESET, IC2.3V3OUT, IC2.VCCIO
- net PDI_UART0_CTS_PIN: now also CONN2.3, CONN8.3, IC1.(OC0B)_PG5, IC7.!CTS; no longer BL20.3, IC2.!CTS, TL20.3, U1.(OC0B)_PG5
- net PDI_UART0_RX_PIN: now also IC1.(RXD0/PCINT8/PDI)_PE0; no longer U1.(RXD0/PCINT8/PDI)_PE0
- net PDI_UART0_TX_PIN: now also IC1.(TXD0/PDO)_PE1; no longer U1.(TXD0/PDO)_PE1
- net PFI: now also IC12.PFI; no longer IC3.PFI
- net PFI_RET: now also IC12.PFI_RET; no longer IC3.PFI_RET
- net PROG1: now also IC5.PROG1; no longer U7.PROG1
- net PROG3: now also IC5.PROG3; no longer U7.PROG3
- net RED_LED: now also CONN12.2, CONN13.2; no longer BOARD.2, LID.2
- net RESET: now also CONN3.17, CONN9.17, IC1.~RESET; no longer BR20.17, TR20.17, U1.~RESET
- net RIGHT: now also CONN3.13, CONN9.13; no longer BR20.13, TR20.13
- net RTC_INT_INTERRUPT_PIN: now also CONN1.6, CONN4.6, CONN7.6, IC1.(T3/INT6)_PE6; no longer B10.6, M10.6, T10.6, U1.(T3/INT6)_PE6
- net RXD: now also CONN2.1, CONN8.1, IC7.RXD; no longer BL20.1, IC2.RXD, TL20.1
- net SD_CARD_DETECT_PIN: now also IC1.(OC3A/AIN1)_PE3; no longer U1.(OC3A/AIN1)_PE3
- net SIM800C_CTS_PIN: now also CONN3.8, CONN9.8, IC1.(ICP1)_PD4; no longer BR20.8, TR20.8, U1.(ICP1)_PD4
- net SIM800C_POWER_PIN: now also CONN3.10, CONN9.10, IC1.(T1)_PD6; no longer BR20.10, TR20.10, U1.(T1)_PD6
- net SIM800C_RX_PIN: now also CONN3.6, CONN9.6, IC1.(RXD1/INT2)_PD2; no longer BR20.6, TR20.6, U1.(RXD1/INT2)_PD2
- net SIM800C_STATUS_PIN: now also CONN3.9, CONN9.9, IC1.(XCK1)_PD5; no longer BR20.9, TR20.9, U1.(XCK1)_PD5
- net SIM800C_TX_PIN: now also CONN3.7, CONN9.7, IC1.(TXD1/INT3)_PD3; no longer BR20.7, TR20.7, U1.(TXD1/INT3)_PD3
- net SPI_FRAM_SS_PIN: now also IC1.(OC3B/INT4)_PE4, IC16.!CS!; no longer IC4.!CS!, U1.(OC3B/INT4)_PE4
- net SPI_MISO_PIN: now also CONN1.3, CONN4.3, CONN7.3, IC1.(MISO/PCINT3)_PB3, IC16.SO; no longer B10.3, IC4.SO, M10.3, T10.3, U1.(MISO/PCINT3)_PB3
- net SPI_MOSI_PIN: now also CONN1.4, CONN4.4, CONN7.4, IC1.(MOSI/PCINT2)_PB2, IC15.B, IC16.SI; no longer B10.4, IC4.SI, IC5.B, M10.4, T10.4, U1.(MOSI/PCINT2)_PB2
- net SPI_OLED_D/C_PIN: now also CONN3.2, CONN9.2, IC1.(OC0A/OC1C/PCINT7)_PB7; no longer BR20.2, TR20.2, U1.(OC0A/OC1C/PCINT7)_PB7
- net SPI_OLED_RESET_PIN: now also CONN3.3, CONN9.3, IC1.(TOSC2)_PG3; no longer BR20.3, TR20.3, U1.(TOSC2)_PG3
- net SPI_SCK_PIN: now also CONN1.5, CONN4.5, CONN7.5, IC1.(SCK/PCINT1)_PB1, IC16.SCK; no longer B10.5, IC4.SCK, M10.5, T10.5, U1.(SCK/PCINT1)_PB1
- net SPI_SS_ADXL345_PIN: now also IC1.(OC3C/INT5)_PE5, IC15.A; no longer IC5.A, U1.(OC3C/INT5)_PE5
- net SPI_SS_OLED_PIN: now also CONN3.4, CONN9.4, IC1.(TOSC1)_PG4; no longer BR20.4, TR20.4, U1.(TOSC1)_PG4
- net SPI_SS_RTC_PIN: now also CONN1.7, CONN4.7, CONN7.7, IC1.(XCK0/AIN0)_PE2; no longer B10.7, M10.7, T10.7, U1.(XCK0/AIN0)_PE2
- net SPI_SS_SD_CARD_PIN: now also IC1.(~SS/PCINT0)_PB0; no longer U1.(~SS/PCINT0)_PB0
- net THERM: now also IC5.THERM; no longer U7.THERM
- net TMP36_SHUTDOWN_PIN: now also IC1.PA0_(AD0), IC3.~SHDN; no longer U1.PA0_(AD0), U5.~SHDN
- net TMP36_VSENSE_PIN: now also IC1.PF0_(ADC0), IC3.VOUT; no longer U1.PF0_(ADC0), U5.VOUT
- net TXD: now also CONN2.2, CONN8.2, IC7.TXD; no longer BL20.2, IC2.TXD, TL20.2
- net UP: now also CONN3.12, CONN9.12; no longer BR20.12, TR20.12
- net USBDM: now also IC7.USBDM; no longer IC2.USBDM
- net USBDP: now also IC7.USBDP; no longer IC2.USBDP
- net VCC: now also CONN12.6, CONN13.6, CONN2.4, CONN3.19, CONN8.4, CONN9.19, IC1.VCC, IC1.VCC_2, IC12.FB, IC12.SEL, IC12.VCC1, IC12.VCC2, IC15.VCC, IC16.!HOLD!, IC16.!WP!, IC16.VCC, IC3.+VS, IC4.FB, IC4.VOUT, L1.1, T1.S, TP2.TP; no longer BL20.4, BOARD.6, BR20.19, IC3.FB, IC3.SEL, IC3.VCC1, IC3.VCC2, IC4.!HOLD!, IC4.!WP!, IC4.VCC, IC5.VCC, L2.1, LID.6, Q1.S, TL20.4, TR20.19, U$9.FB, U$9.VOUT, U1.VCC, U1.VCC_2, U5.+VS, VCC5.TP
- net VCC_SENSE_PIN: now also IC1.PF1_(ADC1); no longer U1.PF1_(ADC1)
- net VGPS: now also CONN1.8, CONN4.8, CONN7.8, IC12.VOUT1, IC12.VOUT2; no longer B10.8, IC3.VOUT1, IC3.VOUT2, M10.8, T10.8
- net VMID: now also IC12.VMID; no longer IC3.VMID
- net VPCC: now also IC5.VPCC; no longer U7.VPCC
- net V_LIION+: now also IC5.VBAT, IC5.VBAT_2, IC5.VBAT_SENSE; no longer U7.VBAT, U7.VBAT_2, U7.VBAT_SENSE
- net V_LIION_REGULATED: now also CONN2.19, CONN8.19, IC4.PS/SYNC, IC4.VIN, IC4.VINA, IC5.OUT, IC5.OUT_2; no longer BL20.19, TL20.19, U$9.PS/SYNC, U$9.VIN, U$9.VINA, U7.OUT, U7.OUT_2
- net V_SUPERCAP_SENSE_PIN: now also IC1.PF2_(ADC2); no longer U1.PF2_(ADC2)
- net XTAL1: now also IC1.XTAL1, Q1.P$1; no longer 8MHZ.P$1, U1.XTAL1
- net XTAL2: now also IC1.XTAL2, Q1.P$2; no longer 8MHZ.P$2, U1.XTAL2
Other:
- note added: "Buzzer"
- moved on the sheet: R52, TP2, U$1

Commit message: - alpha version of PCB along with modified firmware
Connections:
- net BUZZER renamed BUZZER_PIN
- net V_SUPERCAP_SENSE_PIN renamed VGPS_SENSE_PIN
Changed lines of the file:
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@@
 <grid distance="0.1" unitdist="inch" unit="inch" style="lines" multiple="1" display="no" altdistance="0.01" altunitdist="inch" altunit="inch"/>
 <layers>
-<layer number="1" name="Top" color="4" fill="1" visible="yes" active="no"/>
-<layer number="2" name="Route2" color="1" fill="3" visible="yes" active="no"/>
-<layer number="3" name="Route3" color="4" fill="3" visible="yes" active="no"/>
-<layer number="4" name="Route4" color="1" fill="4" visible="yes" active="no"/>
-<layer number="5" name="Route5" color="4" fill="4" visible="yes" active="no"/>
-<layer number="6" name="Route6" color="1" fill="8" visible="yes" active="no"/>
-<layer number="7" name="Route7" color="4" fill="8" visible="yes" active="no"/>
-<layer number="8" name="Route8" color="1" fill="2" visible="yes" active="no"/>
-<layer number="9" name="Route9" color="4" fill="2" visible="yes" active="no"/>
-<layer number="10" name="Route10" color="1" fill="7" visible="yes" active="no"/>
-<layer number="11" name="Route11" color="4" fill="7" visible="yes" active="no"/>
-<layer number="12" name="Route12" color="1" fill="5" visible="yes" active="no"/>
-<layer number="13" name="Route13" color="4" fill="5" visible="yes" active="no"/>
-<layer number="14" name="Route14" color="1" fill="6" visible="yes" active="no"/>
-<layer number="15" name="Route15" color="4" fill="6" visible="yes" active="no"/>
-<layer number="16" name="Bottom" color="1" fill="1" visible="yes" active="no"/>
-<layer number="17" name="Pads" color="2" fill="1" visible="yes" active="no"/>
-<layer number="18" name="Vias" color="2" fill="1" visible="yes" active="no"/>
-<layer number="19" name="Unrouted" color="6" fill="1" visible="yes" active="no"/>
-<layer number="20" name="Dimension" color="15" fill="1" visible="yes" active="no"/>
-<layer number="21" name="tPlace" color="7" fill="1" visible="yes" active="no"/>
-<layer number="22" name="bPlace" color="7" fill="1" visible="yes" active="no"/>
-<layer number="23" name="tOrigins" color="15" fill="1" visible="yes" active="no"/>
-<layer number="24" name="bOrigins" color="15" fill="1" visible="yes" active="no"/>
-<layer number="25" name="tNames" color="7" fill="1" visible="yes" active="no"/>
-<layer number="26" name="bNames" color="7" fill="1" visible="yes" active="no"/>
-<layer number="27" name="tValues" color="7" fill="1" visible="yes" active="no"/>
-<layer number="28" name="bValues" color="7" fill="1" visible="yes" active="no"/>
+<layer number="1" name="Top" color="4" fill="1" visible="no" active="no"/>
+<layer number="2" name="Route2" color="1" fill="3" visible="no" active="no"/>
+<layer number="3" name="Route3" color="4" fill="3" visible="no" active="no"/>
+<layer number="4" name="Route4" color="1" fill="4" visible="no" active="no"/>
+<layer number="5" name="Route5" color="4" fill="4" visible="no" active="no"/>
+<layer number="6" name="Route6" color="1" fill="8" visible="no" active="no"/>
+<layer number="7" name="Route7" color="4" fill="8" visible="no" active="no"/>
+<layer number="8" name="Route8" color="1" fill="2" visible="no" active="no"/>
+<layer number="9" name="Route9" color="4" fill="2" visible="no" active="no"/>
+<layer number="10" name="Route10" color="1" fill="7" visible="no" active="no"/>
+<layer number="11" name="Route11" color="4" fill="7" visible="no" active="no"/>
+<layer number="12" name="Route12" color="1" fill="5" visible="no" active="no"/>
+<layer number="13" name="Route13" color="4" fill="5" visible="no" active="no"/>
+<layer number="14" name="Route14" color="1" fill="6" visible="no" active="no"/>
+<layer number="15" name="Route15" color="4" fill="6" visible="no" active="no"/>
+<layer number="16" name="Bottom" color="1" fill="1" visible="no" active="no"/>
+<layer number="17" name="Pads" color="2" fill="1" visible="no" active="no"/>
+<layer number="18" name="Vias" color="2" fill="1" visible="no" active="no"/>
+<layer number="19" name="Unrouted" color="6" fill="1" visible="no" active="no"/>
+<layer number="20" name="Dimension" color="15" fill="1" visible="no" active="no"/>
+<layer number="21" name="tPlace" color="7" fill="1" visible="no" active="no"/>
+<layer number="22" name="bPlace" color="7" fill="1" visible="no" active="no"/>
+<layer number="23" name="tOrigins" color="15" fill="1" visible="no" active="no"/>
+<layer number="24" name="bOrigins" color="15" fill="1" visible="no" active="no"/>
+<layer number="25" name="tNames" color="7" fill="1" visible="no" active="no"/>
+<layer number="26" name="bNames" color="7" fill="1" visible="no" active="no"/>
+<layer number="27" name="tValues" color="7" fill="1" visible="no" active="no"/>
+<layer number="28" name="bValues" color="7" fill="1" visible="no" active="no"/>
 <layer number="29" name="tStop" color="7" fill="3" visible="no" active="no"/>
 <layer number="30" name="bStop" color="7" fill="6" visible="no" active="no"/>
@@
 <layer number="35" name="tGlue" color="7" fill="4" visible="no" active="no"/>
 <layer number="36" name="bGlue" color="7" fill="5" visible="no" active="no"/>
-<layer number="37" name="tTest" color="7" fill="1" visible="yes" active="no"/>
-<layer number="38" name="bTest" color="7" fill="1" visible="yes" active="no"/>
+<layer number="37" name="tTest" color="7" fill="1" visible="no" active="no"/>
+<layer number="38" name="bTest" color="7" fill="1" visible="no" active="no"/>
 <layer number="39" name="tKeepout" color="4" fill="11" visible="no" active="no"/>
 <layer number="40" name="bKeepout" color="1" fill="11" visible="no" active="no"/>
@@
 <layer number="44" name="Drills" color="7" fill="1" visible="no" active="no"/>
 <layer number="45" name="Holes" color="7" fill="1" visible="no" active="no"/>
-<layer number="46" name="Milling" color="3" fill="1" visible="yes" active="no"/>
-<layer number="47" name="Measures" color="7" fill="1" visible="yes" active="no"/>
-<layer number="48" name="Document" color="7" fill="1" visible="yes" active="no"/>
-<layer number="49" name="Reference" color="7" fill="1" visible="yes" active="no"/>
-<layer number="50" name="dxf" color="7" fill="1" visible="yes" active="no"/>
-<layer number="51" name="tDocu" color="7" fill="1" visible="yes" active="no"/>
-<layer number="52" name="bDocu" color="7" fill="1" visible="yes" active="no"/>
-<layer number="53" name="tGND_GNDA" color="7" fill="9" visible="yes" active="no"/>
-<layer number="54" name="bGND_GNDA" color="1" fill="9" visible="yes" active="no"/>
-<layer number="56" name="wert" color="7" fill="1" visible="yes" active="no"/>
-<layer number="57" name="tCAD" color="7" fill="1" visible="yes" active="no"/>
-<layer number="59" name="tCarbon" color="7" fill="1" visible="yes" active="no"/>
-<layer number="60" name="bCarbon" color="7" fill="1" visible="yes" active="no"/>
+<layer number="46" name="Milling" color="3" fill="1" visible="no" active="no"/>
+<layer number="47" name="Measures" color="7" fill="1" visible="no" active="no"/>
+<layer number="48" name="Document" color="7" fill="1" visible="no" active="no"/>
+<layer number="49" name="Reference" color="7" fill="1" visible="no" active="no"/>
+<layer number="50" name="dxf" color="7" fill="1" visible="no" active="no"/>
+<layer number="51" name="tDocu" color="7" fill="1" visible="no" active="no"/>
+<layer number="52" name="bDocu" color="7" fill="1" visible="no" active="no"/>
+<layer number="53" name="tGND_GNDA" color="7" fill="9" visible="no" active="no"/>
+<layer number="54" name="bGND_GNDA" color="1" fill="9" visible="no" active="no"/>
+<layer number="56" name="wert" color="7" fill="1" visible="no" active="no"/>
+<layer number="57" name="tCAD" color="7" fill="1" visible="no" active="no"/>
+<layer number="59" name="tCarbon" color="7" fill="1" visible="no" active="no"/>
+<layer number="60" name="bCarbon" color="7" fill="1" visible="no" active="no"/>
 <layer number="90" name="Modules" color="5" fill="1" visible="yes" active="yes"/>
 <layer number="91" name="Nets" color="2" fill="1" visible="yes" active="yes"/>
@@
 </segment>
 </net>
-<net name="V_SUPERCAP_SENSE_PIN" class="2">
+<net name="VGPS_SENSE_PIN" class="2">
 <segment>
 <pinref part="R48" gate="G$1" pin="2"/>
@@
 </segment>
 </net>
-<net name="BUZZER" class="3">
+<net name="BUZZER_PIN" class="3">
 <segment>
 <pinref part="CONN2" gate="G$1" pin="14"/>

Commit message: - panelized, added fiducial marks
Parts:
- added U$2, U$3: FIDUCIAL, adafruit:FIDUCIAL
Changed lines of the file:
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@@
 <part name="C35" library="rcl" deviceset="C-EU" device="C0805" value="1nF"/>
 <part name="R56" library="resistor" deviceset="R-EU_" device="R0805" value="1M"/>
+<part name="U$2" library="adafruit" deviceset="FIDUCIAL" device=""/>
+<part name="U$3" library="adafruit" deviceset="FIDUCIAL" device=""/>
 </parts>
 <sheets>
@@
 <instance part="C35" gate="G$1" x="154.94" y="50.8"/>
 <instance part="R56" gate="G$1" x="213.36" y="68.58" rot="R90"/>
+<instance part="U$2" gate="G$1" x="396.24" y="525.78"/>
+<instance part="U$3" gate="G$1" x="421.64" y="525.78"/>
 </instances>
 <busses>

Commit message: - implemented capacitor bank for support of solar panels (see adafruits solar charger)
Parts:
- added C44, C45, C46, C47, C49: 1000µF, rcl:CPOL-EUE22-10AXIAL
- added D2: (no value), eagle-ltspice:SCHOTTKY-DIODEF126Z12
- R48, R58: value 46k -> 150k
- renumbered U$2 to FI1, U$3 to FI2
Connections:
- new net N$6: C44.+, C45.+, C46.+, C47.+, C49.+, D2.A
- net 5V0: now also D2.C
- net GND: now also C44.-, C45.-, C46.-, C47.-, C49.-
Changed lines of the file:
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@@
 <part name="CONN7" library="con-lstb" deviceset="MA10-1" device="" value="top"/>
 <part name="C43" library="EECS5R5H155 Supercap" deviceset="EECS5R5H155" device=""/>
-<part name="R48" library="resistor" deviceset="R-EU_" device="R0805" value="46k"/>
-<part name="R58" library="resistor" deviceset="R-EU_" device="R0805" value="46k"/>
+<part name="R48" library="resistor" deviceset="R-EU_" device="R0805" value="150k"/>
+<part name="R58" library="resistor" deviceset="R-EU_" device="R0805" value="150k"/>
 <part name="CONN5" library="con-lsta" deviceset="FE20-1" device="" value="mid left"/>
 <part name="CONN6" library="con-lsta" deviceset="FE20-1" device="" value="mid right"/>
@@
 <part name="C35" library="rcl" deviceset="C-EU" device="C0805" value="1nF"/>
 <part name="R56" library="resistor" deviceset="R-EU_" device="R0805" value="1M"/>
-<part name="U$2" library="adafruit" deviceset="FIDUCIAL" device=""/>
-<part name="U$3" library="adafruit" deviceset="FIDUCIAL" device=""/>
+<part name="FI1" library="adafruit" deviceset="FIDUCIAL" device=""/>
+<part name="FI2" library="adafruit" deviceset="FIDUCIAL" device=""/>
+<part name="C49" library="rcl" deviceset="CPOL-EU" device="E22-10AXIAL" value="1000µF"/>
+<part name="C44" library="rcl" deviceset="CPOL-EU" device="E22-10AXIAL" value="1000µF"/>
+<part name="C45" library="rcl" deviceset="CPOL-EU" device="E22-10AXIAL" value="1000µF"/>
+<part name="C46" library="rcl" deviceset="CPOL-EU" device="E22-10AXIAL" value="1000µF"/>
+<part name="C47" library="rcl" deviceset="CPOL-EU" device="E22-10AXIAL" value="1000µF"/>
+<part name="D2" library="eagle-ltspice" deviceset="SCHOTTKY-DIODE" device="F126Z12"/>
 </parts>
 <sheets>
@@
 <instance part="C35" gate="G$1" x="154.94" y="50.8"/>
 <instance part="R56" gate="G$1" x="213.36" y="68.58" rot="R90"/>
-<instance part="U$2" gate="G$1" x="396.24" y="525.78"/>
-<instance part="U$3" gate="G$1" x="421.64" y="525.78"/>
+<instance part="FI1" gate="G$1" x="396.24" y="525.78"/>
+<instance part="FI2" gate="G$1" x="421.64" y="525.78"/>
+<instance part="C49" gate="G$1" x="447.04" y="472.44"/>
+<instance part="C44" gate="G$1" x="459.74" y="472.44"/>
+<instance part="C45" gate="G$1" x="472.44" y="472.44"/>
+<instance part="C46" gate="G$1" x="485.14" y="472.44"/>
+<instance part="C47" gate="G$1" x="497.84" y="472.44"/>
+<instance part="D2" gate="G$1" x="436.88" y="474.98" rot="R270"/>
 </instances>
 <busses>
@@
 <label x="264.16" y="81.28" size="1.778" layer="95"/>
 </segment>
+<segment>
+<wire x1="447.04" y1="467.36" x2="459.74" y2="467.36" width="0.1524" layer="91"/>
+<wire x1="459.74" y1="467.36" x2="472.44" y2="467.36" width="0.1524" layer="91"/>
+<wire x1="472.44" y1="467.36" x2="485.14" y2="467.36" width="0.1524" layer="91"/>
+<wire x1="485.14" y1="467.36" x2="497.84" y2="467.36" width="0.1524" layer="91"/>
+<wire x1="447.04" y1="467.36" x2="424.18" y2="467.36" width="0.1524" layer="91"/>
+<label x="424.18" y="467.36" size="1.778" layer="95"/>
+<pinref part="C49" gate="G$1" pin="-"/>
+<junction x="447.04" y="467.36"/>
+<pinref part="C44" gate="G$1" pin="-"/>
+<junction x="459.74" y="467.36"/>
+<pinref part="C45" gate="G$1" pin="-"/>
+<junction x="472.44" y="467.36"/>
+<pinref part="C46" gate="G$1" pin="-"/>
+<junction x="485.14" y="467.36"/>
+<pinref part="C47" gate="G$1" pin="-"/>
+</segment>
 </net>
 <net name="5V0" class="1">
@@
 <label x="335.28" y="220.98" size="1.778" layer="95"/>
 </segment>
+<segment>
+<pinref part="D2" gate="G$1" pin="C"/>
+<wire x1="434.34" y1="474.98" x2="424.18" y2="474.98" width="0.1524" layer="91"/>
+<label x="424.18" y="474.98" size="1.778" layer="95"/>
+</segment>
 </net>
 <net name="MENU_LEFT_BUTTON_PIN" class="2">
@@
 </segment>
 </net>
+<net name="N$6" class="0">
+<segment>
+<wire x1="447.04" y1="474.98" x2="459.74" y2="474.98" width="0.1524" layer="91"/>
+<pinref part="C49" gate="G$1" pin="+"/>
+<pinref part="C44" gate="G$1" pin="+"/>
+<wire x1="459.74" y1="474.98" x2="472.44" y2="474.98" width="0.1524" layer="91"/>
+<junction x="459.74" y="474.98"/>
+<pinref part="C45" gate="G$1" pin="+"/>
+<wire x1="472.44" y1="474.98" x2="485.14" y2="474.98" width="0.1524" layer="91"/>
+<junction x="472.44" y="474.98"/>
+<pinref part="C46" gate="G$1" pin="+"/>
+<wire x1="485.14" y1="474.98" x2="497.84" y2="474.98" width="0.1524" layer="91"/>
+<junction x="485.14" y="474.98"/>
+<pinref part="C47" gate="G$1" pin="+"/>
+<pinref part="D2" gate="G$1" pin="A"/>
+<wire x1="439.42" y1="474.98" x2="447.04" y2="474.98" width="0.1524" layer="91"/>
+<junction x="447.04" y="474.98"/>
+</segment>
+</net>
