File: misko_3_board.brd (EAGLE design)
At the start: 337 x 187 mm, 162 parts, among them CN1 LiPo Battery, IC1 MC1525TT, IC2 FT230XS, IC3 LTC4425, IC4 FM25W256-SOIC, IC5 74HCT1G32, M10 mid, Q1 FDN304P, T10 top, U1 ATMEGA1281-16AU, U2 SN74HCT14DR, U3 SN74LVC1G3157DBVR - BT switch, U4 SN74LVC1G3157DBVR - GPS switch, U5 TMP36GRTZ-REEL7, U7 MCP73871-2AAI/ML

Commit message: - added DS1394U-33+ RTC SPI Module, corrected a few traces
Parts:
- added C32: 0.1µF, rcl:C0805
- added R55: 10k, rcl:M0805
- added U$13: LFXTAL016178R, LFXTAL016178R 32.768kHz crystal:SMD
- added U$6: DS1394U-33+, DS1394U-33+ RTC SPI Module:10UMAX
Connections:
- removed net N$20: NTC.1, R27.2
- removed net PE2: B10.7, M10.7, T10.7, U1.4
- removed net PE3: B10.6, M10.6, T10.6, U1.5
- new net RTC_INT_INTERRUPT_PIN: B10.6, M10.6, T10.6, U$6.!INT!, U1.8
- new net RTC_XTAL1: U$13.XTAL1, U$6.X1
- new net RTC_XTAL2: U$13.XTAL2, U$6.X2
- new net SPI_SS_RTC_PIN: B10.7, M10.7, R55.2, T10.7, U$6.!CS!, U1.4
- new net VBACK: U$6.VBACK
- net GND: now also C32.2, R27.2, U$6.GND
- net N$19: now also NTC.1
- net SD_CARD_DETECT_PIN: now also U1.5; no longer U1.8
- net SPI_MISO_PIN: now also U$6.DOUT
- net SPI_MOSI_PIN: now also U$6.DIN
- net SPI_SCK_PIN: now also U$6.SCLK
- net VCC: now also C32.1, R55.1, U$6.VCC
Routing:
- net SPI_SS_RTC_PIN: track 0.00 -> 50.9 mm
- net RTC_INT_INTERRUPT_PIN: track 0.00 -> 47.5 mm, vias 0 -> 1
- net PE3: track 30.4 -> 0.00 mm
- net PE2: track 29.6 -> 0.00 mm
- net VCC: track 359.5 -> 386.3 mm, vias 26 -> 28
- net GPRS_LED: track 9.01 -> 27.9 mm
- net SPI_SCK_PIN: track 82.9 -> 96.3 mm
- net SPI_MOSI_PIN: track 81.0 -> 93.4 mm, vias 5 -> 6
- net GND: track 104.1 -> 116.1 mm
- net SPI_MISO_PIN: track 43.9 -> 49.1 mm, vias 3 -> 2
- net RTC_XTAL2: track 0.00 -> 4.37 mm
- net RTC_XTAL1: track 0.00 -> 4.37 mm
- net GPS_SW_SERIAL_RX: track 77.7 -> 81.6 mm, vias 1 -> 3
- net SD_CARD_DETECT_PIN: track 7.39 -> 4.86 mm
- net CENTER: track 22.1 -> 24.2 mm, vias 0 -> 1
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
Commit message: - checked against prototype schematic, minor error corrections
Parts:
- added C33: 10µF, rcl:C0805
- added U8: SIM800, SIM800 GPRS Module:SIM800C
- Q1: value FDN304P -> BSS84; device transistor-power:SOT223 -> transistor-small-signal:SOT23
- R40: value 46k -> 10k
- R45, R46: value 270k -> 1k
- R6, R7: value 21 -> 27
- U$1: value SIM800 -> F/UCW03F; device SIM800 GPRS Module:SIM800C -> buzzer:F/UCW03LF
- U$9: value TPS63001DRCR -> TPS63031
- U5: value TMP36GRTZ-REEL7 -> TMP36GRTZ
- moved U$1 163.1 mm to (89.0, 10.0), flipped to the top, turned to 90 degrees
- moved R41 5.32 mm to (318.5, 120.5), flipped to the bottom
- moved R50 5.25 mm to (309.2, 120.5), flipped to the bottom, turned to 180 degrees
- moved BT 4.83 mm to (27.7, 177.0)
- moved BT_LED 3.51 mm to (314.5, 123.8)
- moved GPRS_LED 3.50 mm to (314.5, 120.5)
- moved Q1 2.89 mm to (26.5, 179.5)
- renumbered ANT2 to ANT, U$8 to SUPERCAP
Connections:
- net N$35 renamed BT_LED
- net N$6 renamed USB_RX_LED
- removed net N$33: GPRS_LED.K, R50.1
- removed net VBACK: U$6.VBACK
- new net GPRS_NETLIGHT: BOARD.10, BR20.18, LID.10, MR20.18, R50.1, TR20.18, U8.NETLIGHT
- net AREF: now also C33.1
- net BLUE_LED: now also Q1.3; no longer Q1.2, Q1.4
- net GND: now also C33.2, GPRS_LED.K, R40.1, U$9.11, U7.21, U8.GND10, U8.GND2, U8.GND3, U8.GND4, U8.GND6, U8.GND7, U8.GND8, U8.GND9; no longer R50.2, U$1.GND10, U$1.GND2, U$1.GND3, U$1.GND4, U$1.GND6, U$1.GND7, U$1.GND8, U$1.GND9
- net GPRS_LED: now also R50.2; no longer BOARD.10, BR20.18, LID.10, MR20.18, TR20.18, U$1.NETLIGHT
- net GSM_ANT: now also U8.GSM_ANT; no longer U$1.GSM_ANT
- net SIM800C_CTS_PIN: now also U8.UART1_CTS; no longer U$1.UART1_CTS
- net SIM800C_POWER_PIN: now also U8.PWRKEY; no longer U$1.PWRKEY
- net SIM800C_RX_PIN: now also U8.UART1_TXD; no longer U$1.UART1_TXD
- net SIM800C_STATUS_PIN: now also U8.STATUS; no longer U$1.STATUS
- net SIM800C_TX_PIN: now also U8.UART1_RXD; no longer U$1.UART1_RXD
- net SIM_CLOCK: now also U8.SIM_CLK; no longer U$1.SIM_CLK
- net SIM_DATA: now also U8.SIM_DATA; no longer U$1.SIM_DATA
- net SIM_DETECT: now also U8.SIM_DET; no longer U$1.SIM_DET
- net SIM_RESET: now also U8.SIM_RST; no longer U$1.SIM_RST
- net SIM_VDD: now also U8.SIM_VDD; no longer U$1.SIM_VDD
- net VCC: now also Q1.2; no longer Q1.3, R40.1
- net VGPS: now also U$6.VBACK
- net V_LIION_REGULATED: now also U8.VBAT1, U8.VBAT2, U8.VRTC; no longer U$1.VBAT1, U$1.VBAT2, U$1.VRTC
Routing:
- net GPRS_NETLIGHT: track 0.00 -> 49.5 mm
- net GPRS_LED: track 27.9 -> 3.03 mm
- net VGPS: track 58.3 -> 79.6 mm, vias 1 -> 3
- net BLUETOOTH_WAKEUP_PIN: track 36.4 -> 27.1 mm
- net GND: track 116.1 -> 122.4 mm
- net AREF: track 3.17 -> 8.16 mm
- net VCC: track 386.3 -> 383.5 mm
- net N$33: track 2.62 -> 0.00 mm
- net BLUE_LED: track 65.0 -> 66.9 mm
- net VBACK: track 1.60 -> 0.00 mm, vias 1 -> 0
- net BT_GPIO6: track 7.39 -> 8.80 mm
- net BT_LED: track 2.62 -> 3.68 mm
- net RESET: track 70.9 -> 70.1 mm
- net SPI_MISO_PIN: track 49.1 -> 48.5 mm

Commit message: - added supervisor circuit to monitor VGPS and assert power on once conditions are met (functions as an AND gate: GPS_POWER_CTL_PIN AND min. 3V03 on VGPS will power on the GPS receiver)
Parts:
- removed GPS: PTR1B1,27, testpad:B1,27
- removed R1: 220, resistor:R0805
- added C34: 0.1µF, rcl:C0805
- added C35: 1nF, rcl:C0805
- added GPS_POWER_CTL_PIN: PTR1B1,27, testpad:B1,27
- added R56: 1M, resistor:R0805
- added U6: TPS3808G33DBVT, Texas Instruments_By_element14_Batch_1:SOT95P280X145-6N
- moved U$1 222.3 mm to (271.8, 136.5), turned to 180 degrees
- moved V_GPS1 17.7 mm to (196.5, 114.0)
- moved C15 7.65 mm to (188.5, 111.5), flipped to the bottom, turned to 0 degrees
- moved TP2 6.26 mm to (196.5, 119.5)
- moved R36 3.54 mm to (204.5, 124.0), turned to 180 degrees
- moved C16 1.75 mm to (204.5, 126.5), turned to 180 degrees
Connections:
- net GND: now also C34.1, C35.2, U6.2
- net GPS_ON_OFF: now also R56.1, U6.1; no longer BL20.12, GPS.TP, ML20.12, R1.1, TL20.12, TP2.TP
- net GPS_POWER_CTL_PIN: now also BL20.12, GPS_POWER_CTL_PIN.TP, ML20.12, TL20.12, TP2.TP, U6.3; no longer R1.2
- net VCC: now also C34.2, R56.2, U6.6
- net VGPS: now also C35.1, U6.5
Routing:
- net RESET: track 70.1 -> 167.0 mm
- net GPS_POWER_CTL_PIN: track 5.26 -> 55.8 mm, vias 0 -> 1
- net GPS_ON_OFF: track 45.4 -> 12.8 mm
- net VGPS: track 79.6 -> 106.3 mm, vias 3 -> 5
- net VCC: track 383.5 -> 387.8 mm
- net GPS_SW_SERIAL_TX: track 84.1 -> 85.7 mm
- net BUTTON_DOWN: track 17.8 -> 16.9 mm
- net BUTTON_CENTER: track 20.4 -> 21.0 mm
- net GPRS_BUTTON: track 32.4 -> 31.9 mm

Commit message: - corrected names and place layers for top and bottom
Parts:
- BOARD, LID: value 1.27-10-PIN-HEADER -> (none)
- JTAG: value JTAG-1.27-10-PIN-HEADER -> (none)
- TP6: value TPPAD1-17Y -> GND
- moved U$1 49.1 mm to (223.0, 131.0), turned to 0 degrees
- moved C39 7.75 mm to (210.8, 126.5), turned to 270 degrees
- moved R57 5.82 mm to (216.8, 126.5), turned to 270 degrees
- moved C12 4.06 mm to (213.7, 126.5), turned to 270 degrees
- moved SIM800 3.00 mm to (58.0, 159.8)
- moved C21 2.06 mm to (1.99, 180.5)
- moved BT 0.50 mm to (27.7, 176.5)
- moved C17 0.50 mm to (16.5, 7.00)
- moved R14 0.25 mm to (51.0, 161.8)
- moved R42 0.25 mm to (55.0, 161.8)
- moved V_GPS 0.25 mm to (-8.26, 172.0)
- renumbered CN1 to LIION, JP2 to I2C, OSCI to 8MHZ, S7 to RESET, S8 to POWER, U$2 to GND, U3 to BT-SW, U4 to GPS-SW
Connections:
- net N$1 renamed USB_TX_LED
- removed net PA7: BL20.15, ML20.15, TL20.15, U1.44
- new net BUZZER: BL20.14, ML20.14, TL20.14, U$1.SIGNAL, U1.44
- net BLUE_LED: now also BL20.15, ML20.15, TL20.15; no longer BL20.14, ML20.14, TL20.14
- net GND: now also GND.GND1, GND.GND2, GND.GND3, GND.GND4, GND.GND5, GND.GND6, U$1.GND, U$12.GND2, U$12.GND3, U$3.GND5, U$3.GND6, U$3.GND7, U$3.GND8; no longer GND.GND
Routing:
- net GND: track 122.4 -> 95.3 mm, vias 48 -> 54
- net BUZZER: track 0.00 -> 23.3 mm, vias 0 -> 2
- net VCC: track 387.8 -> 406.2 mm
- net PA7: track 9.68 -> 0.00 mm, vias 2 -> 0
- net OLED_VCC: track 12.0 -> 15.8 mm
- net SIM800C_POWER_PIN: track 76.5 -> 73.7 mm
- net IREF: track 18.6 -> 15.8 mm
- net RESET: track 167.0 -> 165.0 mm, vias 2 -> 1
- net BLUE_LED: track 66.9 -> 65.4 mm
- net VCOMH: track 16.0 -> 14.8 mm
- net BLUETOOTH_WAKEUP_PIN: track 27.1 -> 28.0 mm
- net GPRS_NETLIGHT: track 49.5 -> 48.9 mm
- net MENU_CENTER_BUTTON_PIN: track 17.2 -> 16.7 mm
Other:
- board text added: "1"
- board text added: "10"
- board text added: "2"
- board text added: "32k768"
- board text added: "9"
- board text added: "BT"
- board text added: "BT GPIO6"
- board text added: "BT RST"
- board text added: "BT wakeup"
- board text added: "C"
- board text added: "D"
- board text added: "GND"
- board text added: "GPRS"
- board text added: "GPS G"
- board text added: "GPS PWR"
- board text added: "GPS R"
- board text added: "L"
- board text added: "OFF"
- board text added: "ON"
- board text added: "R"
- board text added: "RX"
- board text added: "SIM800 PWR"
- board text added: "SW CTRL"
- board text added: "TX"
- board text added: "U"
- board text added: "VCC"
- board text added: "VGPS"
- board text added: "VLiIon"

Commit message: - corrected supercap orientation - routed remaining airwires - disapproved any error for last sanity check
Parts:
- moved SUPERCAP 20.1 mm to (3.01, 153.0), turned to 90 degrees
- moved R28 2.93 mm to (56.0, 26.8), turned to 0 degrees
- moved R27 0.78 mm to (53.8, 24.3), turned to 0 degrees
Connections:
- net GND: now also SUPERCAP.-; no longer SUPERCAP.+
- net VGPS: now also SUPERCAP.+; no longer SUPERCAP.-
Routing:
- net VCC: track 406.2 -> 456.4 mm, vias 28 -> 34
- net THERM: track 5.52 -> 2.21 mm
- net N$19: track 1.99 -> 4.77 mm
- net BLUE_LED: track 65.4 -> 64.0 mm

Commit message: - DRC completed
Routing:
- net VCC: track 456.4 -> 458.7 mm, vias 34 -> 35
- net RESET: track 165.0 -> 167.0 mm, vias 1 -> 2
Changed lines of the file:
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@@
 <hole x="319" y="110" drill="2"/>
 <hole x="319" y="124" drill="2"/>
-<wire x1="232.5" y1="137.5" x2="232.5" y2="120" width="0.4" layer="22"/>
+<wire x1="232.5" y1="137.5" x2="232.5" y2="120" width="0.25" layer="22"/>
 <wire x1="51" y1="35.5" x2="51" y2="25" width="0.25" layer="21"/>
 <wire x1="-7" y1="161.5" x2="-7" y2="149" width="0.25" layer="22" style="shortdash"/>
@@
 <wire x1="204" y1="119" x2="209" y2="119" width="0.25" layer="21" style="shortdash"/>
 <wire x1="209" y1="119" x2="209" y2="113.5" width="0.25" layer="21" style="shortdash"/>
-<wire x1="234" y1="121" x2="234" y2="110" width="0.25" layer="21"/>
+<wire x1="234" y1="121" x2="234" y2="109" width="0.25" layer="21"/>
 <wire x1="15.5" y1="172.5" x2="23.5" y2="172.5" width="0.25" layer="21" style="shortdash"/>
 <wire x1="23.5" y1="172.5" x2="23.5" y2="166.5" width="0.25" layer="21" style="shortdash"/>
@@
 <wire x1="44.25" y1="11.75" x2="26" y2="11.75" width="0.25" layer="21"/>
 <wire x1="26" y1="11.75" x2="26" y2="9" width="0.25" layer="21"/>
-<wire x1="205.5" y1="118" x2="222.75" y2="118" width="0.25" layer="21"/>
+<wire x1="205.5" y1="118" x2="222.75" y2="118" width="0.25" layer="22"/>
 <wire x1="44.25" y1="11.75" x2="44.25" y2="6.5" width="0.25" layer="21"/>
 <wire x1="44.25" y1="6.5" x2="59.5" y2="6.5" width="0.25" layer="21"/>
@@
 <wire x1="16.5" y1="150.5" x2="53.25" y2="150.5" width="0.3" layer="21"/>
 <wire x1="53.25" y1="150.5" x2="53.25" y2="148.5" width="0.3" layer="21"/>
+<wire x1="249.25" y1="105" x2="249.25" y2="109" width="0.25" layer="21"/>
+<wire x1="249.25" y1="109" x2="234" y2="109" width="0.25" layer="21"/>
 </plain>
 <attributes>
@@
 <via x="222.75" y="118" extent="1-16" drill="0.5" shape="octagon"/>
 <wire x1="235.55" y1="121" x2="234" y2="121" width="0.3" layer="16"/>
-<via x="234" y="121" extent="1-16" drill="0.6"/>
+<via x="234" y="121" extent="1-16" drill="0.6" shape="octagon"/>
 <wire x1="234" y1="121" x2="235.79" y2="121" width="0.3" layer="1"/>
 <wire x1="235.55" y1="115.5" x2="234" y2="115.5" width="0.3" layer="16"/>
-<via x="234" y="115.5" extent="1-16" drill="0.6"/>
+<via x="234" y="115.5" extent="1-16" drill="0.6" shape="octagon"/>
 <wire x1="234" y1="115.5" x2="235.79" y2="115.5" width="0.3" layer="1"/>
 <wire x1="235.55" y1="110" x2="234" y2="110" width="0.3" layer="16"/>
-<via x="234" y="110" extent="1-16" drill="0.6"/>
+<via x="234" y="110" extent="1-16" drill="0.6" shape="octagon"/>
 <wire x1="234" y1="110" x2="235.79" y2="110" width="0.3" layer="1"/>
 <wire x1="202.49" y1="140.65" x2="202.49" y2="140.51" width="0.4064" layer="1"/>
@@
 <wire x1="240.59" y1="105.35" x2="240.89925625" y2="105.35" width="0.3" layer="1"/>
 <wire x1="240.89925625" y1="105.35" x2="242.67005625" y2="103.5792" width="0.3" layer="1"/>
-<wire x1="242.67005625" y1="103.5792" x2="243.8292" y2="103.5792" width="0.3" layer="1"/>
 <wire x1="255.25" y1="115" x2="255.25" y2="119.5" width="0.3" layer="1"/>
 <wire x1="255.25" y1="119.5" x2="254.75" y2="120" width="0.3" layer="1"/>
 <wire x1="254.75" y1="120" x2="253.63" y2="120" width="0.3" layer="1"/>
-<wire x1="243.8292" y1="103.5792" x2="255.25" y2="115" width="0.3" layer="1"/>
 <wire x1="205.05" y1="116" x2="205.05" y2="117.55" width="0.3" layer="1"/>
 <wire x1="205.05" y1="117.55" x2="205.5" y2="118" width="0.3" layer="1"/>
@@
 <wire x1="52.04623125" y1="150.70376875" x2="53.25" y2="149.5" width="0.3" layer="16"/>
 <wire x1="53.25" y1="149.5" x2="53.25" y2="148.5" width="0.3" layer="16"/>
+<wire x1="242.67005625" y1="103.5792" x2="247.8292" y2="103.5792" width="0.3" layer="1"/>
+<wire x1="247.8292" y1="103.5792" x2="249.25" y2="105" width="0.3" layer="1"/>
+<via x="249.25" y="105" extent="1-16" drill="0.5" shape="octagon"/>
+<wire x1="249.25" y1="105" x2="249.25" y2="109" width="0.3" layer="1"/>
+<wire x1="249.25" y1="109" x2="255.25" y2="115" width="0.3" layer="1"/>
 <wire x1="20.99" y1="164.64520625" x2="44.58" y2="150.2375375" width="0" layer="19" extent="1-16"/>
 <wire x1="21.49" y1="38.65" x2="44.58" y2="148.38" width="0" layer="19" extent="1-1"/>
@@
 <wire x1="182.401" y1="139.901" x2="184.509" y2="142.009" width="0.25" layer="1"/>
 <wire x1="28" y1="10.95" x2="30" y2="10.95" width="0.25" layer="1"/>
+<wire x1="29" y1="10.95" x2="29" y2="13" width="0.25" layer="1"/>
+<via x="29" y="13" extent="1-16" drill="0.5"/>
 <wire x1="34.3932" y1="13.38" x2="37.99" y2="146.04" width="0" layer="19" extent="1-16"/>
+<wire x1="29" y1="10.95" x2="28" y2="10.95" width="0" layer="19" extent="1-1"/>
 <wire x1="54.51" y1="4.76" x2="34.24741875" y2="11.5" width="0" layer="19" extent="1-1"/>
 <wire x1="182.401" y1="139.901" x2="39.5" y2="147.55" width="0" layer="19" extent="1-16"/>

Commit message: - finished board & schematic, corrected BOM
Parts:
- removed 8MHZ: 8MHz, special:QS
- removed U$10: DJNR3015-1R5, DJNR3015-1R5 Inductor:FFF
- removed U$9: TPS63031, TI TPS63031:NEWPVSON-N10
- removed U1: ATMEGA1281-16AU, Atmel_By_element14_Batch_1-00:QFP80P1600X1600X120-64N
- removed U5: TMP36GRTZ, TMP36GRTZ:SOT95P280X145-5N
- removed U7: MCP73871-2AAI/ML, Microchip-MCP73871-2AAI_ML:QFN50P400X400X100-21N
- removed VCC, VCC5: PTR1TP14R, testpad:TP14R
- added IC12: LTC4425, LTC4425 Supercap Charger:DFN12
- added IC15: 74HCT1G32, 74HCT1G32GW:SOT353/5
- added IC16: FM25W256-SOIC, FM25W256 FERAM:SOIC08
- added IC7: FT230XS, ftdichip:SSOP16
- added L1: 33µH, rcl:L0805
- added T1: BSS84, transistor-small-signal:SOT23
- added TP1: GND, testpad:P1-17Y
- added TP4: VCC, testpad:TP14R
- CONN10: value (none) -> JTAG
- CONN12: value (none) -> board
- CONN13: value (none) -> lid
- IC1: value MC1525TT -> ATMEGA1281-16AU; device microchip:SOT23 -> Atmel_By_element14_Batch_1-00:QFP80P1600X1600X120-64N
- IC2: value FT230XS -> MC1525TT; device ftdichip:SSOP16 -> microchip:SOT23
- IC3: value LTC4425 -> TMP36GRTZ; device LTC4425 Supercap Charger:DFN12 -> TMP36GRTZ:SOT95P280X145-5N
- IC4: value FM25W256-SOIC -> TPS63031; device FM25W256 FERAM:SOIC08 -> TI TPS63031:NEWPVSON-N10
- IC5: value 74HCT1G32 -> MCP73871-2AAI/ML; device 74HCT1G32GW:SOT353/5 -> Microchip-MCP73871-2AAI_ML:QFN50P400X400X100-21N
- L2: value 33µH -> DJNR3015-1R5; device rcl:L0805 -> DJNR3015-1R5 Inductor:FFF
- Q1: value BSS84 -> 8MHz; device transistor-small-signal:SOT23 -> special:QS
- R1: value 10k -> NTC 10k
- R14, R42, R43, R44, R52, R53, R55, R57: device rcl:M0805 -> rcl:R0805
- R49: value 4.7k -> 4k7
- TP10, TP11: value PTR1TP14R -> VGPS
- TP2: value PTR1B1,27 -> VCC; device testpad:B1,27 -> testpad:TP14R
- TP3: value PTR1TP14R -> Analogue Switch CRTL Pin
- TP5: value PTR1B1,27 -> GPS Power CTRL Pin
- TP6: value GND -> GPS Power CTRL Pin; device testpad:P1-17Y -> testpad:B1,27
- TP7: value PTR1B1,27 -> SIM800 Power CTRL Pin
- TP8: value PTR1TP14R -> VLiIon Regulated
- TP9: value PTR1TP14R -> Bluetooth Wakeup Pin
- moved IC2 238.3 mm to (32.8, 32.6), flipped to the top, turned to 0 degrees
- moved Q1 171.4 mm to (37.0, 8.45), turned to 180 degrees
- moved TP2 166.8 mm to (69.0, 12.0), flipped to the bottom
- moved TP6 151.8 mm to (196.5, 119.5), turned to 0 degrees
- moved IC3 150.0 mm to (37.0, 33.0), flipped to the top, turned to 90 degrees
- moved IC4 60.1 mm to (70.0, 17.0), flipped to the bottom, turned to 180 degrees
- moved IC5 43.5 mm to (60.0, 29.0), flipped to the bottom, turned to 90 degrees
- moved L2 42.2 mm to (66.0, 17.0), flipped to the bottom, turned to 90 degrees
- moved IC1 12.7 mm to (38.0, 21.0)
- renumbered ANT to CONN15, B10 to CONN1, BL20 to CONN2, BLUETOOTH to S5, BOARD to CONN12, BR20 to CONN3, BT to TP9, BT-SW to IC8, BT_LED to LED5, GND to IC10, GPRS to S4, GPRS_LED to LED6, GPS-SW to IC9, GPS_GREEN_LED to LED1, GPS_POWER_CTL_PIN to TP5, GPS_RED_LED to LED2, I2C to CONN11, JTAG to CONN10, LID to CONN13, LIION to CONN16, M10 to CONN4, ML20 to CONN5, MR20 to CONN6, NTC to R1, OLED to IC18, POWER to S2, RESET to S1, SIM800 to TP7, SJ1 to JP2, SJ2 to JP3, SUPERCAP to C43, T10 to CONN7, TL20 to CONN8, TR20 to CONN9, U$11 to CONN14, U$12 to S3, U$13 to Q2, U$3 to IC13, U$4 to IC14, U$5 to IC17, U$6 to IC19, U$7 to IC20, U2 to IC6, U6 to IC11, U8 to IC21, USB_RX_LED to LED3, USB_TX_LED to LED4, VCC1 to TP3, V_GPS to TP10, V_GPS1 to TP11, V_LIION to TP8
Connections:
- net 5V0: now also IC5.17, IC5.18, IC5.19, IC5.3, IC5.4, IC5.9, IC7.12; no longer IC2.12, U7.17, U7.18, U7.19, U7.3, U7.4, U7.9
- net ADXL345SDA: now also IC15.Y; no longer IC5.Y
- net ADXL345_INT1_INTERRUPT_PIN: now also IC1.9; no longer U1.9
- net ANALOG_SW_CTRL_PIN: now also IC1.16; no longer U1.16
- net AREF: now also IC1.62, IC2.2; no longer IC1.2, U1.62
- net AVCC: now also IC1.64, IC2.1, L1.2; no longer IC1.1, L2.2, U1.64
- net BAT_A_PIN: now also IC1.58; no longer U1.58
- net BLUETOOTH_WAKEUP_PIN: now also IC1.48, T1.1; no longer Q1.1, U1.48
- net BLUE_LED: now also T1.3; no longer Q1.3
- net BUZZER: now also IC1.44; no longer U1.44
- net CBUS1: now also IC7.14; no longer IC2.14
- net CBUS2: now also IC7.7; no longer IC2.7
- net EN: now also IC4.6; no longer U$9.6
- net GND: now also IC1.22, IC1.53, IC1.63, IC12.GND, IC15.GND, IC16.GND, IC2.3, IC3.5, IC4.11, IC4.3, IC4.9, IC5.10, IC5.11, IC5.21, IC7.13, IC7.5, TP1.TP; no longer IC1.3, IC2.13, IC2.5, IC3.GND, IC4.GND, IC5.GND, TP6.TP, U$9.11, U$9.3, U$9.9, U1.22, U1.53, U1.63, U5.5, U7.10, U7.11, U7.21
- net GPS_GREEN_LED_PIN: now also IC1.42; no longer U1.42
- net GPS_POWER_CTL_PIN: now also IC1.49, TP6.TP; no longer TP2.TP, U1.49
- net GPS_RED_LED_PIN: now also IC1.41; no longer U1.41
- net GPS_SW_SERIAL_RX: now also IC1.14; no longer U1.14
- net GPS_SW_SERIAL_TX: now also IC1.15; no longer U1.15
- net GPS_WAKEUP_PIN: now also IC1.50; no longer U1.50
- net I2C_SCL_PIN: now also IC1.25; no longer U1.25
- net I2C_SDA_PIN: now also IC1.26; no longer U1.26
- net JTAG_TCL_PIN: now also IC1.57; no longer U1.57
- net JTAG_TDI_PIN: now also IC1.54; no longer U1.54
- net JTAG_TDO_PIN: now also IC1.55; no longer U1.55
- net JTAG_TMS_PIN: now also IC1.56; no longer U1.56
- net L1: now also IC4.4, L2.P$1; no longer U$10.P$1, U$9.4
- net L2: now also IC4.2, L2.P$2; no longer U$10.P$2, U$9.2
- net LTC4425_EN: now also IC12.EN; no longer IC3.EN
- net LTC4425_PROG: now also IC12.PROG; no longer IC3.PROG
- net MCP73871_CHARGE_STATUS_1_PIN: now also IC1.47, IC5.8; no longer U1.47, U7.8
- net MCP73871_CHARGE_STATUS_2_PIN: now also IC1.46, IC5.7; no longer U1.46, U7.7
- net MCP73871_POWER_GOOD_PIN: now also IC1.45, IC5.6; no longer U1.45, U7.6
- net MENU_BLUETOOTH_POWER_TOGGLE_PIN: now also IC1.39; no longer U1.39
- net MENU_CENTER_BUTTON_PIN: now also IC1.40; no longer U1.40
- net MENU_DOWN_BUTTON_PIN: now also IC1.38; no longer U1.38
- net MENU_GPRS_PUSH_BUTTON_PIN: now also IC1.43; no longer U1.43
- net MENU_LEFT_BUTTON_PIN: now also IC1.35; no longer U1.35
- net MENU_RIGHT_BUTTON_PIN: now also IC1.37; no longer U1.37
- net MENU_UP_BUTTON_PIN: now also IC1.36; no longer U1.36
- net N$10: now also IC7.10, IC7.11, IC7.3; no longer IC2.10, IC2.11, IC2.3
- net PDI_UART0_CTS_PIN: now also IC1.1, IC7.6; no longer IC2.6, U1.1
- net PDI_UART0_RX_PIN: now also IC1.2; no longer U1.2
- net PDI_UART0_TX_PIN: now also IC1.3; no longer U1.3
- net PFI: now also IC12.PFI; no longer IC3.PFI
- net PFI_RET: now also IC12.PFI_RET; no longer IC3.PFI_RET
- net PROG1: now also IC5.13; no longer U7.13
- net PROG3: now also IC5.12; no longer U7.12
- net RESET: now also IC1.20; no longer U1.20
- net RTC_INT_INTERRUPT_PIN: now also IC1.8; no longer U1.8
- net RXD: now also IC7.4; no longer IC2.4
- net SD_CARD_DETECT_PIN: now also IC1.5; no longer U1.5
- net SIM800C_CTS_PIN: now also IC1.29; no longer U1.29
- net SIM800C_POWER_PIN: now also IC1.31; no longer U1.31
- net SIM800C_RX_PIN: now also IC1.27; no longer U1.27
- net SIM800C_STATUS_PIN: now also IC1.30; no longer U1.30
- net SIM800C_TX_PIN: now also IC1.28; no longer U1.28
- net SPI_FRAM_SS_PIN: now also IC1.6, IC16.!CS!; no longer IC4.!CS!, U1.6
- net SPI_MISO_PIN: now also IC1.13, IC16.SO; no longer IC4.SO, U1.13
- net SPI_MOSI_PIN: now also IC1.12, IC15.B, IC16.SI; no longer IC4.SI, IC5.B, U1.12
- net SPI_OLED_D/C_PIN: now also IC1.17; no longer U1.17
- net SPI_OLED_RESET_PIN: now also IC1.18; no longer U1.18
- net SPI_SCK_PIN: now also IC1.11, IC16.SCK; no longer IC4.SCK, U1.11
- net SPI_SS_ADXL345_PIN: now also IC1.7, IC15.A; no longer IC5.A, U1.7
- net SPI_SS_OLED_PIN: now also IC1.19; no longer U1.19
- net SPI_SS_RTC_PIN: now also IC1.4; no longer U1.4
- net SPI_SS_SD_CARD_PIN: now also IC1.10; no longer U1.10
- net THERM: now also IC5.5; no longer U7.5
- net TMP36_SHUTDOWN_PIN: now also IC1.51, IC3.4; no longer U1.51, U5.4
- net TMP36_VSENSE_PIN: now also IC1.61, IC3.1; no longer U1.61, U5.1
- net TXD: now also IC7.1; no longer IC2.1
- net USBDM: now also IC7.9; no longer IC2.9
- net USBDP: now also IC7.8; no longer IC2.8
- net VCC: now also IC1.21, IC1.52, IC12.FB, IC12.SEL, IC12.VCC1, IC12.VCC2, IC15.VCC, IC16.!HOLD!, IC16.!WP!, IC16.VCC, IC3.2, IC4.1, IC4.10, L1.1, T1.2, TP2.TP, TP4.TP; no longer IC3.FB, IC3.SEL, IC3.VCC1, IC3.VCC2, IC4.!HOLD!, IC4.!WP!, IC4.VCC, IC5.VCC, L2.1, Q1.2, U$9.1, U$9.10, U1.21, U1.52, U5.2, VCC.TP, VCC5.TP
- net VCC_SENSE_PIN: now also IC1.60; no longer U1.60
- net VGPS: now also IC12.VOUT1, IC12.VOUT2; no longer IC3.VOUT1, IC3.VOUT2
- net VMID: now also IC12.VMID; no longer IC3.VMID
- net VPCC: now also IC5.2; no longer U7.2
- net V_LIION+: now also IC5.14, IC5.15, IC5.16; no longer U7.14, U7.15, U7.16
- net V_LIION_REGULATED: now also IC4.5, IC4.7, IC4.8, IC5.1, IC5.20; no longer U$9.5, U$9.7, U$9.8, U7.1, U7.20
- net V_SUPERCAP_SENSE_PIN: now also IC1.59; no longer U1.59
- net XTAL1: now also IC1.24, Q1.1; no longer 8MHZ.1, U1.24
- net XTAL2: now also IC1.23, Q1.2; no longer 8MHZ.2, U1.23
Other:
- board text added: "Bluetooth"
- board text added: "GPS"
- board text added: "Hrvoje Ivanić"
- board text added: "IC10"
- board text added: "IC13"
- board text added: "IC17"
- board text added: "IC20"
- board text added: "IC21"
- board text added: "Miško"
- board text added: "R1"
- board text added: "SCL"
- board text added: "SDA"
- board text added: "Stjenka Bojanić"

Commit message: - alpha version of PCB along with modified firmware
Connections:
- net BUZZER renamed BUZZER_PIN
- net V_SUPERCAP_SENSE_PIN renamed VGPS_SENSE_PIN
Changed lines of the file:
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@@
 <layer number="21" name="tPlace" color="7" fill="1" visible="yes" active="yes"/>
 <layer number="22" name="bPlace" color="7" fill="1" visible="yes" active="yes"/>
-<layer number="23" name="tOrigins" color="15" fill="1" visible="yes" active="yes"/>
-<layer number="24" name="bOrigins" color="15" fill="1" visible="yes" active="yes"/>
+<layer number="23" name="tOrigins" color="15" fill="1" visible="no" active="yes"/>
+<layer number="24" name="bOrigins" color="15" fill="1" visible="no" active="yes"/>
 <layer number="25" name="tNames" color="7" fill="1" visible="yes" active="yes"/>
 <layer number="26" name="bNames" color="7" fill="1" visible="yes" active="yes"/>
@@
 <wire x1="51.67" y1="180.04" x2="51.5" y2="180.05" width="0.254" layer="16"/>
 </signal>
-<signal name="V_SUPERCAP_SENSE_PIN" class="2">
+<signal name="VGPS_SENSE_PIN" class="2">
 <contactref element="R48" pad="2"/>
 <contactref element="R58" pad="1"/>
@@
 <wire x1="316.2" y1="123.75" x2="318.5" y2="121.45" width="0.25" layer="16"/>
 </signal>
-<signal name="BUZZER" class="3">
+<signal name="BUZZER_PIN" class="3">
 <contactref element="CONN2" pad="14"/>
 <contactref element="CONN5" pad="14"/>
