File: misko_1_board.sch (EAGLE design)
At the start: 167 parts, among them IC1 ATMEGA1281-16AU, IC10 ORG1510-MK4, IC11 TPS3808G33DBVT, IC12 LTC4425, IC13 RN-42, IC14 ADXL345, IC15 74HCT1G32, IC16 FM25W256-SOIC, IC17 MICROSD_SPI_MODE, IC18 FH12-30S-0.5SH, IC19 DS1394U-33+, IC2 MC1525TT, IC20 115Q-BCA0, IC21 SIM800, IC3 TMP36GRTZ, IC4 TPS63031, IC5 MCP73871-2AAI/ML, IC6 SN74HCT14DR, IC7 FT230XS, IC8 SN74LVC1G3157DBVR - BT switch, IC9 SN74LVC1G3157DBVR - GPS switch, Q1 8MHz, Q2 LFXTAL016178R, T1 BSS84

Commit message: - preliminary placement done. beer is now needed!
Parts:
- removed CONN14: MX500075-1517USB_MINI-B, MX500075-1517 USB Mini-B straight socket:MX500075-1517USB_MINI-B
- removed Q1: 8MHz, special:OSCILATOR
- removed S1: RESET, switch-omron:10-XX
- removed S4: gprs, switch-omron:10-XX
- removed S5: bt, switch-omron:10-XX
- added BT, GPRS, RESET: (no value), Wurth_Elektronik_Electromechanic_Switch_rev17c:430152050836
- added JTAG: JTAG-1.27-10-PIN-HEADER, JTAG 1.27mm 10pin header:JTAG-1.27-10-PIN-HEADER
- added U$3: ABM3B, ABM3B-8MHZ-10-1-U-T - Quartz Resonator:ABM3B
- added U$4: MX-67503-1230, MX-67503-1230 USB Mini-B SMT straight socket:MX-67503-1230
- added UI1, UI2: 1.27-10-PIN-HEADER, 1.27mm 10pin header:1.27-10-PIN-HEADER
- R25, R35: value 200k -> 150k
- R37, R38: value 100k -> 150k
- renumbered IC10 to U$2
Connections:
- new net N$11: UI1.10
- new net N$12: UI2.1
- new net N$13: UI2.2
- new net N$14: UI2.3
- new net N$15: UI2.4
- new net N$16: UI2.5
- new net N$17: UI2.6
- new net N$18: UI2.7
- new net N$2: UI1.1
- new net N$20: UI2.8
- new net N$21: UI2.9
- new net N$22: UI2.10
- new net N$23: UI1.7
- new net N$24: UI1.8
- new net N$3: UI1.2
- new net N$4: UI1.3
- new net N$5: UI1.4
- new net N$7: UI1.5
- new net N$8: UI1.6
- new net N$9: UI1.9
- net 5V0: now also L3.1; no longer L3.2
- net BUTTON_BLUETOOTH: now also BT.2, BT.4; no longer S5.S, S5.S1
- net GND: now also BT.1, BT.3, GPRS.1, GPRS.3, RESET.1, RESET.3, U$3.GND1, U$3.GND2, U$4.GND1, U$4.GND2, U$4.GND3, U$4.GND4, U$4.GND5; no longer CONN14.GND, S1.P, S1.P1, S4.P, S4.P1, S5.P, S5.P1, U$2.GND6
- net GPRS_BUTTON: now also GPRS.2, GPRS.4; no longer S4.S, S4.S1
- net RESET: now also RESET.2, RESET.4; no longer S1.S, S1.S1
- net USB_D+: now also U$4.D+; no longer CONN14.DP
- net USB_D-: now also U$4.D-; no longer CONN14.DN
- net VUSB: now also L3.2, U$4.VBUS; no longer CONN14.VBUS, L3.1
- net XTAL1: now also U$3.Q2; no longer Q1.P$1
- net XTAL2: now also U$3.Q1; no longer Q1.P$2
Other:
- moved on the sheet: L3

Commit message: - single board redrawn, pin mapping updated in pin_definitions.h - ERC&DRC to be checked next
Parts:
- removed C19: 100µF, rcl:C-EUC0805
- removed CONN11: I2C, jumper:JP1E
- removed IC6: SN74HCT14DR, Texas Instruments_By_element14_Batch_1:SN74HCT14DR
- removed JTAG: JTAG-1.27-10-PIN-HEADER, JTAG 1.27mm 10pin header:JTAG-1.27-10-PIN-HEADER
- removed R36: 10k, resistor:R-EU_R0805
- removed R48, R58: 150k, resistor:R-EU_R0805
- removed S3: MICROJOYSTICK, micro joystick:MICROJOYSTICK
- removed TP11: VGPS, testpad:PTR1TP14R
- removed TP2, TP4: VCC, testpad:PTR1TP14R
- removed TP5: GPS Power CTRL Pin, testpad:PTR1B1,27
- removed UI1, UI2: 1.27-10-PIN-HEADER, 1.27mm 10pin header:1.27-10-PIN-HEADER
- added C48: 100µF, rcl:C-EUC0805
- added GND, VCC, VUSB: GND, testpad:TPPAD1-17Y
- added I2C: (no value), jumper:JP4E
- added U$10: MICROJOYSTICK, micro joystick:MICROJOYSTICK
- added U$5: JTAG-1.27-10-PIN-HEADER, JTAG 1.27mm 10pin header:JTAG-1.27-10-PIN-HEADER
- added U$6, U$7, U$8, U$9: SN74LVC2G14DBVT, SN74LVC2G14 - Schmitt Trigger, inverting:SN74LVC2G14DBVT
- IC4: device TI TPS63031:TPS63001DRCR -> TPS63031 - Buck Boost Voltage Regulator:TPS63001DRCR
- IC5: device Microchip-MCP73871-2AAI_ML:MCP73871-2AAI/ML -> MCP73871 - Powerpath and Charge Controller:MCP73871-2AAI/ML
- TP1: value GND -> VCC; device testpad:TPPAD1-17Y -> testpad:PTR1TP14R
Connections:
- net GPRS_BUTTON renamed BUTTON_GPRS
- removed net MENU_BLUETOOTH_POWER_TOGGLE_PIN: IC1.PC4_(A12), IC6.5Y
- removed net N$11: UI1.10
- removed net N$12: UI2.1
- removed net N$13: UI2.2
- removed net N$14: UI2.3
- removed net N$15: UI2.4
- removed net N$16: UI2.5
- removed net N$17: UI2.6
- removed net N$18: UI2.7
- removed net N$2: UI1.1
- removed net N$20: UI2.8
- removed net N$21: UI2.9
- removed net N$22: UI2.10
- removed net N$23: UI1.7
- removed net N$24: UI1.8
- removed net N$3: UI1.2
- removed net N$4: UI1.3
- removed net N$5: UI1.4
- removed net N$7: UI1.5
- removed net N$8: UI1.6
- removed net N$9: UI1.9
- new net GPRS: C30.2, R22.2, U$8.1A
- new net MENU_BLUETOOTH_POWER_BUTTON_PIN: IC1.PG1_(~RD), U$8.2Y
- new net N$1: IC1.PA4_(AD4)
- new net N$25: IC1.PA5_(AD5)
- new net N$26: IC1.PA6_(AD6)
- net 5V0: now also IC5.!TE!, IC5.IN1, IC5.IN2; no longer IC5.*TE, IC5.IN, IC5.IN_2
- net BLUETOOTH: now also U$8.2A; no longer IC6.5A
- net BLUETOOTH_WAKEUP_PIN: now also IC1.PC5_(A13); no longer IC1.PA3_(AD3)
- net BUTTON_CENTER: now also U$10.CENTER; no longer S3.CENTER
- net BUTTON_DOWN: now also U$10.DOWN; no longer S3.DOWN
- net BUTTON_LEFT: now also U$10.LEFT; no longer S3.LEFT
- net BUTTON_RIGHT: now also U$10.RIGHT; no longer S3.RIGHT
- net BUTTON_UP: now also U$10.UP; no longer S3.UP
- net CENTER: now also U$7.2A; no longer IC6.4A
- net DOWN: now also U$9.2A; no longer IC6.6A
- net GND: now also GND.TP, I2C.1, IC12.GND1, IC12.GND2, IC12.GND3, IC5.GND1, IC5.GND2, IC5.GND3, IC5.GND4, IC5.GND5, IC5.GND6, U$10.GND1, U$10.GND2, U$10.GND3, U$5.GND1, U$5.GND2, U$6.2A, U$6.GND, U$7.GND, U$8.GND, U$9.GND; no longer IC12.GND, IC5.EP, IC5.VSS, IC5.VSS_2, IC6.GND, R36.2, R58.2, S3.GND1, S3.GND2, S3.GND3, TP1.TP
- net GPS_GREEN_LED_PIN: now also IC1.PG2_(ALE); no longer IC1.PC7_(A15)
- net GPS_ON_OFF: no longer R36.1
- net GPS_POWER_CTL_PIN: now also IC1.(T0)_PD7; no longer IC1.PA2_(AD2), TP5.TP
- net GPS_RED_LED_PIN: now also IC1.PC7_(A15); no longer IC1.PC6_(A14)
- net GPS_WAKEUP_PIN: now also IC1.PC6_(A14); no longer IC1.PA1_(AD1)
- net I2C_SCL_PIN: now also I2C.3; no longer CONN11.1
- net I2C_SDA_PIN: now also I2C.4; no longer CONN11.2
- net JTAG_TCL_PIN: now also U$5.TCK
- net JTAG_TDI_PIN: now also U$5.TDI
- net JTAG_TDO_PIN: now also U$5.TDO
- net JTAG_TMS_PIN: now also U$5.TMS
- net LEFT: now also U$7.1A; no longer IC6.1A
- net MCP73871_CHARGE_STATUS_1_PIN: now also IC1.PA1_(AD1), IC5.STAT1/!LBO!; no longer IC1.PA4_(AD4), IC5.STAT1/*LBO
- net MCP73871_CHARGE_STATUS_2_PIN: now also IC1.PA2_(AD2); no longer IC1.PA5_(AD5)
- net MCP73871_POWER_GOOD_PIN: now also IC1.PA3_(AD3), IC5.!PG!; no longer IC1.PA6_(AD6), IC5.*PG
- net MENU_CENTER_BUTTON_PIN: now also IC1.PC3_(A11), U$7.2Y; no longer IC1.PC5_(A13), IC6.4Y
- net MENU_DOWN_BUTTON_PIN: now also IC1.PC1_(A9), U$9.2Y; no longer IC1.PC3_(A11), IC6.6Y
- net MENU_GPRS_PUSH_BUTTON_PIN: now also IC1.PG0_(~WR), U$8.1Y; no longer C30.2, IC1.PG2_(ALE), R22.2
- net MENU_LEFT_BUTTON_PIN: now also IC1.PC2_(A10), U$7.1Y; no longer IC1.PC0_(A8), IC6.1Y
- net MENU_RIGHT_BUTTON_PIN: now also IC1.PC0_(A8), U$9.1Y; no longer IC1.PC2_(A10), IC6.3Y
- net MENU_UP_BUTTON_PIN: now also IC1.PC4_(A12), U$6.1Y; no longer IC1.PC1_(A9), IC6.2Y
- net RESET: now also U$5.RESET
- net RIGHT: now also U$9.1A; no longer IC6.3A
- net SD_CARD_DETECT_PIN: now also IC1.(XCK0/AIN0)_PE2; no longer IC1.(OC3A/AIN1)_PE3
- net SPI_SS_ADXL345_PIN: now also IC1.(~SS/PCINT0)_PB0; no longer IC1.(OC3C/INT5)_PE5
- net SPI_SS_RTC_PIN: now also IC1.(OC3C/INT5)_PE5; no longer IC1.(XCK0/AIN0)_PE2
- net SPI_SS_SD_CARD_PIN: now also IC1.(OC3A/AIN1)_PE3; no longer IC1.(~SS/PCINT0)_PB0
- net UP: now also U$6.1A; no longer IC6.2A
- net VCC: now also I2C.2, TP1.TP, U$5.VCC, U$6.VCC, U$7.VCC, U$8.VCC, U$9.VCC, VCC.TP; no longer C19.1, IC6.VCC, TP2.TP, TP4.TP
- net VGPS: now also C48.1; no longer R48.1, TP11.TP
- net VGPS_SENSE_PIN: no longer R48.2, R58.1
- net VMID: now also C48.2; no longer C19.2
- net VUSB: now also VUSB.TP
- net V_LIION+: now also IC5.VBAT1, IC5.VBAT2; no longer IC5.VBAT, IC5.VBAT_2
- net V_LIION_REGULATED: now also IC5.OUT1, IC5.OUT2; no longer IC5.OUT, IC5.OUT_2
Other:
- note removed: "VUSB (aka. supercap voltage) measurement"
- moved on the sheet: C2, C20, C4, C5, C7, C9, IC4, R10, R11, R12, R13, R16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

Commit message: - finished 1board layout, renamed pins where applicable, introduced WiFi module
Parts:
- removed BT, GPRS: (no value), Wurth_Elektronik_Electromechanic_Switch_rev17c:430152050836
- removed C44, C45, C46, C47, C49: 1000µF, rcl:CPOL-EUE22-10AXIAL
- removed C48: 100µF, rcl:C-EUC0805
- removed CONN15: U.FL-R-SMT 1, discrete:ANTENNASMD
- removed FI1, FI2: FIDUCIAL, adafruit:FIDUCIAL
- removed GND, VCC, VUSB: GND, testpad:TPPAD1-17Y
- removed I2C: (no value), jumper:JP4E
- removed LED6: red, led:LEDSQR2X5
- removed R37, R59: 150k, resistor:R-EU_R0805
- removed R50: 1k, resistor:R-EU_R0805
- removed R51: 47k, resistor:R-EU_R0805
- removed R52, R54: 1k, rcl:R-EU_R0805
- removed R53, R55: 10k, rcl:R-EU_R0805
- removed R56: 1M, resistor:R-EU_R0805
- removed R57: 390k, rcl:R-EU_R0805
- removed U$1: F/UCW03F, buzzer:F/UCW03F
- removed U$10: MICROJOYSTICK, micro joystick:MICROJOYSTICK
- removed U$4: MX-67503-1230, MX-67503-1230 USB Mini-B SMT straight socket:MX-67503-1230
- removed U$6, U$7, U$8, U$9: SN74LVC2G14DBVT, SN74LVC2G14 - Schmitt Trigger, inverting:SN74LVC2G14DBVT
- added C19: 1nF, rcl:C-EUC0805
- added CONN2: I2C, jumper:JP4E
- added CONN4: USB mini B, MX-67503-1230 USB Mini-B SMT straight socket:MX-67503-1230
- added CONN5: U.FL-R-SMT 1, discrete:ANTENNASMD
- added D3: (no value), diode:DIODE-SOD123
- added IC22: SIM800, SIM800 GPRS Module:SIM800
- added IC6: MAX6818, MAX6818 CMOS Switch debouncer:MAX6818
- added R36: 1k, rcl:R-EU_R0805
- added R48: 150k, resistor:R-EU_R0805
- added SJ1, SJ4: GPIO6, jumper:SJW
- added SW3: MICROJOYSTICK, micro joystick:MICROJOYSTICK
- added SW4, SW5: PB6156RSL, PB6156RSL Illuminated Tact SPST-NO switch:PB6156RSL
- added T2: BSS84, transistor-small-signal:BSS84
- added TP2: GND, testpad:TPPAD1-17Y
- added TP4: VCC, testpad:PTR1TP14R
- added TP5: VLiIon Regulated, testpad:PTR1TP14R
- C1: value 1µF -> 18pF; device resistor:C-EUC0805 -> rcl:C-EUC0805
- C10: value 100nF -> 1µF; device resistor:C-EUC0805 -> rcl:C-EUC0805
- C11: value 10µF -> 1µF; device resistor:C-EUC0805 -> rcl:C-EUC0805
- C12: value 4.7µF / 25V -> 10µF
- C13: value 10µF -> 15pF
- C15: value 18pF -> 1µF; device resistor:C-EUC0805 -> rcl:C-EUC0805
- C16: value 18pF -> 1µF
- C17, C34: value 0.1µF -> 10µF
- C18: value 10µF -> 2.2µF / 25V
- C2: value 0.47µF -> 1µF
- C20: value 100µF -> 0.1µF
- C21, C41: device rcl:C-EUC0805 -> resistor:C-EUC0805
- C22, C33: device resistor:C-EUC0805 -> rcl:C-EUC0805
- C23: value 15pF -> 10µF; device resistor:C-EUC0805 -> rcl:C-EUC0805
- C24: value 15pF -> 10µF
- C25: value 10µF -> 10pF
- C26: value 0.1µF -> (none); device rcl:C-EUC0805 -> EECS5R5H155 Supercap:EECS5R5H155
- C27: value 10µF -> 33pF
- C28: value 10µF -> 1000µF; device rcl:C-EUC0805 -> rcl:CPOL-EUE5-10.5
- C29: value 0.1µF -> 10µF; device resistor:C-EUC0805 -> rcl:C-EUC0805
- C30: value 0.47µF -> 1000µF; device resistor:C-EUC0805 -> rcl:CPOL-EUE5-10.5
- C31: value 0.1µF -> 1000µF; device rcl:C-EUC0805 -> rcl:CPOL-EUE5-10.5
- C35: value 1nF -> 1000µF; device rcl:C-EUC0805 -> rcl:CPOL-EUE5-10.5
- C36: value 1µF -> 0.1µF
- C37: value 1µF -> 10µF; device rcl:C-EUC0805 -> resistor:C-EUC0805
- C38: value 1µF -> 1000µF; device rcl:C-EUC0805 -> rcl:CPOL-EUE5-10.5
- C39: value 2.2µF -> 100µF
- C4: value 0.47µF -> 0.1µF; device resistor:C-EUC0805 -> rcl:C-EUC0805
- C40: value 1µF -> 100µF
- C42: value 4.7µF -> 100nF; device rcl:C-EUC0805 -> resistor:C-EUC0805
- C43: value EECS5R5H155 -> 0.1µF; device EECS5R5H155 Supercap:EECS5R5H155 -> rcl:C-EUC0805
- C5: value 0.47µF -> 10µF
- C6: value 10µF -> 4.7µF
- C7: value 0.47µF -> 10µF; device resistor:C-EUC0805 -> rcl:C-EUC0805
- C8: value 0.47µF -> 18pF
- C9: value 0.47µF -> 15pF
- CONN1: value JTAG-1.27-10-PIN-HEADER -> JTAG
- IC20: value 115Q-BCA0 -> ATWINC1500-MR210PB; device 115Q-BCA0 Micro-SIM Socket:115Q-BCA0 -> ATWINC1500-MR210PB WiFi Module:ATWINC1500-MR210PB
- IC21: value SIM800 -> 115Q-BCA0; device SIM800 GPRS Module:SIM800 -> 115Q-BCA0 Micro-SIM Socket:115Q-BCA0
- LED1: value green -> yellow; device led:LEDSQR2X5 -> led:LEDCHIPLED_1206
- LED2: value red -> yellow; device led:LEDSQR2X5 -> led:LEDCHIPLED_1206
- LED3: value yellow -> green; device led:LEDCHIPLED_1206 -> led:LEDSQR2X5
- LED4: value yellow -> red; device led:LEDCHIPLED_1206 -> led:LEDSQR2X5
- LED5: value blue -> red
- R1: value NTC 10k -> 47k; device rcl:R-EU_0204/5 -> rcl:R-EU_R0805
- R10, R47: value 47k -> 150k
- R11, R13, R21, R45: value 1k -> 10k
- R12: value 47k -> 27; device rcl:R-EU_R0805 -> resistor:R-EU_R0805
- R15: value 1k -> 270k; device resistor:R-EU_R0805 -> rcl:R-EU_R0805
- R16, R17: value 47k -> 1k; device rcl:R-EU_R0805 -> resistor:R-EU_R0805
- R2: value 3k3 -> 150k; device rcl:R-EU_R0805 -> resistor:R-EU_R0805
- R23: value 100k -> 1M
- R24: value 270k -> 1k; device rcl:R-EU_R0805 -> resistor:R-EU_R0805
- R25: value 150k -> 1k
- R26: value 47k -> 1k
- R27: value 270k -> 100k
- R28: value 1k -> 47k
- R29: value 47k -> 390k
- R3: value 3k3 -> 4k7
- R30: value 47k -> 10k; device rcl:R-EU_R0805 -> resistor:R-EU_R0805
- R31: value 1k -> 10k; device rcl:R-EU_R0805 -> resistor:R-EU_R0805
- R32: value 100k -> 1M; device rcl:R-EU_R0805 -> resistor:R-EU_R0805
- R33: value 150k -> 1k; device rcl:R-EU_R0805 -> resistor:R-EU_R0805
- R34: value 150k -> 47k; device rcl:R-EU_R0805 -> resistor:R-EU_R0805
- R35: value 150k -> 10k
- R38: value 150k -> 1k; device resistor:R-EU_R0805 -> rcl:R-EU_R0805
- R4, R5: value 1k -> 3k3; device resistor:R-EU_R0805 -> rcl:R-EU_R0805
- R41: value 1k -> 100k; device resistor:R-EU_R0805 -> rcl:R-EU_R0805
- R42: value 10k -> 1k
- R43: value 10k -> 270k
- R44: value 10k -> NTC 10k; device rcl:R-EU_R0805 -> rcl:R-EU_0204/5
- R46, R9: value 1k -> 150k
- R49: value 4k7 -> 150k; device rcl:R-EU_R0805 -> resistor:R-EU_R0805
- R6: value 27 -> 1k
- R8: value 47k -> 10k
- SW1: value (none) -> RESET
- SW2: value POWER_SWITCH -> POWER SWITCH
- TP1: value VCC -> GND; device testpad:PTR1TP14R -> testpad:TPPAD1-17Y
- TP10: value VGPS -> Bluetooth Wakeup Pin
- TP3: value Analogue Switch CRTL Pin -> GND; device testpad:PTR1TP14R -> testpad:TPPAD1-17Y
- TP6: value GPS Power CTRL Pin -> VGPS; device testpad:PTR1B1,27 -> testpad:PTR1TP14R
- TP7: value SIM800 Power CTRL Pin -> Analogue Switch CRTL Pin; device testpad:PTR1B1,27 -> testpad:PTR1TP14R
- TP8: value VLiIon Regulated -> GPS Power CTRL Pin; device testpad:PTR1TP14R -> testpad:PTR1B1,27
- TP9: value Bluetooth Wakeup Pin -> SIM800 Power CTRL Pin; device testpad:PTR1TP14R -> testpad:PTR1B1,27
- renumbered CONN16 to CONN3, JP2 to SJ2, JP3 to SJ3, RESET to SW1, S2 to SW2, U$2 to IC10, U$3 to Q1, U$5 to CONN1
Connections:
- net L1 renamed L_L1
- removed net BLUETOOTH: C8.2, R17.2, U$8.2A
- removed net BLUE_LED: C6.2, IC13.VCC, LED5.A, T1.D
- removed net BUZZER_PIN: IC1.PA7_(AD7), U$1.SIGNAL
- removed net CENTER: C9.2, R16.2, U$7.2A
- removed net DOWN: C4.2, R10.2, U$9.2A
- removed net GPRS: C30.2, R22.2, U$8.1A
- removed net GPRS_LED: LED6.A, R50.2
- removed net LEFT: C2.2, R8.2, U$7.1A
- removed net MENU_GPRS_PUSH_BUTTON_PIN: IC1.PG0_(~WR), U$8.1Y
- removed net N$1: IC1.PA4_(AD4)
- removed net N$25: IC1.PA5_(AD5)
- removed net N$26: IC1.PA6_(AD6)
- removed net OLED_VCC: C39.2, IC18-28.1
- removed net RIGHT: C7.2, R18.2, U$9.1A
- removed net UP: C5.2, R12.2, U$6.1A
- removed net VGPS_SENSE_PIN: IC1.PF2_(ADC2)
- new net !EN!: IC6.!EN!, SJ1.1
- new net BT_NETLIGHT_GATE: R31.2, T1.G
- new net BT_VCC: C7.2, IC13.VCC, T2.D
- new net GPRS_STATUS: IC1.PA6_(AD6), SW5.L1
- new net L_L2: IC4.L2, L2.L2
- new net MENU_GPRS_POWER_BUTTON_PIN: IC1.PC0_(A8), IC6.OUT3
- new net N$15: IC20.RESET_N, R13.1, SJ4.1
- new net N$3: R33.2, T1.S
- new net N$4: LED5.C, R33.1
- new net N$9: R25.1, R26.2, SW5.L2
- new net SPI_CFG: IC20.SPI_CFG, R23.2
- new net SPI_SS_WIFI_MODULE: IC1.PF0_(ADC0), IC20.SPI_SSN
- new net WIFI_EN_PIN: IC1.(T0)_PD7, IC20.CHIP_EN
- new net WIFI_IRQ_PIN: IC1.(OC3B/INT4)_PE4, IC20.IRQN
- new net WIFI_WAKE_PIN: IC1.PG0_(~WR), IC20.WAKE
- net 5V0: now also C42.2, R14.1; no longer C10.2, R23.1
- net ANALOG_SW_CTRL_PIN: now also IC1.PC7_(A15), TP7.TP; no longer IC1.(OC1B/PCINT6)_PB6, TP3.TP
- net ANTENNA: now also C33.2, CONN5.ANT, R42.2; no longer C28.2, CONN15.ANT, R52.2
- net AREF: now also C5.1; no longer C33.1
- net AVCC: now also C41.2; no longer C29.2
- net BAT_A_PIN: now also IC1.PF2_(ADC2), R46.2, R47.1; no longer IC1.PF3_(ADC3), R33.1, R34.2
- net BLUETOOTH_WAKEUP_PIN: now also IC1.PC6_(A14), R6.1, T2.G, TP10.TP; no longer IC1.PC5_(A13), R15.1, T1.G, TP9.TP
- net BT_LED: now also IC13.GPIO5, R24.1; no longer LED5.C, R41.2
- net BUTTON_BLUETOOTH: now also IC6.IN2, SW4.3; no longer BT.2, BT.4, R17.1, R20.1
- net BUTTON_CENTER: now also IC6.IN7, SW3.CENTER; no longer R16.1, R19.1, U$10.CENTER
- net BUTTON_DOWN: now also IC6.IN4, SW3.DOWN; no longer R10.1, R11.1, U$10.DOWN
- net BUTTON_GPRS: now also IC6.IN3, SW5.3; no longer GPRS.2, GPRS.4, R22.1, R54.1
- net BUTTON_LEFT: now also IC6.IN6, SW3.LEFT; no longer R8.1, R9.1, U$10.LEFT
- net BUTTON_RIGHT: now also IC6.IN5, SW3.RIGHT; no longer R18.1, R21.1, U$10.RIGHT
- net BUTTON_UP: now also IC6.IN8, SW3.UP; no longer R12.1, R13.1, U$10.UP
- net CAP1N: now also C10.1; no longer C40.1
- net CAP1P: now also C10.2; no longer C40.2
- net CAP2N: now also C11.1; no longer C36.1
- net CAP2P: now also C11.2; no longer C36.2
- net CBUS1: now also LED2.C; no longer LED4.C
- net CBUS2: now also LED1.C; no longer LED3.C
- net EN: now also R2.2; no longer R59.2
- net GND: now also C13.1, C16.1, C17.1, C19.2, C2.2, C21.2, C22.2, C23.2, C24.2, C25.1, C26.-, C28.-, C3.1, C30.-, C31.-, C33.1, C34.2, C35.-, C36.2, C37.2, C38.-, C4.2, C40.1, C41.1, C43.1, C5.2, CONN2.1, CONN4.GND1, CONN4.GND2, CONN4.GND3, CONN4.GND4, CONN4.GND5, CONN5.GND1, CONN5.GND2, D3.A, IC18-1.1, IC18-30.1, IC20.GND, IC20.PADDLE, IC21.GND1, IC21.GND5, IC22.GND10, IC22.GND2, IC22.GND3, IC22.GND4, IC22.GND6, IC22.GND7, IC22.GND8, IC22.GND9, IC6.GND, R10.2, R15.2, R2.1, R26.1, R29.1, R30.2, R38.2, R41.2, R43.2, R44.2, R47.2, R8.1, SJ1.2, SJ4.2, SW3.GND1, SW3.GND2, SW3.GND3, SW4.1, SW4.GND, SW5.1, SW5.GND, T1.D, TP1.TP; no longer BT.1, BT.3, C10.1, C11.2, C13.2, C16.2, C17.2, C2.1, C21.1, C22.1, C23.1, C24.1, C25.2, C26.1, C28.1, C3.2, C30.1, C31.2, C33.2, C34.1, C35.2, C37.1, C38.1, C39.1, C4.1, C41.2, C43.-, C44.-, C45.-, C46.-, C47.-, C49.-, C5.1, CONN15.GND1, CONN15.GND2, GND.TP, GPRS.1, GPRS.3, I2C.1, IC18-16.1, IC18-17.1, IC18-21.1, IC18-22.1, IC18-23.1, IC18-24.1, IC18-25.1, IC20.GND1, IC20.GND2, IC20.GND3, IC20.GND4, IC20.GND5, IC20.GND6, IC20.GND7, IC21.GND10, IC21.GND8, IC21.GND9, LED6.C, R1.2, R14.2, R24.2, R31.2, R32.2, R33.2, R35.2, R41.1, R42.1, R57.1, R59.1, U$1.GND, U$10.GND1, U$10.GND2, U$10.GND3, U$4.GND1, U$4.GND2, U$4.GND3, U$4.GND4, U$4.GND5, U$6.2A, U$6.GND, U$7.GND, U$8.GND, U$9.GND
- net GPIO4: now also R27.1; no longer R14.1
- net GPIO7: now also R8.2; no longer R42.2
- net GPRS_NETLIGHT: now also IC22.NETLIGHT, R30.1, R31.1; no longer IC21.NETLIGHT, R50.1
- net GPS_GREEN_LED_PIN: now also IC1.PA4_(AD4), R19.1; no longer IC1.PG2_(ALE), R46.1
- net GPS_ON_OFF: now also R32.1; no longer R56.1
- net GPS_POWER_CTL_PIN: now also IC1.PG2_(ALE), TP8.TP; no longer IC1.(T0)_PD7, TP6.TP
- net GPS_RED_LED_PIN: now also IC1.PA5_(AD5), R20.1; no longer IC1.PC7_(A15), R45.1
- net GPS_SW_SERIAL_TX: now also C8.2; no longer C15.2
- net GPS_TX: now also C1.1; no longer C16.1
- net GPS_WAKEUP_PIN: now also IC1.PA7_(AD7); no longer IC1.PC6_(A14)
- net GREEN_LED: now also LED3.C, R19.2; no longer LED1.C, R46.2
- net GSM_ANT: now also C29.2, IC22.GSM_ANT, R42.1; no longer C27.2, IC21.GSM_ANT, R52.1
- net I2C_SCL_PIN: now also CONN2.3; no longer I2C.3
- net I2C_SDA_PIN: now also CONN2.4; no longer I2C.4
- net IREF: now also R29.2; no longer R57.2
- net L2: now also R24.2, SW4.L2; no longer IC4.L2, L2.L2
- net MCP73871_CHARGE_STATUS_1_PIN: now also R28.2; no longer R30.2
- net MCP73871_CHARGE_STATUS_2_PIN: now also R22.2; no longer R29.2
- net MCP73871_POWER_GOOD_PIN: now also R18.2; no longer R26.2
- net MENU_BLUETOOTH_POWER_BUTTON_PIN: now also IC6.OUT2; no longer U$8.2Y
- net MENU_CENTER_BUTTON_PIN: now also IC1.PC4_(A12), IC6.OUT7; no longer IC1.PC3_(A11), U$7.2Y
- net MENU_DOWN_BUTTON_PIN: now also IC6.OUT4; no longer U$9.2Y
- net MENU_LEFT_BUTTON_PIN: now also IC1.PC3_(A11), IC6.OUT6; no longer IC1.PC2_(A10), U$7.1Y
- net MENU_RIGHT_BUTTON_PIN: now also IC1.PC2_(A10), IC6.OUT5; no longer IC1.PC0_(A8), U$9.1Y
- net MENU_UP_BUTTON_PIN: now also IC1.PC5_(A13), IC6.OUT8; no longer IC1.PC4_(A12), U$6.1Y
- net N$10: now also C14.1; no longer C3.1
- net N$19: now also R36.2, R43.1, R44.1; no longer R1.1, R27.1, R28.2
- net N$31: now also C3.2, R1.1; no longer C22.2, R47.1
- net N$6: now also C28.+, C30.+, C31.+, C35.+, C38.+; no longer C44.+, C45.+, C46.+, C47.+, C49.+
- net PDI_UART0_RX_PIN: now also R4.1; no longer R2.1
- net PDI_UART0_TX_PIN: now also R5.1; no longer R3.1
- net PFI: now also R48.1, R49.2; no longer R37.2, R38.1
- net PFI_RET: now also R49.1; no longer R37.1
- net PROG1: now also R38.1; no longer R31.1
- net PROG3: now also R41.1; no longer R32.1
- net RED_LED: now also LED4.C, R20.2; no longer LED2.C, R45.2
- net RESET: now also R1.2, R3.2; no longer R47.2, R49.2
- net RXD: now also R5.2; no longer R3.2
- net SIM800C_CTS_PIN: now also IC22.UART1_CTS; no longer IC21.UART1_CTS
- net SIM800C_POWER_PIN: now also IC22.PWRKEY, R34.1, TP9.TP; no longer IC21.PWRKEY, R51.1, TP7.TP
- net SIM800C_RX_PIN: now also IC22.UART1_TXD; no longer IC21.UART1_TXD
- net SIM800C_STATUS_PIN: now also IC22.STATUS; no longer IC21.STATUS
- net SIM800C_TX_PIN: now also IC22.UART1_RXD; no longer IC21.UART1_RXD
- net SIM_CLOCK: now also IC21.CLK, IC22.SIM_CLK; no longer IC20.CLK, IC21.SIM_CLK
- net SIM_DATA: now also C23.1, IC21.I/O, IC22.SIM_DATA; no longer C25.1, IC20.I/O, IC21.SIM_DATA
- net SIM_DETECT: now also IC21.CD, IC22.SIM_DET; no longer IC20.CD, IC21.SIM_DET
- net SIM_RESET: now also IC21.RST, IC22.SIM_RST; no longer IC20.RST, IC21.SIM_RST
- net SIM_VDD: now also IC21.VCC, IC22.SIM_VDD; no longer IC20.VPP, IC21.SIM_VDD
- net SPI_FRAM_SS_PIN: now also IC1.(~SS/PCINT0)_PB0, R21.1; no longer IC1.(OC3B/INT4)_PE4, R44.1
- net SPI_MISO_PIN: now also IC20.SPI_TXD
- net SPI_MOSI_PIN: now also IC20.SPI_RXD
- net SPI_SCK_PIN: now also IC20.SPI_SCK
- net SPI_SS_ADXL345_PIN: now also IC1.(OC1B/PCINT6)_PB6, R11.2; no longer IC1.(~SS/PCINT0)_PB0, R43.2
- net SPI_SS_RTC_PIN: now also R35.2; no longer R55.2
- net SPI_SS_SD_CARD_PIN: now also R45.1; no longer R53.1
- net THERM: now also R36.1; no longer R28.1
- net TMP36_VSENSE_PIN: now also IC1.PF3_(ADC3); no longer IC1.PF0_(ADC0)
- net TXD: now also R4.2; no longer R2.2
- net USBDM: now also R12.1; no longer R6.1
- net USB_D+: now also CONN4.D+; no longer U$4.D+
- net USB_D-: now also CONN4.D-, R12.2; no longer R6.2, U$4.D-
- net USB_RX_LED: now also LED1.A, R16.2; no longer LED3.A, R4.2
- net USB_TX_LED: now also LED2.A, R17.2; no longer LED4.A, R5.2
- net VCC: now also C12.2, C15.2, C16.2, C17.2, C20.2, C21.1, C22.1, C34.1, C36.1, C4.1, C43.2, CONN2.2, IC18-28.1, IC18-6.1, IC20.VDDIO, IC6.VCC, LED3.A, LED4.A, R11.1, R18.1, R22.1, R23.1, R25.2, R28.1, R3.1, R32.2, R35.1, R45.2, R48.2, R6.2, R9.1, SW4.L1, T2.S, TP3.TP, TP4.TP; no longer C14.1, C17.1, C18.2, C21.2, C31.1, C34.2, C37.2, C41.1, I2C.2, IC20.VCC, LED1.A, LED2.A, R11.2, R15.2, R19.2, R20.2, R25.1, R26.1, R29.1, R30.1, R38.2, R43.1, R44.2, R49.1, R53.2, R54.2, R55.1, R56.2, R9.2, T1.S, TP1.TP, U$6.VCC, U$7.VCC, U$8.VCC, U$9.VCC, VCC.TP
- net VCC_SENSE_PIN: now also R10.1, R9.2; no longer R25.2, R35.1
- net VCOMH: now also C18.2; no longer C12.2
- net VGPS: now also C19.1, C2.1, C26.+, C39.1, TP6.TP; no longer C1.1, C35.1, C43.+, C48.1, TP10.TP
- net VMID: now also C39.2, C40.2; no longer C20.2, C48.2
- net VPCC: now also R14.2, R15.1; no longer R23.2, R24.1
- net VUSB: now also CONN4.VBUS, R16.1, R17.1, TP2.TP; no longer R4.1, R5.1, U$4.VBUS, VUSB.TP
- net V_LIION+: now also C25.2, C27.2, C37.1, D3.C, IC20.VBATT, IC22.VBAT1, IC22.VBAT2, IC22.VRTC, R34.2, R46.1; no longer C13.1, R34.1
- net V_LIION_REGULATED: now also C24.1, C6.2, LED5.A, TP5.TP; no longer C11.1, C26.2, C38.2, C42.2, IC18-6.1, IC21.VBAT1, IC21.VBAT2, IC21.VRTC, R51.2, TP8.TP
- net XTAL1: now also C13.2; no longer C24.2
- net XTAL2: now also C9.2; no longer C23.2
Other:
- note added: "Debouncer"
- note added: "WiFi Module"
- note removed: "Buzzer"
- note removed: "Schmitt Trigger"
- moved on the sheet: C1, C10, C11, C12, C13, C14, C15, C16, C17, C18, C2, C20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

Commit message: - finished rev2 board with updated source code
Parts:
- removed LED5: red, led:LEDSQR2X5
- removed R23: 1M, rcl:R-EU_R0805
- removed R24: 1k, resistor:R-EU_R0805
- removed R48, R49: 150k, resistor:R-EU_R0805
- removed SJ4: GPIO6, jumper:SJW
- removed T2: BSS84, transistor-small-signal:BSS84
- added R37: 100k, rcl:R-EU_R0805
- added TP11: Bluetooth Wakeup Pin, testpad:PTR1TP14R
- C11, C16: value 1µF -> 10µF
- C12: value 10µF -> 15pF; device rcl:C-EUC0805 -> resistor:C-EUC0805
- C13: value 15pF -> 0.1µF
- C14: value 0.1µF -> 1µF; device resistor:C-EUC0805 -> rcl:C-EUC0805
- C17: value 10µF -> 2.2µF / 25V
- C18: value 2.2µF / 25V -> 1nF
- C19: value 1nF -> 0.1µF
- C20, C23: device rcl:C-EUC0805 -> resistor:C-EUC0805
- C21: device resistor:C-EUC0805 -> rcl:C-EUC0805
- C22: value 0.1µF -> 10µF
- C24: value 10µF -> 10pF; device resistor:C-EUC0805 -> rcl:C-EUC0805
- C25: value 10pF -> 1.5F; device rcl:C-EUC0805 -> EECS5R5H155 Supercap:EECS5R5H155
- C26: value (none) -> 33pF; device EECS5R5H155 Supercap:EECS5R5H155 -> rcl:C-EUC0805
- C27: value 33pF -> 1000µF; device rcl:C-EUC0805 -> rcl:CPOL-EUE5-10.5
- C28: value 1000µF -> 10µF; device rcl:CPOL-EUE5-10.5 -> rcl:C-EUC0805
- C42: value 100nF -> 0.1µF
- C7: value 10µF -> 18pF; device rcl:C-EUC0805 -> resistor:C-EUC0805
- C8: value 18pF -> 15pF
- C9: value 15pF -> 1µF; device resistor:C-EUC0805 -> rcl:C-EUC0805
- D2: value (none) -> BAT60AE6327; device eagle-ltspice:SCHOTTKY-DIODEF126Z12 -> diode:BAT60J
- D3: value (none) -> MMSZ5231B-DIO
- IC13: value RN-42 -> RN4678_BT_MODULE; device EN42-I Bluetooth Module:RN-42 -> RN4678 Bluetooth 4.2 Dual Mode:RN4678_BT_MODULE
- R10: value 150k -> 27; device rcl:R-EU_R0805 -> resistor:R-EU_R0805
- R12: value 27 -> 100k; device resistor:R-EU_R0805 -> rcl:R-EU_R0805
- R13: value 10k -> 270k
- R14: value 100k -> 1k; device rcl:R-EU_R0805 -> resistor:R-EU_R0805
- R15: value 270k -> 1k; device rcl:R-EU_R0805 -> resistor:R-EU_R0805
- R16: value 1k -> 47k; device resistor:R-EU_R0805 -> rcl:R-EU_R0805
- R17, R33: device resistor:R-EU_R0805 -> rcl:R-EU_R0805
- R18: value 47k -> 1k
- R19: value 1k -> 10k
- R20, R25: value 1k -> 47k
- R21: value 10k -> 1M
- R22: value 47k -> 1k; device rcl:R-EU_R0805 -> resistor:R-EU_R0805
- R26: value 1k -> 390k
- R27: value 100k -> 10k; device rcl:R-EU_R0805 -> resistor:R-EU_R0805
- R28: value 47k -> 10k; device rcl:R-EU_R0805 -> resistor:R-EU_R0805
- R29: value 390k -> 1M; device rcl:R-EU_R0805 -> resistor:R-EU_R0805
- R30: value 10k -> 1k
- R31: value 10k -> 47k
- R32: value 1M -> 10k; device resistor:R-EU_R0805 -> rcl:R-EU_R0805
- R34: value 47k -> 1k; device resistor:R-EU_R0805 -> rcl:R-EU_R0805
- R35: value 10k -> 1k; device rcl:R-EU_R0805 -> resistor:R-EU_R0805
- R36, R42: value 1k -> 10k; device rcl:R-EU_R0805 -> resistor:R-EU_R0805
- R39: value 1k -> 270k; device resistor:R-EU_R0805 -> rcl:R-EU_R0805
- R40: value 10k -> NTC 10k; device resistor:R-EU_R0805 -> rcl:R-EU_0204/5
- R41: value 100k -> 10k
- R43: value 270k -> 10k; device rcl:R-EU_R0805 -> resistor:R-EU_R0805
- R44: value NTC 10k -> 150k; device rcl:R-EU_0204/5 -> rcl:R-EU_R0805
- R45, R8: value 10k -> 150k
- R46, R47: device rcl:R-EU_R0805 -> resistor:R-EU_R0805
- R6: value 1k -> 27
- R7: value 27 -> 150k; device resistor:R-EU_R0805 -> rcl:R-EU_R0805
- R9: value 150k -> 10k
- SJ1: value GPIO6 -> WiFi RST
Connections:
- removed net BT_GPIO6: IC13.GPIO6, SJ2.2
- removed net BT_NETLIGHT_GATE: R31.2, T1.G
- removed net BT_RST: IC13.RESET, SJ3.2
- removed net BT_VCC: C7.2, IC13.VCC, T2.D
- removed net GPIO4: IC13.GPIO4, R27.1
- removed net GPIO7: IC13.GPIO7, R8.2
- removed net GPRS_STATUS: IC1.PA6_(AD6), SW5.L1
- removed net N$4: LED5.C, R33.1
- removed net N$9: R25.1, R26.2, SW5.L2
- removed net SIM800C_STATUS_PIN: IC1.(XCK1)_PD5, IC22.STATUS
- removed net TMP36_SHUTDOWN_PIN: IC1.PA0_(AD0), IC3.~SHDN
- new net BLUETOOTH_PROF_IND_PIN: IC1.PG2_(ALE), IC13.P0_5, TP11.TP
- new net BLUETOOTH_SWITCH_PIN: IC1.PC6_(A14), IC13.SW_BTN, R43.2
- new net GPRS_NETLIGHT_GATE: R28.2, T1.G
- new net LDO33_O: IC13.LDO33_O, IC13.VDD_IO, SW4.L1
- new net N$1: R30.1, SW5.L2
- new net N$11: IC13.!RST_N!, SJ3.1
- new net SIM800C_POWER_CTRL_PIN: IC1.(XCK1)_PD5, IC22.STATUS, TP10.TP
- net !EN!: now also SJ2.1; no longer SJ1.1
- net 5V0: now also D2.A, R12.1; no longer D2.C, R14.1
- net ANALOG_SW_CTRL_PIN: now also IC1.PA7_(AD7); no longer IC1.PC7_(A15)
- net ANTENNA: now also R38.2; no longer R42.2
- net BAT_A_PIN: now also R44.2, R45.1; no longer R46.2, R47.1
- net BLUETOOTH_RX: now also IC13.RXD; no longer IC13.UART_RX
- net BLUETOOTH_TX: now also IC13.TXD; no longer IC13.UART_TX
- net BLUETOOTH_WAKEUP_PIN: now also IC1.PC7_(A15), IC13.WAKEUP, R42.2; no longer IC1.PC6_(A14), R6.1, T2.G, TP10.TP
- net BT_LED: now also IC13.LED, R22.1; no longer IC13.GPIO5, R24.1
- net BUTTON_BLUETOOTH: now also IC6.IN7; no longer IC6.IN2
- net BUTTON_CENTER: now also IC6.IN5; no longer IC6.IN7
- net BUTTON_DOWN: now also IC6.IN2; no longer IC6.IN4
- net BUTTON_GPRS: now also IC6.IN8; no longer IC6.IN3
- net BUTTON_LEFT: now also IC6.IN4; no longer IC6.IN6
- net BUTTON_RIGHT: now also IC6.IN3; no longer IC6.IN5
- net BUTTON_UP: now also IC6.IN6; no longer IC6.IN8
- net CAP1N: now also C9.1; no longer C10.1
- net CAP1P: now also C9.2; no longer C10.2
- net CAP2N: now also C10.1; no longer C11.1
- net CAP2P: now also C10.2; no longer C11.2
- net GND: now also C11.1, C13.2, C14.1, C18.2, C19.1, C20.2, C24.1, C25.-, C26.1, C27.-, C28.1, C29.2, IC13.GND, R13.2, R34.2, R36.1, R37.2, R39.2, R40.2, R42.1, R43.1, R45.2, R8.2, SJ2.2, SJ3.2; no longer C13.1, C14.2, C18.1, C19.2, C20.1, C24.2, C25.1, C26.-, C27.1, C28.-, C29.1, C9.1, IC13.GND1, IC13.GND2, IC13.GND3, IC13.GND4, IC13.GND5, IC13.GND6, IC13.GND7, IC13.GND8, IC13.GPIO3, R10.2, R15.2, R29.1, R30.2, R38.2, R40.1, R41.2, R43.2, R44.2, R47.2, R8.1, SJ2.1, SJ3.1, SJ4.2
- net GPRS_NETLIGHT: now also R27.1, R28.1; no longer R30.1, R31.1
- net GPS_GREEN_LED_PIN: now also IC1.PA3_(AD3), R17.1; no longer IC1.PA4_(AD4), R19.1
- net GPS_ON_OFF: now also R29.1; no longer R32.1
- net GPS_POWER_CTL_PIN: now also IC1.PA6_(AD6); no longer IC1.PG2_(ALE)
- net GPS_RED_LED_PIN: now also IC1.PA4_(AD4), R18.1; no longer IC1.PA5_(AD5), R20.1
- net GPS_SW_SERIAL_TX: now also C7.2; no longer C8.2
- net GPS_WAKEUP_PIN: now also IC1.PA5_(AD5); no longer IC1.PA7_(AD7)
- net GREEN_LED: now also R17.2; no longer R19.2
- net GSM_ANT: now also C28.2, R38.1; no longer C29.2, R42.1
- net IREF: now also R26.2; no longer R29.2
- net L2: now also R22.2; no longer R24.2
- net LTC4425_EN: now also R35.2; no longer R39.2
- net LTC4425_PROG: now also R36.2; no longer R40.2
- net MCP73871_CHARGE_STATUS_1_PIN: now also IC1.PA0_(AD0), R25.2; no longer IC1.PA1_(AD1), R28.2
- net MCP73871_CHARGE_STATUS_2_PIN: now also IC1.PA1_(AD1), R20.2; no longer IC1.PA2_(AD2), R22.2
- net MCP73871_POWER_GOOD_PIN: now also IC1.PA2_(AD2), R16.2; no longer IC1.PA3_(AD3), R18.2
- net MENU_BLUETOOTH_POWER_BUTTON_PIN: now also IC1.PC4_(A12), IC6.OUT7; no longer IC1.PG1_(~RD), IC6.OUT2
- net MENU_CENTER_BUTTON_PIN: now also IC1.PC2_(A10), IC6.OUT5; no longer IC1.PC4_(A12), IC6.OUT7
- net MENU_DOWN_BUTTON_PIN: now also IC1.PG1_(~RD), IC6.OUT2; no longer IC1.PC1_(A9), IC6.OUT4
- net MENU_GPRS_POWER_BUTTON_PIN: now also IC1.PC5_(A13), IC6.OUT8; no longer IC1.PC0_(A8), IC6.OUT3
- net MENU_LEFT_BUTTON_PIN: now also IC1.PC1_(A9), IC6.OUT4; no longer IC1.PC3_(A11), IC6.OUT6
- net MENU_RIGHT_BUTTON_PIN: now also IC1.PC0_(A8), IC6.OUT3; no longer IC1.PC2_(A10), IC6.OUT5
- net MENU_UP_BUTTON_PIN: now also IC1.PC3_(A11), IC6.OUT6; no longer IC1.PC5_(A13), IC6.OUT8
- net N$10: now also C13.1; no longer C14.1
- net N$15: now also R11.1, SJ1.1; no longer R13.1, SJ4.1
- net N$19: now also R33.2, R39.1, R40.1; no longer R36.2, R43.1, R44.1
- net N$3: now also R30.2; no longer R33.2
- net N$6: now also C27.+, D2.C; no longer C28.+, D2.A
- net PFI: now also R46.1, R47.2; no longer R48.1, R49.2
- net PFI_RET: now also R47.1; no longer R49.1
- net PROG1: now also R34.1; no longer R38.1
- net PROG3: now also R37.1; no longer R41.1
- net RED_LED: now also R18.2; no longer R20.2
- net SIM800C_POWER_PIN: now also R31.1; no longer R34.1
- net SIM_DATA: now also C22.1; no longer C23.1
- net SPI_CFG: now also R21.2; no longer R23.2
- net SPI_FRAM_SS_PIN: now also R19.1; no longer R21.1
- net SPI_SS_ADXL345_PIN: now also R9.2; no longer R11.2
- net SPI_SS_RTC_PIN: now also R32.2; no longer R35.2
- net SPI_SS_SD_CARD_PIN: now also R41.1; no longer R45.1
- net THERM: now also R33.1; no longer R36.1
- net USBDM: now also R10.1; no longer R12.1
- net USBDP: now also R6.2; no longer R7.2
- net USB_D+: now also R6.1; no longer R7.1
- net USB_D-: now also R10.2; no longer R12.2
- net USB_RX_LED: now also R14.2; no longer R16.2
- net USB_TX_LED: now also R15.2; no longer R17.2
- net VCC: now also C11.2, C14.2, C19.2, C20.1, C29.1, IC13.BAT_IN, IC3.~SHDN, R11.2, R16.1, R19.2, R20.1, R21.1, R25.1, R29.2, R32.1, R41.2, R46.2, R7.1; no longer C12.2, C17.2, C20.2, C22.1, R11.1, R13.2, R18.1, R21.2, R22.1, R23.1, R25.2, R28.1, R32.2, R39.1, R45.2, R48.2, R6.2, SW4.L1, T2.S
- net VCC_SENSE_PIN: now also R7.2, R8.1; no longer R10.1, R9.2
- net VCOMH: now also C17.2; no longer C18.2
- net VGPS: now also C18.1, C25.+; no longer C19.1, C26.+
- net VPCC: now also R12.2, R13.1; no longer R14.2, R15.1
- net VUSB: now also R14.1, R15.1; no longer R16.1, R17.1
- net V_LIION+: now also C24.2, C26.2, R31.2, R44.1; no longer C25.2, C27.2, R34.2, R46.1
- net V_LIION_REGULATED: now also C23.1, SW5.L1; no longer C24.1, LED5.A
- net XTAL1: now also C12.2; no longer C13.2
- net XTAL2: now also C8.2; no longer C9.2
Other:
- moved on the sheet: C10, C11, C12, C13, C14, C15, C16, C17, C18, C19, C20, C21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
