File: misko_1_board.sch (EAGLE design)
At the start: 152 parts, among them IC1 ATMEGA1281-16AU, IC10 ORG1510-MK4, IC11 TPS3808G33DBVT, IC12 LTC4425, IC13 RN4678_BT_MODULE, IC14 ADXL345, IC15 74HCT1G32, IC16 FM25W256-SOIC, IC17 MICROSD_SPI_MODE, IC18 FH12-30S-0.5SH, IC19 DS1394U-33+, IC2 MC1525TT, IC20 ATWINC1500-MR210PB, IC21 115Q-BCA0, IC22 SIM800, IC23 SP3012-04UTG, IC3 TMP36GRTZ, IC4 TPS63031, IC5 MCP73871-2AAI/ML, IC6 MAX6818, IC7 FT230XS, IC8 SN74LVC1G3157DBVR - BT switch, IC9 SN74LVC1G3157DBVR - GPS switch, Q1 ABM3B-8MHZ-10-1-U-T, Q2 LFXTAL016178R, SW1 RESET, SW2 POWER SWITCH, SW3 MICROJOYSTICK, SW4 PB6156RSL, SW5 PB6156RSL, T1 BSS84

Commit message: - set LTC4425 resistor divider values to 470k on Vmid pin
Parts:
- R46, R47: value 150k -> 470k
Changed lines of the file:
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@@
 <part name="C1" library="rcl" deviceset="C-EU" device="C0805" value="18pF"/>
 <part name="IC12" library="LTC4425 Supercap Charger" deviceset="LTC4425" device=""/>
-<part name="R47" library="resistor" library_urn="urn:adsk.eagle:library:348" deviceset="R-EU_" device="R0805" package3d_urn="urn:adsk.eagle:package:26059/1" value="150k"/>
-<part name="R46" library="resistor" library_urn="urn:adsk.eagle:library:348" deviceset="R-EU_" device="R0805" package3d_urn="urn:adsk.eagle:package:26059/1" value="150k"/>
+<part name="R47" library="resistor" library_urn="urn:adsk.eagle:library:348" deviceset="R-EU_" device="R0805" package3d_urn="urn:adsk.eagle:package:26059/1" value="470k"/>
+<part name="R46" library="resistor" library_urn="urn:adsk.eagle:library:348" deviceset="R-EU_" device="R0805" package3d_urn="urn:adsk.eagle:package:26059/1" value="470k"/>
 <part name="R35" library="resistor" library_urn="urn:adsk.eagle:library:348" deviceset="R-EU_" device="R0805" package3d_urn="urn:adsk.eagle:package:26059/1" value="1k"/>
 <part name="R36" library="resistor" library_urn="urn:adsk.eagle:library:348" deviceset="R-EU_" device="R0805" package3d_urn="urn:adsk.eagle:package:26059/1" value="10k"/>
