File: eagle design/misko_nucleo.sch (EAGLE design)
At the start: 131 parts, among them CN1 LiPo Battery, IC1 MC1525TT, IC10 LTC4425, IC11 SP3012-04UTG, IC2 ORG1510-MK4, IC3 TPS63031, IC4 FT230XS, IC5 RN4678_BT_MODULE, IC6 FM25W256-SOIC, IC7 MICROSD_SPI_MODE, IC8 DS1394U-33+, IC9 MAX6818, Q1 ABM3B-8MHZ-10-1-U-T, Q2 BSS84, Q3 LFXTAL016178R, SW1 MICROJOYSTICK, SW2 PB6156RSL, SW3 PB6156RSL, U1 SN74LVC1G3157DBVR - BT switch, U2 ATMEGA1281-16AU, U3 TPS3808G33DBVT, U4 TMP36GRTZ, U5 MCP73871-2AAI/ML, U6 SN74LVC1G3157DBVR - GPS switch, X1 FH12-30S-0.5SH

Commit message: in main.c & sch/brd: - ditched dedicated SPI CS pullup resistors and switched to stm32 built-in pullups
Connections:
- net 3V3: no longer R1.2
- net ADXL345_CS: no longer R1.1
Changed lines of the file:
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@@
 <grid distance="0.1" unitdist="inch" unit="inch" style="lines" multiple="1" display="no" altdistance="0.01" altunitdist="inch" altunit="inch"/>
 <layers>
-<layer number="1" name="Top" color="4" fill="1" visible="yes" active="no"/>
-<layer number="2" name="Route2" color="1" fill="3" visible="yes" active="no"/>
-<layer number="3" name="Route3" color="4" fill="3" visible="yes" active="no"/>
-<layer number="4" name="Route4" color="1" fill="4" visible="yes" active="no"/>
-<layer number="5" name="Route5" color="4" fill="4" visible="yes" active="no"/>
-<layer number="6" name="Route6" color="1" fill="8" visible="yes" active="no"/>
-<layer number="7" name="Route7" color="4" fill="8" visible="yes" active="no"/>
-<layer number="8" name="Route8" color="1" fill="2" visible="yes" active="no"/>
-<layer number="9" name="Route9" color="4" fill="2" visible="yes" active="no"/>
-<layer number="10" name="Route10" color="1" fill="7" visible="yes" active="no"/>
-<layer number="11" name="Route11" color="4" fill="7" visible="yes" active="no"/>
-<layer number="12" name="Route12" color="1" fill="5" visible="yes" active="no"/>
-<layer number="13" name="Route13" color="4" fill="5" visible="yes" active="no"/>
-<layer number="14" name="Route14" color="1" fill="6" visible="yes" active="no"/>
-<layer number="15" name="Route15" color="4" fill="6" visible="yes" active="no"/>
-<layer number="16" name="Bottom" color="1" fill="1" visible="yes" active="no"/>
-<layer number="17" name="Pads" color="2" fill="1" visible="yes" active="no"/>
-<layer number="18" name="Vias" color="2" fill="1" visible="yes" active="no"/>
-<layer number="19" name="Unrouted" color="6" fill="1" visible="yes" active="no"/>
-<layer number="20" name="Dimension" color="14" fill="1" visible="yes" active="no"/>
-<layer number="21" name="tPlace" color="7" fill="1" visible="yes" active="no"/>
-<layer number="22" name="bPlace" color="7" fill="1" visible="yes" active="no"/>
-<layer number="23" name="tOrigins" color="15" fill="1" visible="yes" active="no"/>
-<layer number="24" name="bOrigins" color="15" fill="1" visible="yes" active="no"/>
-<layer number="25" name="tNames" color="7" fill="1" visible="yes" active="no"/>
-<layer number="26" name="bNames" color="7" fill="1" visible="yes" active="no"/>
-<layer number="27" name="tValues" color="7" fill="1" visible="yes" active="no"/>
-<layer number="28" name="bValues" color="7" fill="1" visible="yes" active="no"/>
+<layer number="1" name="Top" color="4" fill="1" visible="no" active="no"/>
+<layer number="2" name="Route2" color="1" fill="3" visible="no" active="no"/>
+<layer number="3" name="Route3" color="4" fill="3" visible="no" active="no"/>
+<layer number="4" name="Route4" color="1" fill="4" visible="no" active="no"/>
+<layer number="5" name="Route5" color="4" fill="4" visible="no" active="no"/>
+<layer number="6" name="Route6" color="1" fill="8" visible="no" active="no"/>
+<layer number="7" name="Route7" color="4" fill="8" visible="no" active="no"/>
+<layer number="8" name="Route8" color="1" fill="2" visible="no" active="no"/>
+<layer number="9" name="Route9" color="4" fill="2" visible="no" active="no"/>
+<layer number="10" name="Route10" color="1" fill="7" visible="no" active="no"/>
+<layer number="11" name="Route11" color="4" fill="7" visible="no" active="no"/>
+<layer number="12" name="Route12" color="1" fill="5" visible="no" active="no"/>
+<layer number="13" name="Route13" color="4" fill="5" visible="no" active="no"/>
+<layer number="14" name="Route14" color="1" fill="6" visible="no" active="no"/>
+<layer number="15" name="Route15" color="4" fill="6" visible="no" active="no"/>
+<layer number="16" name="Bottom" color="1" fill="1" visible="no" active="no"/>
+<layer number="17" name="Pads" color="2" fill="1" visible="no" active="no"/>
+<layer number="18" name="Vias" color="2" fill="1" visible="no" active="no"/>
+<layer number="19" name="Unrouted" color="6" fill="1" visible="no" active="no"/>
+<layer number="20" name="Dimension" color="14" fill="1" visible="no" active="no"/>
+<layer number="21" name="tPlace" color="7" fill="1" visible="no" active="no"/>
+<layer number="22" name="bPlace" color="7" fill="1" visible="no" active="no"/>
+<layer number="23" name="tOrigins" color="15" fill="1" visible="no" active="no"/>
+<layer number="24" name="bOrigins" color="15" fill="1" visible="no" active="no"/>
+<layer number="25" name="tNames" color="7" fill="1" visible="no" active="no"/>
+<layer number="26" name="bNames" color="7" fill="1" visible="no" active="no"/>
+<layer number="27" name="tValues" color="7" fill="1" visible="no" active="no"/>
+<layer number="28" name="bValues" color="7" fill="1" visible="no" active="no"/>
 <layer number="29" name="tStop" color="7" fill="3" visible="no" active="no"/>
 <layer number="30" name="bStop" color="7" fill="6" visible="no" active="no"/>
@@
 <layer number="35" name="tGlue" color="7" fill="4" visible="no" active="no"/>
 <layer number="36" name="bGlue" color="7" fill="5" visible="no" active="no"/>
-<layer number="37" name="tTest" color="7" fill="1" visible="yes" active="no"/>
-<layer number="38" name="bTest" color="7" fill="1" visible="yes" active="no"/>
+<layer number="37" name="tTest" color="7" fill="1" visible="no" active="no"/>
+<layer number="38" name="bTest" color="7" fill="1" visible="no" active="no"/>
 <layer number="39" name="tKeepout" color="4" fill="11" visible="no" active="no"/>
 <layer number="40" name="bKeepout" color="1" fill="11" visible="no" active="no"/>
@@
 <layer number="44" name="Drills" color="7" fill="1" visible="no" active="no"/>
 <layer number="45" name="Holes" color="7" fill="1" visible="no" active="no"/>
-<layer number="46" name="Milling" color="3" fill="1" visible="yes" active="no"/>
-<layer number="47" name="Measures" color="7" fill="1" visible="yes" active="no"/>
-<layer number="48" name="Document" color="7" fill="1" visible="yes" active="no"/>
-<layer number="49" name="Reference" color="7" fill="1" visible="yes" active="no"/>
-<layer number="50" name="dxf" color="7" fill="1" visible="yes" active="no"/>
-<layer number="51" name="tDocu" color="7" fill="1" visible="yes" active="no"/>
-<layer number="52" name="bDocu" color="7" fill="1" visible="yes" active="no"/>
-<layer number="53" name="tGND_GNDA" color="7" fill="9" visible="yes" active="no"/>
-<layer number="54" name="bGND_GNDA" color="1" fill="9" visible="yes" active="no"/>
-<layer number="56" name="wert" color="7" fill="1" visible="yes" active="no"/>
-<layer number="57" name="tCAD" color="7" fill="1" visible="yes" active="no"/>
-<layer number="59" name="tCarbon" color="7" fill="1" visible="yes" active="no"/>
-<layer number="60" name="bCarbon" color="7" fill="1" visible="yes" active="no"/>
+<layer number="46" name="Milling" color="3" fill="1" visible="no" active="no"/>
+<layer number="47" name="Measures" color="7" fill="1" visible="no" active="no"/>
+<layer number="48" name="Document" color="7" fill="1" visible="no" active="no"/>
+<layer number="49" name="Reference" color="7" fill="1" visible="no" active="no"/>
+<layer number="50" name="dxf" color="7" fill="1" visible="no" active="no"/>
+<layer number="51" name="tDocu" color="7" fill="1" visible="no" active="no"/>
+<layer number="52" name="bDocu" color="7" fill="1" visible="no" active="no"/>
+<layer number="53" name="tGND_GNDA" color="7" fill="9" visible="no" active="no"/>
+<layer number="54" name="bGND_GNDA" color="1" fill="9" visible="no" active="no"/>
+<layer number="56" name="wert" color="7" fill="1" visible="no" active="no"/>
+<layer number="57" name="tCAD" color="7" fill="1" visible="no" active="no"/>
+<layer number="59" name="tCarbon" color="7" fill="1" visible="no" active="no"/>
+<layer number="60" name="bCarbon" color="7" fill="1" visible="no" active="no"/>
 <layer number="88" name="SimResults" color="9" fill="1" visible="yes" active="yes"/>
 <layer number="89" name="SimProbes" color="9" fill="1" visible="yes" active="yes"/>
@@
 <part name="SUPPLY5" library="Power_Symbols" library_urn="urn:adsk.eagle:library:16502351" deviceset="GND-BAR" device="" value="GND"/>
 <part name="IC2" library="74HCT1G32GW - OR Gate" deviceset="74HCT1G32GW" device="-DC" value="74HCT1G32GW"/>
-<part name="R1" library="rcl" deviceset="R-EU_" device="R0402" value="10k"/>
-<part name="SUPPLY1" library="Power_Symbols" library_urn="urn:adsk.eagle:library:16502351" deviceset="3V3-CIRCLE" device="" value="3V3"/>
 <part name="SUPPLY6" library="Power_Symbols" library_urn="urn:adsk.eagle:library:16502351" deviceset="3V3-CIRCLE" device="" value="3V3"/>
 <part name="SUPPLY7" library="Power_Symbols" library_urn="urn:adsk.eagle:library:16502351" deviceset="GND-BAR" device="" value="GND"/>
@@
 <attribute name="VALUE" x="116.84" y="96.52" size="1.778" layer="96"/>
 </instance>
-<instance part="R1" gate="G$1" x="35.56" y="22.86" smashed="yes" rot="R90">
-<attribute name="NAME" x="38.1" y="22.86" size="1.778" layer="95"/>
-<attribute name="VALUE" x="38.1" y="20.32" size="1.778" layer="96"/>
-</instance>
-<instance part="SUPPLY1" gate="G$1" x="35.56" y="35.56" smashed="yes">
-<attribute name="VALUE" x="35.56" y="40.64" size="1.778" layer="96" rot="R180" align="center"/>
-</instance>
 <instance part="SUPPLY6" gate="G$1" x="58.42" y="27.94" smashed="yes">
 <attribute name="VALUE" x="58.42" y="33.02" size="1.778" layer="96" rot="R180" align="center"/>
@@
 <pinref part="IC1" gate="G$1" pin="!CS!"/>
 <pinref part="IC2" gate="G$1" pin="A"/>
-</segment>
-<segment>
-<pinref part="R1" gate="G$1" pin="1"/>
-<wire x1="35.56" y1="17.78" x2="35.56" y2="12.7" width="0.1524" layer="91"/>
-<label x="35.56" y="12.7" size="1.778" layer="95" rot="R180"/>
 </segment>
 </net>
@@
 </segment>
 <segment>
-<pinref part="R1" gate="G$1" pin="2"/>
-<wire x1="35.56" y1="27.94" x2="35.56" y2="33.02" width="0.1524" layer="91"/>
-<pinref part="SUPPLY1" gate="G$1" pin="3V3"/>
-</segment>
-<segment>

Commit message: in brd & sch: - added FeRAM module
- created and tested fm25w256 driver
Parts:
- removed C22: 0.1µF, rcl:C-EUC0805
- removed IC6: FM25W256-SOIC, FM25W256 FERAM:FM25W256-SOIC
- removed R18: 10k, rcl:R-EU_R0805
Connections:
- removed net SPI_FRAM_CS: BRD1CN10.PA6
- new net FRAM_!HOLD!: IC1.!HOLD!
- new net FRAM_!WP!: IC1.!WP!
- new net SPI1_FRAM_CS: BRD1CN10.PA6, IC1.!CS!
- net 3V3: now also IC1.VCC
- net GND: no longer C22.2, IC6.GND
- net SPI1_MISO: now also IC1.SO
- net SPI1_MOSI: now also IC1.SI
- net SPI1_SCK: now also IC1.SCK
- net SPI_MISO_PIN: no longer IC6.SO
- net SPI_MOSI_PIN: no longer IC6.SI
- net SPI_SCK_PIN: no longer IC6.SCK
- net SPI_SS_FRAM_PIN: no longer IC6.!CS!, R18.1
- net VCC: no longer C22.1, IC6.!HOLD!, IC6.!WP!, IC6.VCC, R18.2
Other:
- moved on the sheet: BRD1CN10, BRD1CN7

Commit message: in sch & brd: - updated SD card module library - added SD card module to sch
- added ST's FileX middleware
- added sd.c/.h skeleton
Parts:
- removed C31: 0.1µF, rcl:C-EUC0805
- removed IC7: MICROSD_SPI_MODE, Molex SD-47309 SD Card Slot:MICROSD_SPI_MODE
- removed R37: 10k, rcl:R-EU_R0805
Connections:
- removed net PA1: BRD1CN7.PA1
- removed net PB0: BRD1CN7.PB0
- new net SD_CD: BRD1CN7.PB0, IC1.POL
- new net SPI1_SD_CS: BRD1CN7.PA1, IC1.CD/DAT3
- net 3V3: now also IC1.DET, IC1.VDD
- net GND: now also IC1.VSS; no longer C31.2, IC7.GND1, IC7.GND2, IC7.GND3, IC7.GND4
- net SD_CARD_DETECT_PIN: no longer IC7.CARD_DETECT
- net SPI1_MISO: now also IC1.DAT0
- net SPI1_MOSI: now also IC1.CMD
- net SPI1_SCK: now also IC1.CLK
- net SPI_MISO_PIN: no longer IC7.DO
- net SPI_MOSI_PIN: no longer IC7.DI
- net SPI_SCK_PIN: no longer IC7.CLK
- net SPI_SS_SD_CARD_PIN: no longer IC7.CS, R37.1
- net VCC: no longer C31.1, IC7.VCC, R37.2
