File: eagle design/misko_nucleo.sch (EAGLE design)
At the start: 125 parts, among them CN1 LiPo Battery, IC1 MC1525TT, IC10 LTC4425, IC11 SP3012-04UTG, IC2 ORG1510-MK4, IC3 TPS63031, IC4 FT230XS, IC5 RN4678_BT_MODULE, IC8 DS1394U-33+, IC9 MAX6818, Q1 ABM3B-8MHZ-10-1-U-T, Q2 BSS84, Q3 LFXTAL016178R, SW1 MICROJOYSTICK, SW2 PB6156RSL, SW3 PB6156RSL, U1 SN74LVC1G3157DBVR - BT switch, U2 ATMEGA1281-16AU, U3 TPS3808G33DBVT, U4 TMP36GRTZ, U5 MCP73871-2AAI/ML, U6 SN74LVC1G3157DBVR - GPS switch, X1 FH12-30S-0.5SH

Commit message: - moved gps components into misko nucleo schematic - corrected component library issues
Parts:
- removed C28, C38: 0.1µF, rcl:C-EUC0805
- removed C29: 10µF, rcl:C-EUC0805
- removed C30, C33: 1000µF, rcl:CPOL-EUE5-10.5
- removed C32: 10µF, resistor:C-EUC0805
- removed C34, C35: 100µF, rcl:C-EUC0805
- removed C36, C37: 0.1µF, resistor:C-EUC0805
- removed IC10: LTC4425, LTC4425 Supercap Charger:LTC4425
- removed IC11: SP3012-04UTG, SP3012 TVS Diode Array:SP3012-04UTG
- removed IC8: DS1394U-33+, DS1394U-33+ RTC SPI Module:DS1394U-33+
- removed IC9: MAX6818, MAX6818 CMOS Switch debouncer:MAX6818
- removed R34: 100k, rcl:R-EU_R0805
- removed R35: 270k, rcl:R-EU_R0805
- removed R36: NTC 10k, rcl:R-EU_0204/5
- removed R38, R39: 150k, rcl:R-EU_R0805
- removed R40, R41: 470k, resistor:R-EU_R0805
- removed U6: SN74LVC1G3157DBVR - GPS switch, Texas Instruments_By_element14_Batch_1:SN74LVC1G3157DBVR
- added C22: 10µF, rcl:C-EUC0805
- added IC6: MAX6818, MAX6818 CMOS Switch debouncer:MAX6818
- added IC7: SP3012-04UTG, SP3012 TVS Diode Array:SP3012-04UTG
- added R18: 1k, resistor:R-EU_R0805
- C1: value 18pF -> 0.1µF; device rcl:C-EUC0805 -> resistor:C-EUC0805
- C10: value 1µF -> 0.1µF; device rcl:C-EUC0805 -> resistor:C-EUC0805
- C11: value 22µF -> 1µF
- C12: value 7pF -> 1µF; device resistor:C-EUC0805 -> rcl:C-EUC0805
- C13, C3: value 0.1µF -> 10µF; device resistor:C-EUC0805 -> rcl:C-EUC0805
- C14: value 1µF -> 2.2µF / 25V
- C15, C2: value 1µF -> 10µF
- C16: value 10µF -> 0.1µF; device rcl:C-EUC0805 -> resistor:C-EUC0805
- C17: value 2.2µF / 25V -> 10µF; device rcl:C-EUC0805 -> resistor:C-EUC0805
- C18: value 1nF -> 1000µF; device rcl:C-EUC0805 -> rcl:CPOL-EUE5-10.5
- C19: value 10µF -> 1000µF; device rcl:C-EUC0805 -> rcl:CPOL-EUE5-10.5
- C20: value 0.1µF -> 1000µF; device rcl:C-EUC0805 -> rcl:CPOL-EUE5-10.5
- C21: device resistor:C-EUC0805 -> rcl:C-EUC0805
- C23: value 10µF -> 1000µF; device resistor:C-EUC0805 -> rcl:CPOL-EUE5-10.5
- C24: value 1.5F -> 10µF; device EECS5R5H155 Supercap:EECS5R5H155 -> resistor:C-EUC0805
- C26, C27: value 1000µF -> 0.1µF; device rcl:CPOL-EUE5-10.5 -> resistor:C-EUC0805
- C4: value 10µF -> 0.1µF; device resistor:C-EUC0805 -> rcl:C-EUC0805
- C5: value 10µF -> 7pF; device rcl:C-EUC0805 -> resistor:C-EUC0805
- C6: value 0.1µF -> 1µF
- C7: value 18pF -> 1µF; device resistor:C-EUC0805 -> rcl:C-EUC0805
- C8: value 7pF -> 22µF; device resistor:C-EUC0805 -> rcl:C-EUC0805
- C9: value 1µF -> 7pF; device rcl:C-EUC0805 -> resistor:C-EUC0805
- IC2: value ORG1510-MK4 -> TPS63031; device ORG1510-MK4 GPS module:ORG1510-MK4 -> TPS63031 - Buck Boost Voltage Regulator:TPS63001DRCR
- IC3: value TPS63031 -> FT230XS; device TPS63031 - Buck Boost Voltage Regulator:TPS63001DRCR -> ftdichip:FT230XS
- IC4: value FT230XS -> RN4678_BT_MODULE; device ftdichip:FT230XS -> RN4678 Bluetooth 4.2 Dual Mode:RN4678_BT_MODULE
- IC5: value RN4678_BT_MODULE -> DS1394U-33+; device RN4678 Bluetooth 4.2 Dual Mode:RN4678_BT_MODULE -> DS1394U-33+ RTC SPI Module:DS1394U-33+
- R14: value 10k -> 47k; device resistor:R-EU_R0805 -> rcl:R-EU_R0805
- R15: value 47k -> 1k
- R17: value 1k -> 47k
- R20: value 1k -> 390k; device resistor:R-EU_R0805 -> rcl:R-EU_R0805
- R21: value 47k -> 10k; device rcl:R-EU_R0805 -> resistor:R-EU_R0805
- R22: value 390k -> 10k; device rcl:R-EU_R0805 -> resistor:R-EU_R0805
- R23: value 10k -> 1k
- R25: value 1k -> 10k
- R26: value 1M -> 10k; device resistor:R-EU_R0805 -> rcl:R-EU_R0805
- R27, R28: value 10k -> 1k; device resistor:R-EU_R0805 -> rcl:R-EU_R0805
- R29: value 10k -> 100k
- R30: value 1k -> 270k
- R31: value 1k -> NTC 10k; device rcl:R-EU_R0805 -> rcl:R-EU_0204/5
- R32: value 1k -> 150k; device resistor:R-EU_R0805 -> rcl:R-EU_R0805
- R33: value 10k -> 150k; device resistor:R-EU_R0805 -> rcl:R-EU_R0805
- U3: value TPS3808G33DBVT -> TMP36GRTZ; device Texas Instruments_By_element14_Batch_1:TPS3808G33DBVT -> TMP36GRTZ:TMP36GRTZ-REEL7
- U4: value TMP36GRTZ -> MCP73871-2AAI/ML; device TMP36GRTZ:TMP36GRTZ-REEL7 -> MCP73871 - Powerpath and Charge Controller:MCP73871-2AAI/ML
- U5: value MCP73871-2AAI/ML -> SN74LVC1G3157DBVR - GPS switch; device MCP73871 - Powerpath and Charge Controller:MCP73871-2AAI/ML -> Texas Instruments_By_element14_Batch_1:SN74LVC1G3157DBVR
Connections:
- removed net LTC4425_EN: IC10.EN, R32.2
- removed net LTC4425_PROG: IC10.PROG, R33.2
- removed net UART1_RX: BRD1CN10.PB15
- removed net UART1_TX: BRD1CN10.PB14
- new net PROG: IC2.PROG, R14.2
- net 3V3: now also C2.1, C22.1, IC2.FB, IC2.SEL, IC2.VDD, IC2.VIN, R18.1, R18.2
- net ANALOG_SW_CTRL_PIN: now also U5.S; no longer U6.S
- net AREF: now also C2.1; no longer C4.1
- net AVCC: now also C26.2; no longer C36.2
- net BAT_A_PIN: now also R32.2, R33.1; no longer R38.2, R39.1
- net BLUETOOTH_PROF_IND_PIN: now also IC4.P0_5; no longer IC5.P0_5
- net BLUETOOTH_RX: now also IC4.RXD; no longer IC5.RXD
- net BLUETOOTH_SWITCH_PIN: now also IC4.SW_BTN, R25.2; no longer IC5.SW_BTN, R28.2
- net BLUETOOTH_TX: now also IC4.TXD, U5.B1; no longer IC5.TXD, U6.B1
- net BLUETOOTH_WAKEUP_PIN: now also IC4.WAKEUP, R24.2; no longer IC5.WAKEUP, R27.2
- net BT_LED: now also IC4.LED, R18.1; no longer IC5.LED, R20.1
- net BUTTON_BLUETOOTH: now also IC6.IN7; no longer IC9.IN7
- net BUTTON_CENTER: now also IC6.IN5; no longer IC9.IN5
- net BUTTON_DOWN: now also IC6.IN2; no longer IC9.IN2
- net BUTTON_GPRS: now also IC6.IN8; no longer IC9.IN8
- net BUTTON_LEFT: now also IC6.IN4; no longer IC9.IN4
- net BUTTON_RIGHT: now also IC6.IN3; no longer IC9.IN3
- net BUTTON_UP: now also IC6.IN6; no longer IC9.IN6
- net CAP1N: now also C6.1; no longer C9.1
- net CAP1P: now also C6.2; no longer C9.2
- net CAP2N: now also C7.1; no longer C10.1
- net CAP2P: now also C7.2; no longer C10.2
- net CBUS1: now also IC3.CBUS1; no longer IC4.CBUS1
- net CBUS2: now also IC3.CBUS2; no longer IC4.CBUS2
- net D+: now also IC7.4; no longer IC11.4
- net D-: now also IC7.2; no longer IC11.2
- net EN: now also IC2.EN, R18.2; no longer IC3.EN
- net GND: now also C1.1, C10.2, C13.1, C15.2, C16.2, C17.2, C18.-, C19.-, C20.-, C22.2, C23.-, C24.2, C26.1, C27.1, C9.1, IC2.5_GND, IC2.PGND, IC2.POWERPAD, IC3.GND@1, IC6.!EN!, IC6.GND, IC7.GND, R14.1, R20.1, R21.2, R24.1, R25.1, R28.2, R29.2, R30.2, R33.2, U4.GND1, U4.GND2, U4.GND3, U4.GND4, U4.GND5, U4.GND6, U5.GND; no longer C13.2, C15.1, C16.1, C17.1, C18.2, C19.2, C20.1, C23.2, C26.-, C27.-, C28.2, C29.2, C30.-, C32.2, C33.-, C35.1, C36.1, C37.1, C38.1, C6.2, C7.1, IC10.GND1, IC10.GND2, IC10.GND3, IC11.GND, IC3.PGND, IC3.POWERPAD, IC4.GND@1, IC8.GND, IC9.!EN!, IC9.GND, R14.2, R22.1, R23.2, R27.1, R28.1, R33.1, R34.2, R35.2, R36.2, R39.2, U4.GND, U5.GND1, U5.GND2, U5.GND3, U5.GND4, U5.GND5, U5.GND6, U6.GND
- net GPRS_NETLIGHT: now also R21.1, R22.1; no longer R23.1, R24.1
- net GPRS_NETLIGHT_GATE: now also R22.2; no longer R24.2
- net GPS_GREEN_LED_PIN: now also R15.1; no longer R16.1
- net GPS_ON_OFF: now also IC2.!RESET!, IC2.1_ON_OFF, R18.1; no longer IC2.ON_OFF, R26.1, U3.~RESET
- net GPS_POWER_CTL_PIN: now also IC2.!MR!; no longer R14.1, U3.~MR
- net GPS_RED_LED_PIN: now also R16.1; no longer R17.1
- net GPS_SW_SERIAL_RX: now also U5.A; no longer U6.A
- net GPS_SW_SERIAL_TX: now also BRD1CN10.PB14, IC2.RX_10; no longer C7.2, IC2.RX
- net GPS_TX: now also BRD1CN10.PB15, C22.1, IC2.3_TX, U5.B2; no longer C1.1, IC2.TX, U6.B2
- net GPS_WAKEUP_PIN: now also IC2.WAKEUP_6; no longer IC2.WAKEUP
- net GREEN_LED: now also R15.2; no longer R16.2
- net ID: now also IC7.5; no longer IC11.5
- net IREF: now also R20.2; no longer R22.2
- net L2: now also R18.2; no longer R20.2
- net LDO33_O: now also IC4.LDO33_O, IC4.VDD_IO; no longer IC5.LDO33_O, IC5.VDD_IO
- net L_L1: now also IC2.L1; no longer IC3.L1
- net L_L2: now also IC2.L2; no longer IC3.L2
- net MCP73871_CHARGE_STATUS_1_PIN: now also R19.2, U4.STAT1/!LBO!; no longer R21.2, U5.STAT1/!LBO!
- net MCP73871_CHARGE_STATUS_2_PIN: now also R17.2, U4.STAT2; no longer R19.2, U5.STAT2
- net MCP73871_POWER_GOOD_PIN: now also R14.2, U4.!PG!; no longer R15.2, U5.!PG!
- net MENU_BLUETOOTH_POWER_BUTTON_PIN: now also IC6.OUT7; no longer IC9.OUT7
- net MENU_CENTER_BUTTON_PIN: now also IC6.OUT5; no longer IC9.OUT5
- net MENU_DOWN_BUTTON_PIN: now also IC6.OUT2; no longer IC9.OUT2
- net MENU_GPRS_POWER_BUTTON_PIN: now also IC6.OUT8; no longer IC9.OUT8
- net MENU_LEFT_BUTTON_PIN: now also IC6.OUT4; no longer IC9.OUT4
- net MENU_RIGHT_BUTTON_PIN: now also IC6.OUT3; no longer IC9.OUT3
- net MENU_UP_BUTTON_PIN: now also IC6.OUT6; no longer IC9.OUT6
- net N$1: now also R23.1; no longer R25.1
- net N$10: now also C10.1, IC3.!RESET, IC3.3V3OUT, IC3.VCCIO; no longer C13.1, IC4.!RESET, IC4.3V3OUT, IC4.VCCIO
- net N$11: now also IC4.!RST_N!; no longer IC5.!RST_N!
- net N$19: now also R27.2, R30.1, R31.1; no longer R30.2, R35.1, R36.1
- net N$3: now also R23.2; no longer R25.2
- net N$31: now also C1.2; no longer C3.2
- net N$4: now also IC7.1; no longer IC11.1
- net N$6: now also C18.+, C19.+, C20.+, C23.+; no longer C26.+, C27.+, C30.+, C33.+
- net OLD_5V0: now also C27.2, IC3.VCC, IC7.10, U4.!TE!, U4.CE, U4.IN1, U4.IN2, U4.PROG2, U4.SEL; no longer C37.2, IC11.10, IC4.VCC, U5.!TE!, U5.CE, U5.IN1, U5.IN2, U5.PROG2, U5.SEL
- net PDI_UART0_CTS_PIN: now also IC3.!CTS; no longer IC4.!CTS
- net PFI: now also IC2.PFI; no longer IC10.PFI, R40.1, R41.2
- net PFI_RET: now also IC2.PFI_RET; no longer IC10.PFI_RET, R41.1
- net PROG1: now also R28.1, U4.PROG1; no longer R31.1, U5.PROG1
- net PROG3: now also R29.1, U4.PROG3; no longer R34.1, U5.PROG3
- net RED_LED: now also R16.2; no longer R17.2
- net RTC_INT_INTERRUPT_PIN: now also IC5.!INT!; no longer IC8.!INT!
- net RTC_XTAL1: now also IC5.X1; no longer IC8.X1
- net RTC_XTAL2: now also IC5.X2; no longer IC8.X2
- net RXD: now also IC3.RXD; no longer IC4.RXD
- net SPI_MISO_PIN: now also IC5.DOUT; no longer IC8.DOUT
- net SPI_MOSI_PIN: now also IC5.DIN; no longer IC8.DIN
- net SPI_SCK_PIN: now also IC5.SCLK; no longer IC8.SCLK
- net SPI_SS_RTC_PIN: now also IC5.!CS!, R26.2; no longer IC8.!CS!, R29.2
- net THERM: now also R27.1, U4.THERM; no longer R30.1, U5.THERM
- net TMP36_VSENSE_PIN: now also U3.VOUT; no longer U4.VOUT
- net TXD: now also IC3.TXD; no longer IC4.TXD
- net USBDM: now also IC3.USBDM; no longer IC4.USBDM
- net USBDP: now also IC3.USBDP; no longer IC4.USBDP
- net USB_D+: now also IC7.7; no longer IC11.7
- net USB_D-: now also IC7.9; no longer IC11.9
- net USB_ID: now also IC7.6; no longer IC11.6
- net VCC: now also C12.2, C13.2, C15.1, C16.1, C22.1, C8.2, IC2.FB, IC2.VOUT, IC4.BAT_IN, IC5.VCC, IC6.VCC, R14.1, R17.1, R26.1, U3.+VS, U3.~SHDN, U5.VCC; no longer C14.2, C15.2, C16.2, C19.1, C20.2, C28.1, C29.1, C38.2, IC10.FB, IC10.SEL, IC10.VCC1, IC10.VCC2, IC3.FB, IC3.VOUT, IC5.BAT_IN, IC8.VCC, IC9.VCC, R15.1, R21.1, R26.2, R29.1, R32.1, R40.2, U3.VDD, U4.+VS, U4.~SHDN, U6.VCC
- net VCOMH: now also C14.2; no longer C17.2
- net VGPS: now also C1.1, IC2.4_VCC, IC2.SENSE, IC2.VOUT, IC5.VBACK; no longer C18.1, C34.1, IC10.VOUT1, IC10.VOUT2, IC2.VCC, IC8.VBACK, U3.SENSE
- net VMID: now also C1.1, IC2.VMID; no longer C34.2, C35.2, IC10.VMID
- net VPCC: now also U4.VPCC; no longer U5.VPCC
- net V_LIION+: now also C24.1, R32.1, U4.VBAT1, U4.VBAT2, U4.VBAT_SENSE; no longer C32.1, R38.1, U5.VBAT1, U5.VBAT2, U5.VBAT_SENSE
- net V_LIION_REGULATED: now also C17.1, C3.2, C4.1, IC2.PS/SYNC, IC2.VIN, IC2.VINA, U4.OUT1, U4.OUT2; no longer C23.1, C5.2, C6.1, IC3.PS/SYNC, IC3.VIN, IC3.VINA, U5.OUT1, U5.OUT2
- net XTAL1: now also C9.2; no longer C12.2
- net XTAL2: now also C5.2; no longer C8.2
Other:
- moved on the sheet: C1, C10, C11, C12, C13, C14, C15, C16, C17, C2, C21, C25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

Commit message: - corrected net names in modules
Connections:
- removed net GPS_ON_OFF: IC2.!RESET!, IC2.1_ON_OFF, R18.1
- new net !MR!: IC2.!MR!
- new net !RESET!: IC2.!RESET!, R18.1
- new net FORCE-ON: IC2.1_FORCE-ON
- new net RX: IC2.RX_10
- new net SENSE: C1.1, IC2.SENSE
- new net TX: C22.1, IC2.3_TX
- new net VOUT: C24.+, IC2.VOUT
- new net WAKEUP: IC2.WAKEUP_6
- net GPS_POWER_CTL_PIN: no longer IC2.!MR!
- net GPS_SW_SERIAL_TX: no longer IC2.RX_10
- net GPS_TX: no longer C22.1, IC2.3_TX
- net GPS_WAKEUP_PIN: no longer IC2.WAKEUP_6
- net VGPS: no longer C1.1, C24.+, IC2.SENSE, IC2.VOUT

Commit message: - removed not needed components (crystal, voltage reference, etc.) from original schematic
Parts:
- removed C1, C16, C26: 0.1µF, resistor:C-EUC0805
- removed C19, C20, C23, C25: 1000µF, rcl:CPOL-EUE5-10.5
- removed C2: 10µF, resistor:C-EUC0805
- removed C5, C9: 7pF, resistor:C-EUC0805
- removed CONN2: JTAG, JTAG 1.27mm 10pin header:JTAG-1.27-10-PIN-HEADER
- removed D1: 1N4148, Diode2:1N4148
- removed IC1: MC1525TT, microchip:MC1525TT
- removed JP1: I2C, jumper:JP4E
- removed L2: DL0805-33 33µH, rcl:L-US
- removed Q1: ABM3B-8MHZ-10-1-U-T, ABM3B-8MHZ-10-1-U-T - Quartz Resonator:ABM3B
- removed R1: 47k, rcl:R-EU_R0805
- removed R3: 4k7, rcl:R-EU_R0805
- removed R7, R8: 150k, rcl:R-EU_R0805
- removed S1: RESET, Wurth_Elektronik_Electromechanic_Switch_rev17c:430152050836
- removed TP1, TP2, TP3: GND, testpad:TPPAD1-17Y
- removed TP11: Bluetooth Wakeup Pin, testpad:PTR1TP14R
- removed TP4: VCC, testpad:PTR1TP14R
- removed TP5: VLiIon Regulated, testpad:PTR1TP14R
- removed TP6: VGPS, testpad:PTR1TP14R
- removed TP7: Analogue Switch CRTL Pin, testpad:PTR1TP14R
- removed TP8: GPS Power CTRL Pin, testpad:PTR1B1,27
- removed U3: TMP36GRTZ, TMP36GRTZ:TMP36GRTZ-REEL7
Connections:
- removed net ADXL345_INT2: IC1.INT2
- removed net FRAM_!HOLD!: IC1.!HOLD!
- removed net FRAM_!WP!: IC1.!WP!
- removed net N$31: C1.2, D1.A, R1.1
- net 3V3: no longer C2.1, IC1.DET, IC1.VCC, IC1.VDD, IC1.VDDIO, IC1.VS
- net ADXL345SDA: no longer IC1.SDA
- net ADXL345_CS: no longer IC1.!CS!
- net ADXL345_INT1: no longer IC1.INT1
- net ADXL345_INT1_INTERRUPT_PIN: no longer JP1.3
- net ANALOG_SW_CTRL_PIN: no longer TP7.TP
- net AREF: no longer C2.1, IC1.VO
- net AVCC: no longer C26.2, IC1.VIN, L2.2
- net BLUETOOTH_PROF_IND_PIN: no longer TP11.TP
- net GND: no longer C1.1, C1.2, C16.2, C19.-, C2.2, C20.-, C23.-, C25.-, C26.1, C5.1, C9.1, CONN2.GND1, CONN2.GND2, IC1.GND, IC1.VSS, JP1.1, Q1.GND1, Q1.GND2, R8.2, S1.1, S1.3, TP1.TP, U3.GND
- net GPS_POWER_CTL_PIN: no longer TP8.TP
- net JTAG_TCL_PIN: no longer CONN2.TCK
- net JTAG_TDI_PIN: no longer CONN2.TDI
- net JTAG_TDO_PIN: no longer CONN2.TDO
- net JTAG_TMS_PIN: no longer CONN2.TMS
- net N$6: no longer C19.+, C20.+, C23.+, C25.+
- net RESET: no longer CONN2.RESET, R1.2, R3.2, S1.2, S1.4
- net RTC_INT_INTERRUPT_PIN: no longer JP1.4
- net SD_CD: no longer IC1.POL
- net SENSE: no longer C1.1
- net SPI1_FRAM_CS: no longer IC1.!CS!
- net SPI1_MISO: no longer IC1.DAT0, IC1.SDO, IC1.SO
- net SPI1_MOSI: no longer IC1.CMD, IC1.SI
- net SPI1_SCK: no longer IC1.CLK, IC1.SCK, IC1.SCL
- net SPI1_SD_CS: no longer IC1.CD/DAT3
- net TMP36_VSENSE_PIN: no longer U3.VOUT
- net VCC: no longer C16.1, CONN2.VCC, D1.C, JP1.2, L2.1, R3.1, R7.1, TP3.TP, TP4.TP, U3.+VS, U3.~SHDN
- net VCC_SENSE_PIN: no longer R7.2, R8.1
- net VGPS: no longer C2.1, TP6.TP
- net VMID: no longer C1.1
- net VUSB: no longer TP2.TP
- net V_LIION_REGULATED: no longer TP5.TP
- net XTAL1: no longer C9.2, Q1.Q2
- net XTAL2: no longer C5.2, Q1.Q1
Other:
- note removed: "AVCC Circuit"
- note removed: "Oscillator Circuit"

Commit message: - added/coded and routed ORG1510-MK4 GPS module reset and LTC4425 SuperCap Charger enable pins
Connections:
- net PB6 renamed GPS_!RESET!
- net PB7 renamed SUPERCAP_!EN!
- removed net FORCE-ON: IC2.1_FORCE-ON
- removed net RX: IC2.RX_10
- removed net WAKEUP: IC2.WAKEUP_6
- new net !EN!: IC2.EN
- net 3V3: no longer R18.1
- net EN: no longer R18.2
- net GND: no longer IC2.5_GND
- net TX: no longer IC2.3_TX
- net VGPS: no longer IC2.4_VCC

Commit message: - updated ORG1510 library - added low pass filter to GPS module UART pins
Connections:
- removed net TX: C22.1
- new net CT: IC2.CT
- new net GPS_RX: R2.2
- new net RX: R2.1
- net GPS_TX: now also C22.1
Other:
- note added: "50ms delay DS. p. 11"
- note added: "low-pass 3dB cutoff: 146.1478 MHz"

Commit message: - removed RTC IC
Parts:
- removed C21: 0.1µF, rcl:C-EUC0805
- removed IC5: DS1394U-33+, DS1394U-33+ RTC SPI Module:DS1394U-33+
- removed Q3: LFXTAL016178R, LFXTAL016178R 32.768kHz crystal:LFXTAL016178R
- removed R26: 10k, rcl:R-EU_R0805
Connections:
- net GPS_SW_SERIAL_TX renamed GPS_MCU_RX
- removed net RTC_XTAL1: IC5.X1, Q3.XTAL1
- removed net RTC_XTAL2: IC5.X2, Q3.XTAL2
- removed net VGPS: IC5.VBACK
- new net GPS_MCU_TX: BRD1CN10.PB15, U5.B2
- net 3V3: no longer C22.1
- net GND: no longer C21.2, IC5.GND
- net GPS_TX: no longer BRD1CN10.PB15, U5.B2
- net RTC_INT_INTERRUPT_PIN: no longer IC5.!INT!
- net SPI_MISO_PIN: no longer IC5.DOUT
- net SPI_MOSI_PIN: no longer IC5.DIN
- net SPI_SCK_PIN: no longer IC5.SCLK
- net SPI_SS_RTC_PIN: no longer IC5.!CS!, R26.2
- net VCC: no longer C21.1, IC5.VCC, R26.1
Other:
- note added: "Ct open 50ms delay DS. p. 11"
- note removed: "50ms delay DS. p. 11"

Commit message: in misko.ioc/main.c/.h & sch/brd: - added yellow LED, defined GPIO, placed components roughly on brd
Parts:
- removed C15, C22: 10µF, rcl:C-EUC0805
- removed C17, C24: 10µF, resistor:C-EUC0805
- removed C18: 1000µF, rcl:CPOL-EUE5-10.5
- removed C27: 0.1µF, resistor:C-EUC0805
- removed CONN1: USB mini B, MX-67503-1230 USB Mini-B SMT straight socket:MX-67503-1230
- removed D4: BAT60AE6327, diode:BAT60J
- removed F1: PTS120615V050, SparkFun-Fuses:PPTC_THREE-QUARTER-AMP
- removed IC4: RN4678_BT_MODULE, RN4678 Bluetooth 4.2 Dual Mode:RN4678_BT_MODULE
- removed IC6: MAX6818, MAX6818 CMOS Switch debouncer:MAX6818
- removed IC7: SP3012-04UTG, SP3012 TVS Diode Array:SP3012-04UTG
- removed LED1: TX, led:LEDCHIPLED_1206
- removed LED2: RX, led:LEDCHIPLED_1206
- removed LED3: green, led:LEDSQR2X5
- removed LED4: red, led:LEDSQR2X5
- removed Q2: BSS84, transistor-small-signal:BSS84
- removed R21, R22, R24, R25: 10k, resistor:R-EU_R0805
- removed R23: 1k, resistor:R-EU_R0805
- removed R27, R28: 1k, rcl:R-EU_R0805
- removed R29: 100k, rcl:R-EU_R0805
- removed R30: 270k, rcl:R-EU_R0805
- removed R31: NTC 10k, rcl:R-EU_0204/5
- removed R32, R33: 150k, rcl:R-EU_R0805
- removed S2: POWER SWITCH, smd-special:SWS001
- removed U5: SN74LVC1G3157DBVR - GPS switch, Texas Instruments_By_element14_Batch_1:SN74LVC1G3157DBVR
- added C1: 10µF, rcl:C-EUC0805
- added C2: 0.1µF, rcl:C-EUC0805
- added C5: 22µF, rcl:C-EUC0805
- added C9: 2.2µF / 25V, rcl:C-EUC0805
- added D1: BZG05C3V6-E3-TR3, zener:ZENER
- added IC1: TPS63031, TPS63031 - Buck Boost Voltage Regulator:TPS63001DRCR
- added Q1: BSS84, transistor-small-signal:BSS84
- added R1: 10k, resistor:R-EU_R0805
- added R3: 270k, rcl:R-EU_R0805
- added R7: 47k, rcl:R-EU_R0805
- added R8: 390k, rcl:R-EU_R0805
- added S1: POWER SWITCH, smd-special:SWS001
- added U3: MCP73871-2AAI/ML, MCP73871 - Powerpath and Charge Controller:MCP73871-2AAI/ML
- C10: value 0.1µF -> 10µF; device resistor:C-EUC0805 -> rcl:C-EUC0805
- C11: value 1µF -> 10µF; device rcl:C-EUC0805 -> resistor:C-EUC0805
- C12: value 1µF -> 1000µF; device rcl:C-EUC0805 -> rcl:CPOL-EUE5-10.5
- C14: value 2.2µF / 25V -> 10µF; device rcl:C-EUC0805 -> resistor:C-EUC0805
- C3: value 10µF -> 1µF
- C4: value 0.1µF -> 1µF
- C8: value 22µF -> 10µF
- D2: value BZG05C3V6-E3-TR3 -> SZ1SMB5916BT3G; device zener:ZENER -> diode:DIODE-SMB
- D3: value SZ1SMB5916BT3G -> BAT60AE6327; device diode:DIODE-SMB -> diode:BAT60J
- IC2: value TPS63031 -> RN4678_BT_MODULE; device TPS63031 - Buck Boost Voltage Regulator:TPS63001DRCR -> RN4678 Bluetooth 4.2 Dual Mode:RN4678_BT_MODULE
- IC3: value FT230XS -> MAX6818; device ftdichip:FT230XS -> MAX6818 CMOS Switch debouncer:MAX6818
- R10: value 100k -> 10k; device rcl:R-EU_R0805 -> resistor:R-EU_R0805
- R11: value 270k -> 1k; device rcl:R-EU_R0805 -> resistor:R-EU_R0805
- R12, R13: value 1k -> 10k
- R14: value 47k -> 1k
- R16: value 1k -> 100k
- R17: value 47k -> 270k
- R18: value 1k -> NTC 10k; device resistor:R-EU_R0805 -> rcl:R-EU_0204/5
- R19: value 47k -> 150k
- R2: value 10k -> 100k; device resistor:R-EU_R0805 -> rcl:R-EU_R0805
- R20: value 390k -> 150k
- R4, R5: value 3k3 -> 47k
- R6: value 27 -> 1k
- R9: value 27 -> 10k
- U4: value MCP73871-2AAI/ML -> SN74LVC1G3157DBVR - GPS switch; device MCP73871 - Powerpath and Charge Controller:MCP73871-2AAI/ML -> Texas Instruments_By_element14_Batch_1:SN74LVC1G3157DBVR
Connections:
- net GPS_GREEN_LED renamed LED_GREEN
- net GPS_RED_LED renamed LED_RED
- net PC0 renamed LED_YELLOW
- net PC13 renamed GPS_YELLOW_LED
- removed net CBUS1: IC3.CBUS1, LED2.C
- removed net CBUS2: IC3.CBUS2, LED1.C
- removed net D+: CONN1.D+, IC7.4
- removed net D-: CONN1.D-, IC7.2
- removed net GREEN_LED: LED3.C, R15.2
- removed net ID: CONN1.ID, IC7.5
- removed net N$10: C10.1, IC3.!RESET, IC3.3V3OUT, IC3.VCCIO
- removed net N$4: F1.2, IC7.1
- removed net RED_LED: LED4.C, R16.2
- removed net RXD: IC3.RXD, R5.2
- removed net TXD: IC3.TXD, R4.2
- removed net USBDM: IC3.USBDM, R9.1
- removed net USBDP: IC3.USBDP, R6.2
- removed net USB_D+: IC7.7, R6.1
- removed net USB_D-: IC7.9, R9.2
- removed net USB_ID: IC7.6
- removed net USB_RX_LED: LED1.A, R12.2
- removed net USB_TX_LED: LED2.A, R13.2
- removed net VUSB: CONN1.VBUS, F1.1, R12.1, R13.1
- new net ADXL345_INT2: IC1.INT2
- new net FORCE-ON: IC1.FORCE-ON
- new net FRAM_!HOLD!: IC1.!HOLD!
- new net FRAM_!WP!: IC1.!WP!
- new net GREEN: Q1.G
- new net G_A: Q1.D
- new net G_C: R3.1
- new net R_C: R1.1
- new net TX: R1.1
- new net VGPS: C1.1, C2.1, IC1.VCC
- new net WAKEUP: IC1.WAKEUP
- new net Y_C: R2.1
- net !RESET!: now also IC1.!RESET!
- net 3V3: now also C1.1, C2.1, IC1.DET, IC1.VCC, IC1.VDD, IC1.VDDIO, IC1.VS, R1.2, R2.2, R3.2
- net ADXL345SDA: now also IC1.SDA
- net ADXL345_CS: now also IC1.!CS!
- net ADXL345_INT1: now also IC1.INT1
- net ANALOG_SW_CTRL_PIN: now also U4.S; no longer U5.S
- net BAT_A_PIN: now also R19.2, R20.1; no longer R32.2, R33.1
- net BLUETOOTH_PROF_IND_PIN: now also IC2.P0_5; no longer IC4.P0_5
- net BLUETOOTH_RX: now also IC2.RXD; no longer IC4.RXD
- net BLUETOOTH_SWITCH_PIN: now also IC2.SW_BTN, R13.2; no longer IC4.SW_BTN, R25.2
- net BLUETOOTH_TX: now also IC2.TXD, U4.B1; no longer IC4.TXD, U5.B1
- net BLUETOOTH_WAKEUP_PIN: now also IC2.WAKEUP, R12.2; no longer IC4.WAKEUP, R24.2
- net BT_LED: now also IC2.LED, R6.1; no longer IC4.LED, R18.1
- net BUTTON_BLUETOOTH: now also IC3.IN7; no longer IC6.IN7
- net BUTTON_CENTER: now also IC3.IN5; no longer IC6.IN5
- net BUTTON_DOWN: now also IC3.IN2; no longer IC6.IN2
- net BUTTON_GPRS: now also IC3.IN8; no longer IC6.IN8
- net BUTTON_LEFT: now also IC3.IN4; no longer IC6.IN4
- net BUTTON_RIGHT: now also IC3.IN3; no longer IC6.IN3
- net BUTTON_UP: now also IC3.IN6; no longer IC6.IN6
- net CAP1N: now also C3.1; no longer C6.1
- net CAP1P: now also C3.2; no longer C6.2
- net CAP2N: now also C4.1; no longer C7.1
- net CAP2P: now also C4.2; no longer C7.2
- net EN: now also IC1.EN, R1.2, S1.1; no longer IC2.EN, R2.2, S2.1
- net GND: now also C1.1, C1.2, C11.2, C12.-, C13.2, C14.2, C2.2, C5.1, C6.1, C7.1, C9.1, D1.AN, D2.A, IC1.GND, IC1.PGND, IC1.POWERPAD, IC1.VSS, IC3.!EN!, Q1.D, Q1.S, R1.1, R12.1, R13.1, R15.2, R16.2, R17.2, R18.2, R20.2, R3.2, R8.1, R9.2, U3.GND1, U3.GND2, U3.GND3, U3.GND4, U3.GND5, U3.GND6, U4.GND; no longer C11.1, C12.1, C13.1, C14.1, C15.2, C17.2, C18.-, C22.2, C24.-, C24.2, C27.1, C3.1, CONN1.GND1, CONN1.GND2, CONN1.GND3, CONN1.GND4, CONN1.GND5, D2.AN, D3.A, IC2.PGND, IC2.POWERPAD, IC3.GND@1, IC4.GND, IC6.!EN!, IC6.GND, IC7.GND, Q2.D, R11.2, R2.1, R20.1, R21.2, R24.1, R25.1, R28.2, R29.2, R30.2, R31.2, R33.2, U4.GND1, U4.GND2, U4.GND3, U4.GND4, U4.GND5, U4.GND6, U5.GND
- net GPRS_NETLIGHT: now also R10.1, R9.1; no longer R21.1, R22.1
- net GPRS_NETLIGHT_GATE: now also Q1.G, R10.2; no longer Q2.G, R22.2
- net GPS_GREEN_LED_PIN: no longer R15.1
- net GPS_MCU_TX: now also U4.B2; no longer U5.B2
- net GPS_RED_LED_PIN: no longer R16.1
- net GPS_RX: now also IC1.RX
- net GPS_SW_SERIAL_RX: now also U4.A; no longer U5.A
- net GPS_TX: now also IC1.TX, R1.2; no longer C22.1
- net IREF: now also R8.2; no longer R20.2
- net L2: now also R6.2; no longer R18.2
- net LDO33_O: now also IC2.LDO33_O, IC2.VDD_IO; no longer IC4.LDO33_O, IC4.VDD_IO
- net L_L1: now also IC1.L1; no longer IC2.L1
- net L_L2: now also IC1.L2; no longer IC2.L2
- net MCP73871_CHARGE_STATUS_1_PIN: now also R7.2, U3.STAT1/!LBO!; no longer R19.2, U4.STAT1/!LBO!
- net MCP73871_CHARGE_STATUS_2_PIN: now also R5.2, U3.STAT2; no longer R17.2, U4.STAT2
- net MCP73871_POWER_GOOD_PIN: now also R4.2, U3.!PG!; no longer R14.2, U4.!PG!
- net MENU_BLUETOOTH_POWER_BUTTON_PIN: now also IC3.OUT7; no longer IC6.OUT7
- net MENU_CENTER_BUTTON_PIN: now also IC3.OUT5; no longer IC6.OUT5
- net MENU_DOWN_BUTTON_PIN: now also IC3.OUT2; no longer IC6.OUT2
- net MENU_GPRS_POWER_BUTTON_PIN: now also IC3.OUT8; no longer IC6.OUT8
- net MENU_LEFT_BUTTON_PIN: now also IC3.OUT4; no longer IC6.OUT4
- net MENU_RIGHT_BUTTON_PIN: now also IC3.OUT3; no longer IC6.OUT3
- net MENU_UP_BUTTON_PIN: now also IC3.OUT6; no longer IC6.OUT6
- net N$1: now also R11.1; no longer R23.1
- net N$11: now also IC2.!RST_N!; no longer IC4.!RST_N!
- net N$19: now also R14.2, R17.1, R18.1; no longer R27.2, R30.1, R31.1
- net N$3: now also Q1.S, R11.2; no longer Q2.S, R23.2
- net N$6: now also C12.+, D3.C; no longer C18.+, D4.C
- net OLD_5V0: now also D3.A, R2.1, U3.!TE!, U3.CE, U3.IN1, U3.IN2, U3.PROG2, U3.SEL; no longer C27.2, D4.A, IC3.VCC, IC7.10, R10.1, U4.!TE!, U4.CE, U4.IN1, U4.IN2, U4.PROG2, U4.SEL
- net PDI_UART0_CTS_PIN: no longer IC3.!CTS
- net PDI_UART0_RX_PIN: no longer R4.1
- net PDI_UART0_TX_PIN: no longer R5.1
- net PROG1: now also R15.1, U3.PROG1; no longer R28.1, U4.PROG1
- net PROG3: now also R16.1, U3.PROG3; no longer R29.1, U4.PROG3
- net SD_CD: now also IC1.POL
- net SENSE: now also C1.1
- net SPI1_FRAM_CS: now also IC1.!CS!
- net SPI1_MISO: now also IC1.DAT0, IC1.SDO, IC1.SO
- net SPI1_MOSI: now also IC1.CMD, IC1.SI
- net SPI1_SCK: now also IC1.CLK, IC1.SCK, IC1.SCL
- net SPI1_SD_CS: now also IC1.CD/DAT3
- net THERM: now also R14.1, U3.THERM; no longer R27.1, U4.THERM
- net VCC: now also C10.1, C13.1, C5.2, C6.2, C7.2, D1.CAT, D2.C, IC1.FB, IC1.VOUT, IC2.BAT_IN, IC3.VCC, R4.1, R5.1, R7.1, U4.VCC; no longer C11.2, C12.2, C13.2, C15.1, C22.1, D2.CAT, D3.C, IC2.FB, IC2.VOUT, IC4.BAT_IN, IC6.VCC, LED3.A, LED4.A, R14.1, R17.1, R19.1, U5.VCC
- net VCOMH: now also C9.2; no longer C14.2
- net VMID: now also C1.1
- net VOUT: no longer C24.+
- net VPCC: now also R2.2, R3.1, U3.VPCC; no longer R10.2, R11.1, U4.VPCC
- net V_LIION+: now also C14.1, R19.1, U3.VBAT1, U3.VBAT2, U3.VBAT_SENSE; no longer C24.1, R32.1, U4.VBAT1, U4.VBAT2, U4.VBAT_SENSE
- net V_LIION_REGULATED: now also C1.2, C11.1, C2.1, IC1.PS/SYNC, IC1.VIN, IC1.VINA, S1.2, U3.OUT1, U3.OUT2; no longer C17.1, C3.2, C4.1, IC2.PS/SYNC, IC2.VIN, IC2.VINA, S2.2, U4.OUT1, U4.OUT2
Other:
- note added: "Vf = 2.2V R = 1.1V/20mA = 55 Ohm / 125mW"
- note added: "Vf = 2.65V R = 0.65V/20mA = 32 Ohm / 125mW"
- note added: "Vf = 2V R = 1.3V/20mA = 65 Ohm / 125mW"
- note removed: "Status LEDs"
- moved on the sheet: C10, C11, C13, C14, C3, C4, C6, C7, C8, R10, R11, R12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
