File: eagle design/misko_nucleo.brd (EAGLE design)
At the start: 115 x 115 mm, 132 parts, among them CN1 LiPo Battery, IC1 MC1525TT, IC10 LTC4425, IC101 ADXL345, IC102 74HCT1G32GW, IC11 SP3012-04UTG, IC2 ORG1510-MK4, IC3 TPS63031, IC4 FT230XS, IC5 RN4678_BT_MODULE, IC8 DS1394U-33+, IC9 MAX6818, Q1 ABM3B-8MHZ-10-1-U-T, Q2 BSS84, Q3 LFXTAL016178R, SW1 MICROJOYSTICK, SW2 PB6156RSL, SW3 PB6156RSL, U1 SN74LVC1G3157DBVR - BT switch, U2 ATMEGA1281-16AU, U3 TPS3808G33DBVT, U4 TMP36GRTZ, U5 MCP73871-2AAI/ML, U6 SN74LVC1G3157DBVR - GPS switch, X1 FH12-30S-0.5SH

Commit message: - moved gps components into misko nucleo schematic - corrected component library issues
Parts:
- removed C28, C38: 0.1µF, rcl:C0805
- removed C30, C33: 1000µF, rcl:E5-10,5
- removed C32: 10µF, resistor:C0805
- removed C34, C35: 100µF, rcl:C0805
- removed C36, C37: 0.1µF, resistor:C0805
- removed IC10: LTC4425, LTC4425 Supercap Charger:MSOP
- removed IC8: DS1394U-33+, DS1394U-33+ RTC SPI Module:10UMAX
- removed R34: 100k, rcl:R0805
- removed R35: 270k, rcl:R0805
- removed R36: NTC 10k, rcl:0204/5
- removed R38, R39: 150k, rcl:R0805
- removed R40, R41: 470k, resistor:R0805
- removed U6: SN74LVC1G3157DBVR - GPS switch, Texas Instruments_By_element14_Batch_1:SOT95P280X145-6N
- added GPS:ORG1510:C2: 1u / 16V, resistor:C0402
- added GPS:ORG1510:C22, GPS:ORG1510:C31: 18p / 16V, rcl:C0402
- added GPS:ORG1510:IC2: ORG1510MK4, ORG1510-MK4 GPS module:PACKAGE
- added GPS:SUPERCAP_CHARGER:C1, GPS:SUPERCAP_CHARGER:C34: 100u / 16V, rcl:C1210
- added GPS:SUPERCAP_CHARGER:C24: 1.5F, EECS5R5H155 Supercap:TH
- added GPS:SUPERCAP_CHARGER:C38, GPS:VOLTAGE_SUPERVISOR:C2: 0.1u / 16V, rcl:C0402
- added GPS:SUPERCAP_CHARGER:IC2: (no value), LTC4425 Supercap Charger:MSOP-12
- added GPS:SUPERCAP_CHARGER:R14: 10k, resistor:R0402
- added GPS:SUPERCAP_CHARGER:R18: 1k, resistor:R0402
- added GPS:SUPERCAP_CHARGER:R40, GPS:SUPERCAP_CHARGER:R41: 150k, resistor:R0402
- added GPS:VOLTAGE_SUPERVISOR:C1: 1n / 16V, rcl:C0402
- added GPS:VOLTAGE_SUPERVISOR:IC2: TPS3808G33DBVT, TPS3808 - Supervisory Circuit:SOT23-6
- added GPS:VOLTAGE_SUPERVISOR:R18: 1M, resistor:R0402
- added R18: 1k, resistor:R0805
- C1: value 18pF -> 0.1µF; device rcl:C0805 -> resistor:C0805
- C10: value 1µF -> 0.1µF; device rcl:C0805 -> resistor:C0805
- C11: value 22µF -> 1µF
- C12: value 7pF -> 1µF; device resistor:C0805 -> rcl:C0805
- C13, C3: value 0.1µF -> 10µF; device resistor:C0805 -> rcl:C0805
- C14: value 1µF -> 2.2µF / 25V
- C15, C2: value 1µF -> 10µF
- C16: value 10µF -> 0.1µF; device rcl:C0805 -> resistor:C0805
- C17: value 2.2µF / 25V -> 10µF; device rcl:C0805 -> resistor:C0805
- C18: value 1nF -> 1000µF; device rcl:C0805 -> rcl:E5-10,5
- C19: value 10µF -> 1000µF; device rcl:C0805 -> rcl:E5-10,5
- C20: value 0.1µF -> 1000µF; device rcl:C0805 -> rcl:E5-10,5
- C21: device resistor:C0805 -> rcl:C0805
- C23: value 10µF -> 1000µF; device resistor:C0805 -> rcl:E5-10,5
- C24: value 1.5F -> 10µF; device EECS5R5H155 Supercap:TH -> resistor:C0805
- C26, C27: value 1000µF -> 0.1µF; device rcl:E5-10,5 -> resistor:C0805
- C4: value 10µF -> 0.1µF; device resistor:C0805 -> rcl:C0805
- C5: value 10µF -> 7pF; device rcl:C0805 -> resistor:C0805
- C6: value 0.1µF -> 1µF
- C7: value 18pF -> 1µF; device resistor:C0805 -> rcl:C0805
- C8: value 7pF -> 22µF; device resistor:C0805 -> rcl:C0805
- C9: value 1µF -> 7pF; device rcl:C0805 -> resistor:C0805
- IC2: value ORG1510-MK4 -> TPS63031; device ORG1510-MK4 GPS module:PACKAGE -> TPS63031 - Buck Boost Voltage Regulator:SMT
- IC3: value TPS63031 -> FT230XS; device TPS63031 - Buck Boost Voltage Regulator:SMT -> ftdichip:SSOP16
- IC4: value FT230XS -> RN4678_BT_MODULE; device ftdichip:SSOP16 -> RN4678 Bluetooth 4.2 Dual Mode:SMT
- IC5: value RN4678_BT_MODULE -> DS1394U-33+; device RN4678 Bluetooth 4.2 Dual Mode:SMT -> DS1394U-33+ RTC SPI Module:10UMAX
- R14: value 10k -> 47k; device resistor:R0805 -> rcl:R0805
- R15: value 47k -> 1k
- R17: value 1k -> 47k
- R20: value 1k -> 390k; device resistor:R0805 -> rcl:R0805
- R21: value 47k -> 10k; device rcl:R0805 -> resistor:R0805
- R22: value 390k -> 10k; device rcl:R0805 -> resistor:R0805
- R23: value 10k -> 1k
- R25: value 1k -> 10k
- R26: value 1M -> 10k; device resistor:R0805 -> rcl:R0805
- R27, R28: value 10k -> 1k; device resistor:R0805 -> rcl:R0805
- R29: value 10k -> 100k
- R30: value 1k -> 270k
- R31: value 1k -> NTC 10k; device rcl:R0805 -> rcl:0204/5
- R32: value 1k -> 150k; device resistor:R0805 -> rcl:R0805
- R33: value 10k -> 150k; device resistor:R0805 -> rcl:R0805
- U3: value TPS3808G33DBVT -> TMP36GRTZ; device Texas Instruments_By_element14_Batch_1:SOT95P280X145-6N -> TMP36GRTZ:SOT95P280X145-5N
- U4: value TMP36GRTZ -> MCP73871-2AAI/ML; device TMP36GRTZ:SOT95P280X145-5N -> MCP73871 - Powerpath and Charge Controller:QFN50P400X400X100-21N
- U5: value MCP73871-2AAI/ML -> SN74LVC1G3157DBVR - GPS switch; device MCP73871 - Powerpath and Charge Controller:QFN50P400X400X100-21N -> Texas Instruments_By_element14_Batch_1:SOT95P280X145-6N
- moved C19 107.9 mm to (115.2, 118.0), flipped to the top
- moved R20 97.0 mm to (103.8, 67.5)
- moved C7 93.6 mm to (92.2, 67.5), turned to 0 degrees
- moved C10 89.4 mm to (181.5, 73.0)
- moved C1 80.3 mm to (111.8, 16.8), turned to 180 degrees
- moved C15 79.8 mm to (163.5, 21.5), flipped to the bottom, turned to 270 degrees
- moved C18 76.5 mm to (135.2, 118.0)
- moved C3 75.4 mm to (159.0, 75.5), turned to 90 degrees
- moved C13 74.0 mm to (107.8, 67.5), flipped to the top, turned to 180 degrees
- moved C20 72.5 mm to (195.2, 118.0), turned to 270 degrees
- moved R23 66.2 mm to (194.2, 35.8), turned to 90 degrees
- moved C17 65.9 mm to (173.2, 74.5), flipped to the top, turned to 270 degrees
- moved C6 60.9 mm to (96.2, 67.5), turned to 0 degrees
- moved C11 58.8 mm to (94.2, 67.5), flipped to the top, turned to 0 degrees
- moved R17 57.2 mm to (143.0, 78.0)
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- renumbered C29 to C22, IC11 to IC7, IC9 to IC6
Connections:
- removed net GPS_ON_OFF: IC2.ON_OFF, R26.1, U3.1
- removed net LTC4425_EN: IC10.EN, R32.2
- removed net LTC4425_PROG: IC10.PROG, R33.2
- removed net PFI: IC10.PFI, R40.1, R41.2
- removed net PFI_RET: IC10.PFI_RET, R41.1
- removed net UART1_RX: BRD1.CN10_26, BRD1.CN10_37
- removed net UART1_TX: BRD1.CN10_28, BRD1.CN10_35
- removed net VMID: C34.2, C35.2, IC10.VMID
- new net GPS:GPS_ON_OFF: GPS:ORG1510:IC2.1_ON_OFF, GPS:VOLTAGE_SUPERVISOR:IC2.!RESET!, GPS:VOLTAGE_SUPERVISOR:R18.1
- new net GPS:SUPERCAP_CHARGER:EN: GPS:SUPERCAP_CHARGER:IC2.EN, GPS:SUPERCAP_CHARGER:R18.2
- new net GPS:SUPERCAP_CHARGER:PFI: GPS:SUPERCAP_CHARGER:IC2.PFI, GPS:SUPERCAP_CHARGER:R40.1, GPS:SUPERCAP_CHARGER:R41.2
- new net GPS:SUPERCAP_CHARGER:PFI_RET: GPS:SUPERCAP_CHARGER:IC2.PFI_RET, GPS:SUPERCAP_CHARGER:R41.1
- new net GPS:SUPERCAP_CHARGER:PROG: GPS:SUPERCAP_CHARGER:IC2.PROG, GPS:SUPERCAP_CHARGER:R14.2
- new net GPS:SUPERCAP_CHARGER:VMID: GPS:SUPERCAP_CHARGER:C1.1, GPS:SUPERCAP_CHARGER:C34.2, GPS:SUPERCAP_CHARGER:IC2.VMID
- new net GPS:VGPS: GPS:ORG1510:C2.1, GPS:ORG1510:IC2.4_VCC, GPS:SUPERCAP_CHARGER:C24.+, GPS:SUPERCAP_CHARGER:C34.1, GPS:SUPERCAP_CHARGER:IC2.VOUT1, GPS:SUPERCAP_CHARGER:IC2.VOUT2, GPS:VOLTAGE_SUPERVISOR:C1.1, GPS:VOLTAGE_SUPERVISOR:IC2.SENSE
- new net GPS:VOLTAGE_SUPERVISOR:3V3: GPS:VOLTAGE_SUPERVISOR:C2.1, GPS:VOLTAGE_SUPERVISOR:IC2.VDD, GPS:VOLTAGE_SUPERVISOR:R18.2
- net 3V3: now also GPS:SUPERCAP_CHARGER:C38.1, GPS:SUPERCAP_CHARGER:IC2.FB, GPS:SUPERCAP_CHARGER:IC2.SEL, GPS:SUPERCAP_CHARGER:IC2.VIN1, GPS:SUPERCAP_CHARGER:IC2.VIN2, GPS:SUPERCAP_CHARGER:R18.1, GPS:SUPERCAP_CHARGER:R40.2
- net ANALOG_SW_CTRL_PIN: now also U5.6; no longer U6.6
- net AREF: now also C2.1; no longer C4.1
- net AVCC: now also C26.2; no longer C36.2
- net BAT_A_PIN: now also R32.2, R33.1; no longer R38.2, R39.1
- net BLUETOOTH_PROF_IND_PIN: now also IC4.P0_5; no longer IC5.P0_5
- net BLUETOOTH_RX: now also IC4.RXD; no longer IC5.RXD
- net BLUETOOTH_SWITCH_PIN: now also IC4.SW_BTN, R25.2; no longer IC5.SW_BTN, R28.2
- net BLUETOOTH_TX: now also IC4.TXD, U5.3; no longer IC5.TXD, U6.3
- net BLUETOOTH_WAKEUP_PIN: now also IC4.WAKEUP, R24.2; no longer IC5.WAKEUP, R27.2
- net BT_LED: now also IC4.LED, R18.1; no longer IC5.LED, R20.1
- net CAP1N: now also C6.1; no longer C9.1
- net CAP1P: now also C6.2; no longer C9.2
- net CAP2N: now also C7.1; no longer C10.1
- net CAP2P: now also C7.2; no longer C10.2
- net CBUS1: now also IC3.14; no longer IC4.14
- net CBUS2: now also IC3.7; no longer IC4.7
- net EN: now also IC2.6_EN; no longer IC3.6_EN
- net GND: now also C1.1, C10.2, C13.1, C15.2, C16.2, C17.2, C18.-, C19.-, C20.-, C23.-, C24.2, C26.1, C27.1, C9.1, GPS:ORG1510:C2.2, GPS:ORG1510:C22.2, GPS:ORG1510:C31.2, GPS:ORG1510:IC2.5_GND, GPS:ORG1510:IC2.GND1, GPS:ORG1510:IC2.GND10, GPS:ORG1510:IC2.GND11, GPS:ORG1510:IC2.GND12, GPS:ORG1510:IC2.GND13, GPS:ORG1510:IC2.GND14, GPS:ORG1510:IC2.GND15, GPS:ORG1510:IC2.GND2, GPS:ORG1510:IC2.GND4, GPS:ORG1510:IC2.GND5, GPS:ORG1510:IC2.GND6, GPS:ORG1510:IC2.GND7, GPS:ORG1510:IC2.GND8, GPS:ORG1510:IC2.GND9, GPS:SUPERCAP_CHARGER:C1.2, GPS:SUPERCAP_CHARGER:C24.-, GPS:SUPERCAP_CHARGER:C38.2, GPS:SUPERCAP_CHARGER:IC2.GND, GPS:SUPERCAP_CHARGER:R14.1, GPS:VOLTAGE_SUPERVISOR:C1.2, GPS:VOLTAGE_SUPERVISOR:C2.2, GPS:VOLTAGE_SUPERVISOR:IC2.GND, IC2.3_PGND, IC2.9_GND1, IC3.13, IC3.5, IC4.GND, IC4.GND1, IC4.GND10, IC4.GND11, IC4.GND12, IC4.GND2, IC4.GND3, IC4.GND4, IC4.GND5, IC4.GND6, IC4.GND7, IC4.GND8, IC4.GND9, R20.1, R21.2, R24.1, R25.1, R28.2, R29.2, R30.2, R33.2, U3.5, U4.10_GND1, U4.11_GND2, U4.GND2, U4.GND3, U4.GND4, U4.GND5, U4.GND6, U5.2; no longer C1.2, C13.2, C15.1, C16.1, C17.1, C18.2, C19.2, C20.1, C23.2, C24.-, C26.-, C27.-, C28.2, C30.-, C32.2, C33.-, C35.1, C36.1, C37.1, C38.1, C6.2, C7.1, IC10.GND1, IC10.GND2, IC10.GND3, IC2.GND1, IC2.GND5, IC3.3_PGND, IC3.9_GND1, IC3.GND2, IC3.GND3, IC3.GND4, IC4.13, IC4.5, IC5.GND1, IC5.GND10, IC5.GND11, IC5.GND12, IC5.GND2, IC5.GND3, IC5.GND4, IC5.GND5, IC5.GND6, IC5.GND7, IC5.GND8, IC5.GND9, IC8.GND, R14.2, R22.1, R23.2, R27.1, R28.1, R33.1, R34.2, R35.2, R36.2, R39.2, U3.2, U4.5, U5.10_GND1, U5.11_GND2, U5.GND2, U5.GND3, U5.GND4, U5.GND5, U5.GND6, U6.2
- net GPRS_NETLIGHT: now also R21.1, R22.1; no longer R23.1, R24.1
- net GPRS_NETLIGHT_GATE: now also R22.2; no longer R24.2
- net GPS_GREEN_LED_PIN: now also R15.1; no longer R16.1
- net GPS_POWER_CTL_PIN: no longer R14.1, U3.3
- net GPS_PWR_CTRL: now also GPS:VOLTAGE_SUPERVISOR:IC2.!MR!
- net GPS_RED_LED_PIN: now also R16.1; no longer R17.1
- net GPS_SW_SERIAL_RX: now also U5.4; no longer U6.4
- net GPS_SW_SERIAL_TX: now also BRD1.CN10_28, BRD1.CN10_35, GPS:ORG1510:C31.1, GPS:ORG1510:IC2.RX_10; no longer C7.2, IC2.RX
- net GPS_TX: now also BRD1.CN10_26, BRD1.CN10_37, GPS:ORG1510:C22.1, GPS:ORG1510:IC2.3_TX, U5.1; no longer C1.1, IC2.TX, U6.1
- net GPS_WAKEUP_PIN: no longer IC2.WAKEUP
- net GPS_WKUP: now also GPS:ORG1510:IC2.WAKEUP_6
- net GREEN_LED: now also R15.2; no longer R16.2
- net IREF: now also R20.2; no longer R22.2
- net L2: now also R18.2; no longer R20.2
- net LDO18_O: now also IC4.LDO18_O; no longer IC5.LDO18_O
- net LDO33_O: now also IC4.LDO33_O, IC4.VDD_IO; no longer IC5.LDO33_O, IC5.VDD_IO
- net L_L1: now also IC2.4_L1; no longer IC3.4_L1
- net L_L2: now also IC2.2_L2; no longer IC3.2_L2
- net MCP73871_CHARGE_STATUS_1_PIN: now also R19.2, U4.8_STAT1; no longer R21.2, U5.8_STAT1
- net MCP73871_CHARGE_STATUS_2_PIN: now also R17.2, U4.7_STAT2; no longer R19.2, U5.7_STAT2
- net MCP73871_POWER_GOOD_PIN: now also R14.2, U4.!6_PG!; no longer R15.2, U5.!6_PG!
- net N$1: now also R23.1; no longer R25.1
- net N$10: now also C10.1, IC3.10, IC3.11, IC3.3; no longer C13.1, IC4.10, IC4.11, IC4.3
- net N$11: now also IC4.!RST_N!; no longer IC5.!RST_N!
- net N$19: now also R27.2, R30.1, R31.1; no longer R30.2, R35.1, R36.1
- net N$3: now also R23.2; no longer R25.2
- net N$31: now also C1.2; no longer C3.2
- net N$6: now also C18.+, C19.+, C20.+, C23.+; no longer C26.+, C27.+, C30.+, C33.+
- net OLD_5V0: now also C27.2, IC3.12, U4.17_CE, U4.18_IN1, U4.19_IN2, U4.3_SEL, U4.4_PROG2, U4.9_!TE!; no longer C37.2, IC4.12, U5.17_CE, U5.18_IN1, U5.19_IN2, U5.3_SEL, U5.4_PROG2, U5.9_!TE!
- net PDI_UART0_CTS_PIN: now also IC3.6; no longer IC4.6
- net PROG1: now also R28.1, U4.13_PROG1; no longer R31.1, U5.13_PROG1
- net PROG3: now also R29.1, U4.12_PROG3; no longer R34.1, U5.12_PROG3
- net RED_LED: now also R16.2; no longer R17.2
- net RTC_INT_INTERRUPT_PIN: now also IC5.!INT!; no longer IC8.!INT!
- net RTC_XTAL1: now also IC5.X1; no longer IC8.X1
- net RTC_XTAL2: now also IC5.X2; no longer IC8.X2
- net RXD: now also IC3.4; no longer IC4.4
- net SPI_MISO_PIN: now also IC5.DOUT; no longer IC8.DOUT
- net SPI_MOSI_PIN: now also IC5.DIN; no longer IC8.DIN
- net SPI_SCK_PIN: now also IC5.SCLK; no longer IC8.SCLK
- net SPI_SS_RTC_PIN: now also IC5.!CS!, R26.2; no longer IC8.!CS!, R29.2
- net THERM: now also R27.1, U4.5_THERM; no longer R30.1, U5.5_THERM
- net TMP36_VSENSE_PIN: now also U3.1; no longer U4.1
- net TXD: now also IC3.1; no longer IC4.1
- net USBDM: now also IC3.9; no longer IC4.9
- net USBDP: now also IC3.8; no longer IC4.8
- net VCC: now also C12.2, C13.2, C15.1, C16.1, C8.2, IC2.10_FB, IC2.1_VOUT, IC4.BAT_IN, IC5.VCC, R14.1, R17.1, R26.1, U3.2, U3.4, U5.5; no longer C14.2, C15.2, C16.2, C19.1, C20.2, C28.1, C38.2, IC10.FB, IC10.SEL, IC10.VIN1, IC10.VIN2, IC3.10_FB, IC3.1_VOUT, IC5.BAT_IN, IC8.VCC, R15.1, R21.1, R26.2, R29.1, R32.1, R40.2, U3.6, U4.2, U4.4, U6.5
- net VCOMH: now also C14.2; no longer C17.2
- net VGPS: now also IC5.VBACK; no longer C18.1, C2.1, C24.+, C34.1, IC10.VOUT1, IC10.VOUT2, IC2.VCC, IC8.VBACK, U3.5
- net VPCC: now also U4.2_VPCC; no longer U5.2_VPCC
- net V_LIION+: now also C24.1, R32.1, U4.14_VBAT1, U4.15_VBAT2, U4.16_BAT_SENSE; no longer C32.1, R38.1, U5.14_VBAT1, U5.15_VBAT2, U5.16_BAT_SENSE
- net V_LIION_REGULATED: now also C17.1, C3.2, C4.1, IC2.5_VIN, IC2.7_PS/SYNC, IC2.8_VINA, U4.1_OUT1, U4.20_OUT2; no longer C23.1, C5.2, C6.1, IC3.5_VIN, IC3.7_PS/SYNC, IC3.8_VINA, U5.1_OUT1, U5.20_OUT2
- net XTAL1: now also C9.2; no longer C12.2
- net XTAL2: now also C5.2; no longer C8.2
Routing:
- net GPS_WAKEUP_PIN: track 57.9 -> 0.00 mm
- net VGPS: track 101.5 -> 52.4 mm, vias 2 -> 1
- net GPS_POWER_CTL_PIN: track 46.4 -> 0.00 mm, vias 1 -> 0
- net GPS_TX: track 37.2 -> 0.76 mm, vias 1 -> 0
- net VCC: track 410.1 -> 385.2 mm, vias 16 -> 15
- net GPS_ON_OFF: track 21.5 -> 0.00 mm, vias 2 -> 0
- net VMID: track 15.0 -> 0.00 mm, vias 1 -> 0
- net UART1_TX: track 9.56 -> 0.00 mm
- net UART1_RX: track 9.56 -> 0.00 mm
- net GPS_SW_SERIAL_TX: track 92.8 -> 84.8 mm
- net PFI_RET: track 7.04 -> 0.00 mm, vias 1 -> 0
- net PFI: track 4.91 -> 0.00 mm, vias 1 -> 0
- net LTC4425_PROG: track 3.35 -> 0.00 mm
- net LTC4425_EN: track 3.16 -> 0.00 mm, vias 1 -> 0
- net GND: vias 40 -> 37
